Commit message: Rm head offset

File: triago_description/urdf/calibration_constants.urdf.xacro (robot description, xacro)
@@ -12,6 +12,4 @@
 	<xacro:property name="camera_orientation_p" value="0.0" />
 	<xacro:property name="camera_orientation_y" value="0.0" />
-	<xacro:property name="head_2_joint_offset" value="0" />
-	<xacro:property name="head_1_joint_offset" value="0" />
 	<xacro:property name="torso_lift_joint_offset" value="0" />
 	<xacro:property name="arm_left_1_joint_offset" value="0.0" />

Commit message: Adding arm head constant

File: triago_description/urdf/calibration_constants.urdf.xacro (robot description, xacro)
@@ -27,3 +27,10 @@
   	<xacro:property name="arm_right_6_joint_offset" value="0.0" />
   	<xacro:property name="arm_right_7_joint_offset" value="0.0" />
+	<xacro:property name="arm_head_1_joint_offset" value="0.0" />
+  	<xacro:property name="arm_head_2_joint_offset" value="0.0" />
+  	<xacro:property name="arm_head_3_joint_offset" value="0.0" />
+  	<xacro:property name="arm_head_4_joint_offset" value="0.0" />
+  	<xacro:property name="arm_head_5_joint_offset" value="0.0" />
+  	<xacro:property name="arm_head_6_joint_offset" value="0.0" />
+  	<xacro:property name="arm_head_7_joint_offset" value="0.0" />
 </robot>
