Commit message: reduce joint limits according to test with robot

File: triago_description/urdf/head_arm/arm_limits/spherical-wrist.limits.xacro (robot description, xacro)
@@ -5,6 +5,6 @@
   <xacro:property name="arm_6_joint_ub" value="172" />
   <xacro:property name="arm_6_joint_lb" value="-108" />
-  <xacro:property name="arm_7_joint_ub" value="148.97" />
-  <xacro:property name="arm_7_joint_lb" value="-148.97" />
+  <xacro:property name="arm_7_joint_ub" value="148.5" />
+  <xacro:property name="arm_7_joint_lb" value="-148.5" />
   <!-- Velocity limits -->
   <xacro:property name="arm_5_max_velocity" value="2.35" />
