Commit message: Fix wrist + update joint 6 limit + update motions

File: triago_description/urdf/head_arm/arm_limits/arm.limits.xacro (robot description, xacro)
@@ -6,10 +6,10 @@
   <xacro:property name="arm_k_velocity" value="20"/>
   <!-- Joint limits -->
-  <xacro:property name="arm_1_joint_ub" value="148.97" />
-  <xacro:property name="arm_1_joint_lb" value="-148.97" />
+  <xacro:property name="arm_1_joint_ub" value="210" />
+  <xacro:property name="arm_1_joint_lb" value="-90" />
   <xacro:property name="arm_2_joint_ub" value="63.03" />
   <xacro:property name="arm_2_joint_lb" value="-139.8" />
-  <xacro:property name="arm_3_joint_ub" value="148.97" />
-  <xacro:property name="arm_3_joint_lb" value="-148.97" />
+  <xacro:property name="arm_3_joint_ub" value="210" />
+  <xacro:property name="arm_3_joint_lb" value="-90" />
   <xacro:property name="arm_4_joint_ub" value="63.03" />
   <xacro:property name="arm_4_joint_lb" value="-139.8" />

File: triago_description/urdf/head_arm/arm_limits/spherical-wrist.limits.xacro (robot description, xacro)
@@ -3,6 +3,6 @@
   <xacro:property name="arm_5_joint_ub" value="210" />
   <xacro:property name="arm_5_joint_lb" value="-90" />
-  <xacro:property name="arm_6_joint_ub" value="114.59" />
-  <xacro:property name="arm_6_joint_lb" value="-114.59" />
+  <xacro:property name="arm_6_joint_ub" value="108" />
+  <xacro:property name="arm_6_joint_lb" value="-172" />
   <xacro:property name="arm_7_joint_ub" value="148.97" />
   <xacro:property name="arm_7_joint_lb" value="-148.97" />

File: triago_description/urdf/head_arm/arm_properties/spherical-wrist.properties.xacro (robot description, xacro)
@@ -19,5 +19,5 @@
     </xacro:macro>
     <xacro:macro name="origin_joint_6" params="reflect">
-        <origin xyz="0 -0.0422 0.1654" rpy="-1.5708 0 0" />
+        <origin xyz="0 -0.0422 0.1654" rpy="-1.5708 0 3.14" />
     </xacro:macro>
     <xacro:macro name="inertial_link_7" params="reflect">
@@ -29,5 +29,5 @@
     </xacro:macro>
     <xacro:macro name="origin_joint_7" params="reflect">
-        <origin xyz="-0.07 -0.0534 0.0422" rpy="1.5708 -1.5708 0" />
+        <origin xyz="0.07 -0.0534 -0.0422" rpy="1.5708 -1.5708 0" />
     </xacro:macro>
 </robot>

Commit message: Change joint 3 limits to match real configuration

File: triago_description/urdf/head_arm/arm_limits/arm.limits.xacro (robot description, xacro)
@@ -10,6 +10,6 @@
   <xacro:property name="arm_2_joint_ub" value="63.03" />
   <xacro:property name="arm_2_joint_lb" value="-139.8" />
-  <xacro:property name="arm_3_joint_ub" value="210" />
-  <xacro:property name="arm_3_joint_lb" value="-90" />
+  <xacro:property name="arm_3_joint_ub" value="148.97" />
+  <xacro:property name="arm_3_joint_lb" value="-148.97" />
   <xacro:property name="arm_4_joint_ub" value="63.03" />
   <xacro:property name="arm_4_joint_lb" value="-139.8" />

Commit message: update joint max velocity limit for tiago head arm

File: triago_description/urdf/head_arm/arm_limits/arm.limits.xacro (robot description, xacro)
@@ -15,8 +15,8 @@
   <xacro:property name="arm_4_joint_lb" value="-139.8" />
   <!-- Velocity limits -->
-  <xacro:property name="arm_1_max_velocity" value="1.95" />
-  <xacro:property name="arm_2_max_velocity" value="1.95" />
-  <xacro:property name="arm_3_max_velocity" value="2.35" />
-  <xacro:property name="arm_4_max_velocity" value="2.35" />
+  <xacro:property name="arm_1_max_velocity" value="2.50" />
+  <xacro:property name="arm_2_max_velocity" value="2.50" />
+  <xacro:property name="arm_3_max_velocity" value="2.50" />
+  <xacro:property name="arm_4_max_velocity" value="2.50" />
   <!-- Effort limits -->
   <xacro:property name="arm_1_max_effort" value="43.0" />

File: triago_description/urdf/head_arm/arm_limits/spherical-wrist.limits.xacro (robot description, xacro)
@@ -8,7 +8,7 @@
   <xacro:property name="arm_7_joint_lb" value="-148.5" />
   <!-- Velocity limits -->
-  <xacro:property name="arm_5_max_velocity" value="2.35" />
-  <xacro:property name="arm_6_max_velocity" value="2.35" />
-  <xacro:property name="arm_7_max_velocity" value="2.35" />
+  <xacro:property name="arm_5_max_velocity" value="2.50" />
+  <xacro:property name="arm_6_max_velocity" value="2.50" />
+  <xacro:property name="arm_7_max_velocity" value="2.50" />
   <!-- Effort limits -->
   <xacro:property name="arm_5_max_effort" value="26" />

Commit message: fix joint limit deleting the safety threshold

File: triago_description/urdf/head_arm/arm_limits/arm.limits.xacro (robot description, xacro)
@@ -6,12 +6,12 @@
   <xacro:property name="arm_k_velocity" value="20"/>
   <!-- Joint limits -->
-  <xacro:property name="arm_1_joint_ub" value="148.97" />
-  <xacro:property name="arm_1_joint_lb" value="-148.97" />
-  <xacro:property name="arm_2_joint_ub" value="63.03" />
-  <xacro:property name="arm_2_joint_lb" value="-139.8" />
-  <xacro:property name="arm_3_joint_ub" value="148.97" />
-  <xacro:property name="arm_3_joint_lb" value="-148.97" />
-  <xacro:property name="arm_4_joint_ub" value="63.03" />
-  <xacro:property name="arm_4_joint_lb" value="-139.8" />
+  <xacro:property name="arm_1_joint_ub" value="150" />
+  <xacro:property name="arm_1_joint_lb" value="-150" />
+  <xacro:property name="arm_2_joint_ub" value="65" />
+  <xacro:property name="arm_2_joint_lb" value="-140" />
+  <xacro:property name="arm_3_joint_ub" value="150" />
+  <xacro:property name="arm_3_joint_lb" value="-150" />
+  <xacro:property name="arm_4_joint_ub" value="65" />
+  <xacro:property name="arm_4_joint_lb" value="-140" />
   <!-- Velocity limits -->
   <xacro:property name="arm_1_max_velocity" value="2.50" />

File: triago_description/urdf/head_arm/arm_limits/spherical-wrist.limits.xacro (robot description, xacro)
@@ -5,6 +5,6 @@
   <xacro:property name="arm_6_joint_ub" value="172" />
   <xacro:property name="arm_6_joint_lb" value="-108" />
-  <xacro:property name="arm_7_joint_ub" value="148.5" />
-  <xacro:property name="arm_7_joint_lb" value="-148.5" />
+  <xacro:property name="arm_7_joint_ub" value="150" />
+  <xacro:property name="arm_7_joint_lb" value="-150" />
   <!-- Velocity limits -->
   <xacro:property name="arm_5_max_velocity" value="2.50" />

File: triago_description/urdf/head_arm/arm_limits/straight-wrist.limits.xacro (robot description, xacro)
@@ -1,10 +1,10 @@
 <robot xmlns:xacro="http://ros.org/wiki/xacro">
   <!-- Joint limits -->
-  <xacro:property name="arm_5_joint_ub" value="148.97" />
-  <xacro:property name="arm_5_joint_lb" value="-148.97" />
-  <xacro:property name="arm_6_joint_ub" value="114.59" />
-  <xacro:property name="arm_6_joint_lb" value="-114.59" />
-  <xacro:property name="arm_7_joint_ub" value="148.97" />
-  <xacro:property name="arm_7_joint_lb" value="-148.97" />
+  <xacro:property name="arm_5_joint_ub" value="150" />
+  <xacro:property name="arm_5_joint_lb" value="-150" />
+  <xacro:property name="arm_6_joint_ub" value="115" />
+  <xacro:property name="arm_6_joint_lb" value="-115" />
+  <xacro:property name="arm_7_joint_ub" value="150" />
+  <xacro:property name="arm_7_joint_lb" value="-150" />
   <!-- Velocity limits -->
   <xacro:property name="arm_5_max_velocity" value="2.35" />

Commit message: update vel limits

File: triago_description/urdf/head_arm/arm_limits/arm.limits.xacro (robot description, xacro)
@@ -15,8 +15,8 @@
   <xacro:property name="arm_4_joint_lb" value="-140" />
   <!-- Velocity limits -->
-  <xacro:property name="arm_1_max_velocity" value="2.50" />
-  <xacro:property name="arm_2_max_velocity" value="2.50" />
-  <xacro:property name="arm_3_max_velocity" value="2.50" />
-  <xacro:property name="arm_4_max_velocity" value="2.50" />
+  <xacro:property name="arm_1_max_velocity" value="1.95" />
+  <xacro:property name="arm_2_max_velocity" value="1.95" />
+  <xacro:property name="arm_3_max_velocity" value="3.95" />
+  <xacro:property name="arm_4_max_velocity" value="3.95" />
   <!-- Effort limits -->
   <xacro:property name="arm_1_max_effort" value="43.0" />

File: triago_description/urdf/head_arm/arm_limits/spherical-wrist.limits.xacro (robot description, xacro)
@@ -8,7 +8,7 @@
   <xacro:property name="arm_7_joint_lb" value="-150" />
   <!-- Velocity limits -->
-  <xacro:property name="arm_5_max_velocity" value="2.50" />
-  <xacro:property name="arm_6_max_velocity" value="2.50" />
-  <xacro:property name="arm_7_max_velocity" value="2.50" />
+  <xacro:property name="arm_5_max_velocity" value="3.95" />
+  <xacro:property name="arm_6_max_velocity" value="3.95" />
+  <xacro:property name="arm_7_max_velocity" value="3.95" />
   <!-- Effort limits -->
   <xacro:property name="arm_5_max_effort" value="26" />
