Commit message: Fix wrist inertia

File: triago_description/urdf/head_arm/arm_properties/arm.properties.xacro (robot description, xacro)
@@ -53,7 +53,7 @@
     <xacro:macro name="inertial_tool_changer_link" params="reflect">
         <inertial>
-            <origin xyz="0.0019481 0.0017558 -0.0084934" rpy="0 0 0" />
-            <mass value="0.12272" />
-            <inertia ixx="5.1385E-05" ixy="8.5364E-07" ixz="-9.0329E-08" iyy="4.7962E-05" iyz="-1.8035E-07" izz="9.2935E-05" />
+            <origin xyz="0.003414871500006 0.002458561521477 -0.001077004696741" rpy="0 0 0" />
+            <mass value="0.0655061851536" />
+            <inertia ixx="1.79461992752602E-05" ixy="1.70670100210845E-06" ixz="-2.54814948767968E-09" iyy="1.47274432150498E-05" iyz="1.09471559381518E-07" izz="3.12924968277541E-05" />
         </inertial>
     </xacro:macro>

File: triago_description/urdf/head_arm/arm_properties/spherical-wrist.properties.xacro (robot description, xacro)
@@ -2,7 +2,7 @@
     <xacro:macro name="inertial_link_5" params="reflect">
         <inertial>
-            <origin xyz="-1.1035E-05 -0.027586 0.067845" rpy="0 0 0" />
-            <mass value="0.31076" />
-            <inertia ixx="0.0014015" ixy="9.1728E-08" ixz="-9.3079E-08" iyy="0.0014" iyz="0.00032771" izz="0.00040201" />
+            <origin xyz="1.1053306160504E-05 -0.027586177392457 0.067845360860401" rpy="0 0 0" />
+            <mass value="0.310763344920608" />
+            <inertia ixx="0.001401450896582" ixy="9.16506225733395E-08" ixz="-9.26253840796548E-08" iyy="0.001399994200261" iyz="0.000327712970358816" izz="0.000402007894416599" />
         </inertial>
     </xacro:macro>
@@ -13,7 +13,7 @@
     <xacro:macro name="inertial_link_6" params="reflect">
         <inertial>
-            <origin xyz="-0.0083923 -0.00081501 0.039899" rpy="0 0 0" />
-            <mass value="0.83518" />
-            <inertia ixx="0.00077706" ixy="-0.00012999" ixz="-5.9554E-06" iyy="0.00094237" iyz="-1.5002E-06" izz="0.00086922" />
+            <origin xyz="0.031765231605914 -0.006515108863227 -0.040804517366422" rpy="0 0 0" />
+            <mass value="1.34587360139295" />
+            <inertia ixx="0.001098855044306" ixy="0.000130003468892" ixz="-5.88209416784623E-06" iyy="0.001164948561169" iyz="4.20092116284985E-07" izz="0.001189837857495" />
         </inertial>
     </xacro:macro>
@@ -23,7 +23,7 @@
     <xacro:macro name="inertial_link_7" params="reflect">
         <inertial>
-            <origin xyz="2.1788E-15 7.5568E-05 -0.037565" rpy="0 0 0" />
-            <mass value="0.51032" />
-            <inertia ixx="0.00032121" ixy="-1.7628E-21" ixz="-7.178E-21" iyy="0.00032034" iyz="-1.0206E-06" izz="0.00022179" />
+            <origin xyz="0.00095120830852 -0.000268585760924 1.45881142001869E-05" rpy="0 0 0" />
+            <mass value="0.057209493908896" />
+            <inertia ixx="3.32348045580924E-05" ixy="8.53056519363846E-07" ixz="-2.89819873727239E-07" iyy="3.34386146857115E-05" iyz="8.77813050093602E-08" izz="6.16426730349172E-05" />
         </inertial>
     </xacro:macro>
