Commit message: Inverse joint 6 rotation + update motions accordingly

File: triago_description/urdf/head_arm/arm.urdf.xacro (robot description, xacro)
@@ -183,5 +183,5 @@
       <parent link="${name}_5_link" />
       <child link="${name}_6_link" />
-      <axis xyz="0 0 1" />
+      <axis xyz="0 0 -1" />
       <limit lower="${arm_6_joint_lb * deg_to_rad}" upper="${arm_6_joint_ub * deg_to_rad}" effort="${arm_6_max_effort}" velocity="${arm_6_max_velocity}" />
       <dynamics friction="${arm_friction}" damping="${arm_damping}"/>

File: triago_description/urdf/head_arm/arm_limits/arm.limits.xacro (robot description, xacro)
@@ -6,6 +6,6 @@
   <xacro:property name="arm_k_velocity" value="20"/>
   <!-- Joint limits -->
-  <xacro:property name="arm_1_joint_ub" value="210" />
-  <xacro:property name="arm_1_joint_lb" value="-90" />
+  <xacro:property name="arm_1_joint_ub" value="148.97" />
+  <xacro:property name="arm_1_joint_lb" value="-148.97" />
   <xacro:property name="arm_2_joint_ub" value="63.03" />
   <xacro:property name="arm_2_joint_lb" value="-139.8" />

File: triago_description/urdf/head_arm/arm_limits/spherical-wrist.limits.xacro (robot description, xacro)
@@ -3,6 +3,6 @@
   <xacro:property name="arm_5_joint_ub" value="210" />
   <xacro:property name="arm_5_joint_lb" value="-90" />
-  <xacro:property name="arm_6_joint_ub" value="108" />
-  <xacro:property name="arm_6_joint_lb" value="-172" />
+  <xacro:property name="arm_6_joint_ub" value="172" />
+  <xacro:property name="arm_6_joint_lb" value="-108" />
   <xacro:property name="arm_7_joint_ub" value="148.97" />
   <xacro:property name="arm_7_joint_lb" value="-148.97" />

Commit message: add material + fix 7th joint

File: triago_description/urdf/head_arm/arm.urdf.xacro (robot description, xacro)
@@ -227,7 +227,5 @@
             <mesh filename="package://pal_sea_arm_description/meshes/${mesh_folder}/tool_changer_link.stl" scale="1 1 ${reflect}" />
           </geometry>
-          <material name="">
-            <color rgba="0.29804 0.29804 0.29804 1" />
-          </material>
+          <material name="pal/DarkGrey"/>
         </visual>
         <collision>

File: triago_description/urdf/head_arm/arm_properties/spherical-wrist.properties.xacro (robot description, xacro)
@@ -29,5 +29,5 @@
     </xacro:macro>
     <xacro:macro name="origin_joint_7" params="reflect">
-        <origin xyz="0.07 -0.0534 -0.0422" rpy="1.5708 -1.5708 0" />
+        <origin xyz="0.07 -0.0534 -0.0422" rpy="1.5708 0 0" />
     </xacro:macro>
 </robot>

Commit message: Add correct mesh for head arm

File: triago_description/urdf/head_arm/arm.urdf.xacro (robot description, xacro)
@@ -147,5 +147,5 @@
         <origin xyz="0 0 0" rpy="0 0 0" />
         <geometry>
-          <mesh filename="package://pal_sea_arm_description/meshes/${mesh_folder}/${wrist_model}/arm_5_link_collision.stl" scale="1 1 ${reflect}" />
+          <mesh filename="package://pal_sea_arm_description/meshes/${mesh_folder}/${wrist_model}/arm_5_link.stl" scale="1 1 ${reflect}" />
         </geometry>
       </collision>

Commit message: Removing collision arm 7 link

File: triago_description/urdf/head_arm/arm.urdf.xacro (robot description, xacro)
@@ -198,10 +198,4 @@
         <material name="pal/DarkGrey"/>
       </visual>
-      <collision>
-        <origin xyz="0 0 0" rpy="0 0 0" />
-        <geometry>
-          <mesh filename="package://pal_sea_arm_description/meshes/${mesh_folder}/${wrist_model}/arm_7_link_collision.stl" scale="1 1 ${reflect}" />
-        </geometry>
-      </collision>
     </link>
     <!-- ARM 7 JOINT -->

Commit message: Adding simplified mesh

File: triago_description/urdf/head_arm/arm.urdf.xacro (robot description, xacro)
@@ -198,4 +198,10 @@
         <material name="pal/DarkGrey"/>
       </visual>
+      <collision>
+        <origin xyz="0 0 0" rpy="0 0 0" />
+        <geometry>
+          <cylinder radius="0.0375" length="0.0366"/>
+        </geometry>
+      </collision>
     </link>
     <!-- ARM 7 JOINT -->

Commit message: Change back to collision model

File: triago_description/urdf/head_arm/arm.urdf.xacro (robot description, xacro)
@@ -147,5 +147,5 @@
         <origin xyz="0 0 0" rpy="0 0 0" />
         <geometry>
-          <mesh filename="package://pal_sea_arm_description/meshes/${mesh_folder}/${wrist_model}/arm_5_link.stl" scale="1 1 ${reflect}" />
+          <mesh filename="package://pal_sea_arm_description/meshes/${mesh_folder}/${wrist_model}/arm_5_link_collision.stl" scale="1 1 ${reflect}" />
         </geometry>
       </collision>
