Commit message: Fix version

File: triago_description/urdf/torso/torso_dual.urdf.xacro (robot description, xacro)
@@ -61,5 +61,5 @@
   </joint>
   <!-- Middle extending  -->
-  <!--link name="${name}_fixed_column_link">
+  <link name="${name}_fixed_column_link">
     <inertial>
       <origin rpy="0 0 0" xyz="0 0 0" />
@@ -92,5 +92,5 @@
     <child link="${name}_fixed_column_link" />
     <axis xyz="0 0 0" />
-  </joint-->
+  </joint>
   <link
     name="${name}_lift_link">

Commit message: Fixing torso controller

File: triago_description/urdf/torso/torso_dual.urdf.xacro (robot description, xacro)
@@ -138,5 +138,5 @@
     <child link="${name}_lift_link" />
     <axis xyz="0 0 1" />
-    <limit effort="0" lower="0" upper="0.35" velocity="0" />
+    <limit effort="0" lower="0" upper="0.35" velocity="${torso_max_vel}" />
   </joint>
   <link

Commit message: Fixing arm joint

File: triago_description/urdf/torso/torso_dual.urdf.xacro (robot description, xacro)
@@ -183,5 +183,5 @@
     name="${name}_arm_left_joint"
     type="fixed">
-    <origin xyz="0.0898413194899453 0.159181203216899 -0.0920547375491735" rpy="-2.06788770984932 0 -1.22173047639603" />
+    <origin xyz="0.0898413194899453 0.159181203216899 0.46245" rpy="-2.06788770984932 0 -1.22173047639603" />
     <parent
       link="${name}_lift_link" />
@@ -234,5 +234,5 @@
     name="${name}_arm_right_joint"
     type="fixed">
-    <origin xyz="0.0898413194899453 -0.1591812032169 -0.0920547375491731" rpy="-2.06788770984932 0 -1.91986217719377" />
+    <origin xyz="0.0898413194899453 -0.1591812032169 0.46245" rpy="-2.06788770984932 0 -1.91986217719377" />
     <parent
       link="${name}_lift_link" />

Commit message: Fix inertias

File: triago_description/urdf/torso/torso_dual.urdf.xacro (robot description, xacro)
@@ -19,12 +19,9 @@
   <!-- Bottom fixed part of column -->
   <link name="${name}_fixed_link">
-    <inertial>
-      <origin  xyz="0.0014857 -0.0077054 0.14693" rpy="0 0 0" />
-      <mass
-        value="14.56648" />
-      <inertia
-        ixx="499.42373004E-03" ixy="1.75882948E-03" ixz="11.19298375E-03"
-        iyy="526.82969543E-03" iyz="6.04744042E-03" izz="132.79782947E-03" />
-    </inertial>
+     <inertial>
+        <origin xyz="-0.043624513712351 -5.47054746000779E-05 0.0277532809798974" rpy="0 0 0" />
+        <mass value="1.00223030186675" />
+        <inertia ixx="0.00660602943010985" ixy="3.32767644990319E-05" ixz="-0.000408545705396379" iyy="0.00690807320580873" iyz="8.29177467923023E-06" izz="0.0122016808119362" />
+      </inertial>
     <visual>
       <origin
@@ -96,16 +93,7 @@
     name="${name}_lift_link">
     <inertial>
-      <origin
-        xyz="-29.57E-03 2.01E-03 371.47E-03"
-        rpy="0 0 0" />
-      <mass
-        value="12.11844" />
-      <inertia
-        ixx="377.29243241E-03"
-        ixy="2.00311792E-03"
-        ixz="-103.51344863E-03"
-        iyy="449.91209878E-03"
-        iyz="0.27176838E-03"
-        izz="224.52741499E-03" />
+      <origin xyz="-29.57E-03 2.01E-03 371.47E-03" rpy="0 0 0" />
+        <mass value="3.24266045177967" />
+        <inertia ixx="0.0295369723560087" ixy="-7.85101789883696E-07" ixz="-8.58576921315497E-05" iyy="0.0170989395656347" iyz="-8.17944373020342E-06" izz="0.0290055792681799" />
     </inertial>
     <visual>

Commit message: Fix inertias

File: triago_description/urdf/torso/torso_dual.urdf.xacro (robot description, xacro)
@@ -93,5 +93,5 @@
     name="${name}_lift_link">
     <inertial>
-      <origin xyz="-29.57E-03 2.01E-03 371.47E-03" rpy="0 0 0" />
+      <origin xyz="0 0 0" rpy="0 0 0" />
         <mass value="3.24266045177967" />
         <inertia ixx="0.0295369723560087" ixy="-7.85101789883696E-07" ixz="-8.58576921315497E-05" iyy="0.0170989395656347" iyz="-8.17944373020342E-06" izz="0.0290055792681799" />

Commit message: Lift torso_lift link of 5mm because a part was added to prevent collsion due the the 3rd arm + modify range of torso_lift

File: triago_description/urdf/torso/torso_dual.urdf.xacro (robot description, xacro)
@@ -128,9 +128,9 @@
   </link>
   <joint name="${name}_lift_joint" type="prismatic">
-    <origin rpy="0.0 0.0 0.0" xyz="0.0 0.0 0.0" />
+    <origin rpy="0.0 0.0 0.0" xyz="0.0 0.0 0.005" />
     <parent link="${name}_fixed_link" />
     <child link="${name}_lift_link" />
     <axis xyz="0 0 1" />
-    <limit effort="0" lower="0" upper="0.35" velocity="${torso_max_vel}" />
+    <limit effort="0" lower="0" upper="0.34" velocity="${torso_max_vel}" />
   </joint>
   <link

Commit message: Fix vel in urdf

File: triago_description/urdf/torso/torso_dual.urdf.xacro (robot description, xacro)
@@ -14,5 +14,5 @@
 <robot xmlns:xacro="http://ros.org/wiki/xacro">
   <!--Constant parameters-->
-  <xacro:property name="torso_max_vel"  value="0.07" />
+  <xacro:property name="torso_max_vel"  value="0.035" />
   <xacro:property name="torso_eps"      value="0.02" />
   <xacro:macro name="triago_torso" params="name parent">

Commit message: Revert inertias

File: triago_description/urdf/torso/torso_dual.urdf.xacro (robot description, xacro)
@@ -19,5 +19,5 @@
   <!-- Bottom fixed part of column -->
   <link name="${name}_fixed_link">
-     <inertial>
+      <inertial>
         <origin xyz="-0.043624513712351 -5.47054746000779E-05 0.0277532809798974" rpy="0 0 0" />
         <mass value="1.00223030186675" />
@@ -93,7 +93,13 @@
     name="${name}_lift_link">
     <inertial>
-      <origin xyz="0 0 0" rpy="0 0 0" />
-        <mass value="3.24266045177967" />
-        <inertia ixx="0.0295369723560087" ixy="-7.85101789883696E-07" ixz="-8.58576921315497E-05" iyy="0.0170989395656347" iyz="-8.17944373020342E-06" izz="0.0290055792681799" />
+      <origin xyz="-0.12355 -0.00014821 0.47959" rpy="0 0 0" />
+        <mass value="3.2902" />
+    <inertia
+        ixx="0.029638"
+        ixy="-8.5368E-07"
+        ixz="-5.793E-05"
+        iyy="0.017504"
+        iyz="-7.5566E-06"
+        izz="0.029034" />
     </inertial>
     <visual>

Commit message: Modifying the camera model

File: triago_description/urdf/torso/torso_dual.urdf.xacro (robot description, xacro)
@@ -92,14 +92,8 @@
   <link
     name="${name}_lift_link">
-    <inertial>
-      <origin xyz="-0.12355 -0.00014821 0.47959" rpy="0 0 0" />
-        <mass value="3.2902" />
-    <inertia
-        ixx="0.029638"
-        ixy="-8.5368E-07"
-        ixz="-5.793E-05"
-        iyy="0.017504"
-        iyz="-7.5566E-06"
-        izz="0.029034" />
+     <inertial>
+      <origin xyz="0 0 0" rpy="0 0 0" />
+        <mass value="3.24266045177967" />
+        <inertia ixx="0.0295369723560087" ixy="-7.85101789883696E-07" ixz="-8.58576921315497E-05" iyy="0.0170989395656347" iyz="-8.17944373020342E-06" izz="0.0290055792681799" />
     </inertial>
     <visual>

Commit message: update max velocity for the torso lift

File: triago_description/urdf/torso/torso_dual.urdf.xacro (robot description, xacro)
@@ -14,5 +14,5 @@
 <robot xmlns:xacro="http://ros.org/wiki/xacro">
   <!--Constant parameters-->
-  <xacro:property name="torso_max_vel"  value="0.035" />
+  <xacro:property name="torso_max_vel"  value="0.093" />
   <xacro:property name="torso_eps"      value="0.02" />
   <xacro:macro name="triago_torso" params="name parent">
