Commit message: Removing unused code

File: triago_description/urdf/end_effector/end_effector.urdf.xacro (robot description, xacro)
@@ -39,28 +39,4 @@
     </xacro:allegro_hand>
   </xacro:if>
-  <!-- Custom -->
-  <!-- <xacro:if value="${type == 'custom' and not is_dual}">
-    <xacro:include filename="$(find custom_ee_description)/urdf/end-effector.urdf.xacro" />
-    <xacro:end_effector parent="${parent}">
-      <origin xyz="0.0 0 0" rpy="0 0 0"/>
-    </xacro:end_effector>
-  </xacro:if> -->
-  <!-- Custom dual-->
-  <!-- <xacro:if value="${type == 'custom' and is_dual}"> -->
-   <!-- If right -->
-    <!-- <xacro:if value="${reflect == 1}">
-    <xacro:include filename="$(find custom_dual_ee_description)/urdf/end-effector-right.urdf.xacro" />
-    <xacro:end_effector_right parent="${parent}">
-      <origin xyz="0.0 0 0" rpy="0 0 0"/>
-    </xacro:end_effector_right>
-    </xacro:if> -->
-     <!-- If left -->
-    <!-- <xacro:if value="${reflect == -1}">
-    <xacro:include filename="$(find custom_dual_ee_description)/urdf/end-effector-left.urdf.xacro" />
-    <xacro:end_effector_left parent="${parent}">
-      <origin xyz="0.0 0 0" rpy="0 0 0"/>
-    </xacro:end_effector_left>
-    </xacro:if>
-  </xacro:if> -->
   </xacro:macro>
 </robot>

Commit message: Fixing pose gripper

File: triago_description/urdf/end_effector/end_effector.urdf.xacro (robot description, xacro)
@@ -28,5 +28,5 @@
     <xacro:include filename="$(find pal_pro_gripper_description)/urdf/gripper.urdf.xacro" />
           <xacro:pal_pro_gripper name="${name}" parent="${parent}" tool_changer="true">
-      <origin xyz="-0.0 0.0 0.066" rpy="0 0 0"/>
+      <origin xyz="-0.0 0.0 0.0" rpy="0 0 0"/>
     </xacro:pal_pro_gripper>
   </xacro:if>

Commit message: Add missing coupler link for the allegro hand

File: triago_description/urdf/end_effector/end_effector.urdf.xacro (robot description, xacro)
@@ -34,5 +34,73 @@
   <xacro:if value="${type == 'allegro-hand'}">
     <xacro:include filename="$(find allegro_hand_description)/urdf/allegro_hand.urdf.xacro" />
-    <xacro:allegro_hand name="${name}" parent="${parent}" reflect="${reflect}">
+    <link name="${name}_coupler_link">
+        <inertial>
+            <origin xyz="-7.7517E-05 -0.00017089 0.003965" rpy="0 0 0"/>
+            <mass value="0.033254"/>
+            <inertia
+                ixx="1.2371E-05" ixy="1.4319E-07" ixz="2.7745E-07"
+                iyy="1.5119E-05" iyz="-2.1946E-08"
+                izz="2.722E-05"/>
+        </inertial>
+        <visual>
+            <geometry>
+                <mesh filename="package://allegro_hand_description/meshes/allegro_coupler_link.STL" scale="${reflect} 1 1" />
+            </geometry>
+            <origin rpy="0 0 0" xyz="0 0 0 "/>
+            <material name="pal/DarkGrey"/>
+        </visual>
+        <collision>
+            <origin xyz="0 0 0.004" rpy="0 0 0"/>
+            <geometry>
+              <cylinder radius="0.0375" length="0.008"/>
+            </geometry>
+        </collision>
+    </link>
+    <gazebo reference="${name}_coupler_link">
+        <material>Gazebo/DarkGrey</material>
+        <mu1>0.9</mu1>
+        <mu2>0.9</mu2>
+    </gazebo>
+    <joint name="${name}_coupler_joint" type="fixed">
+        <parent link="${parent}" />
+        <child link="${name}_coupler_link" />
+        <origin xyz="0.0 0.0 0.0" rpy="0 0 0"/>
+        <axis xyz="0 0 0" />
+    </joint>
+    <link name="${name}_allegro_tc_out_link">
+        <inertial>
+            <origin xyz="-0.00052526 0.0003415 -0.0041487" rpy="0 0 0"/>
+            <mass value="0.03447"/>
+            <inertia
+                ixx="1.6829E-05" ixy="2.9746E-07" ixz="-4.1936E-08"
+                iyy="1.4935E-05" iyz="2.7742E-08"
+                izz="3.0915E-05"/>
+        </inertial>
+        <visual>
+            <geometry>
+                <mesh filename="package://allegro_hand_description/meshes/allegro_tc_out_link.STL" scale="${reflect} 1 1" />
+            </geometry>
+            <origin rpy="0 0 0" xyz="0 0 0 "/>
+            <material name="pal/DarkGrey"/>
+        </visual>
+        <collision>
+            <origin xyz="0 0 -0.006" rpy="0 0 0"/>
+            <geometry>
+              <cylinder radius="0.0375" length="0.012"/>
+            </geometry>
+        </collision>
+    </link>
+    <gazebo reference="${name}_allegro_tc_out_link">
+        <material>Gazebo/DarkGrey</material>
+        <mu1>0.9</mu1>
+        <mu2>0.9</mu2>
+    </gazebo>
+    <joint name="${name}_tc_joint" type="fixed">
+        <parent link="${name}_coupler_link" />
+        <child link="${name}_allegro_tc_out_link" />
+        <origin xyz="0 0 0.018" rpy="0 0 0" />
+        <axis xyz="0 0 0" />
+    </joint>
+    <xacro:allegro_hand name="${name}" parent="${name}_allegro_tc_out_link" reflect="${reflect}">
       <origin xyz="-0.00956 -0.001 0.094" rpy="0.0 0.0 ${-180.0 * deg_to_rad}"/>
     </xacro:allegro_hand>

Commit message: Revert hand to not be bothered by the wrist while grasping objects

File: triago_description/urdf/end_effector/end_effector.urdf.xacro (robot description, xacro)
@@ -103,5 +103,5 @@
     </joint>
     <xacro:allegro_hand name="${name}" parent="${name}_allegro_tc_out_link" reflect="${reflect}">
-      <origin xyz="-0.00956 -0.001 0.094" rpy="0.0 0.0 ${-180.0 * deg_to_rad}"/>
+      <origin xyz="0.00956 0.001 0.094" rpy="0.0 0.0 0"/>
     </xacro:allegro_hand>
   </xacro:if>

Commit message: Modify coupler path

File: triago_description/urdf/end_effector/end_effector.urdf.xacro (robot description, xacro)
@@ -45,5 +45,5 @@
         <visual>
             <geometry>
-                <mesh filename="package://allegro_hand_description/meshes/allegro_coupler_link.STL" scale="${reflect} 1 1" />
+                <mesh filename="package://pal_sea_arm_description/meshes/arm_tiago_pro/allegro_coupler_link.STL" scale="${reflect} 1 1" />
             </geometry>
             <origin rpy="0 0 0" xyz="0 0 0 "/>
@@ -79,5 +79,5 @@
         <visual>
             <geometry>
-                <mesh filename="package://allegro_hand_description/meshes/allegro_tc_out_link.STL" scale="${reflect} 1 1" />
+                <mesh filename="package://pal_sea_arm_description/meshes/arm_tiago_pro/allegro_tc_out_link.STL" scale="${reflect} 1 1" />
             </geometry>
             <origin rpy="0 0 0" xyz="0 0 0 "/>

Commit message: removing camera from end effector xacro

File: triago_description/urdf/end_effector/end_effector.urdf.xacro (robot description, xacro)
@@ -20,4 +20,5 @@
     - reflect: Set to 1 for a right end effector, or to -1 for a left end effector
   -->
+  <xacro:include filename="$(find realsense2_description)/urdf/_d405.urdf.xacro" />
   <xacro:macro name="triago_end_effector" params="name parent type has_end_effector reflect is_dual:=false camera_position">
   <!-- No end-effector -->
@@ -145,4 +146,12 @@
       <axis xyz="0 0 0" />
     </joint>
+    <xacro:sensor_d405
+      name="${name}_camera_rgbd"
+      parent="${name}_camera_link"
+      topics_ns="triago_end_effector">
+      <origin
+      xyz="0.0 0.0 0.0"
+      rpy="0.0 0.0 0.0"/>
+    </xacro:sensor_d405>
   </xacro:if>
   </xacro:macro>

Commit message: Fix end effector xacro

File: triago_description/urdf/end_effector/end_effector.urdf.xacro (robot description, xacro)
@@ -107,52 +107,4 @@
     </xacro:allegro_hand>
   </xacro:if>
-  <!--Camera-->
-  <xacro:if value="${type == 'camera-tools'}">
-    <link name="${name}_camera_link">
-      <inertial>
-        <origin xyz="-7.7517E-05 -0.00017089 0.003965" rpy="0 0 0"/>
-        <mass
-          value="0.073091" />
-        <inertia
-          ixx="2.656E-05" ixy="-2.4789E-08" ixz="-2.1125E-07"
-          iyy="1.3652E-05" iyz="-2.6011E-09"
-          izz="1.8641E-05" />
-      </inertial>
-      <visual>
-      <origin xyz="0 0 0" rpy="0 0 0" />
-        <geometry>
-          <mesh filename="package://pal_sea_arm_description/meshes/arm_tiago_pro/camera_link.STL" />
-        </geometry>
-        <material name="">
-          <color rgba="0.75294 0.75294 0.75294 1" />
-        </material>
-      </visual>
-      <collision>
-        <origin xyz="0 0 0" rpy="0 0 0" />
-        <geometry>
-          <mesh filename="package://pal_sea_arm_description/meshes/arm_tiago_pro/camera_link.STL" />
-        </geometry>
-      </collision>
-    </link>
-    <joint name="${name}_camera_joint" type="fixed">
-      <xacro:if value="${camera_position == 'up'}">
-        <origin xyz="0.0406 0 -0.003" rpy="3.1416 -1.5708 0" />
-      </xacro:if>
-      <xacro:if value="${camera_position == 'down'}">
-        <origin xyz="-0.0406 0 -0.003" rpy="0 -1.5708 0" />
-      </xacro:if>
-      <parent link="${parent}" />
-      <child link="${name}_camera_link" />
-      <axis xyz="0 0 0" />
-    </joint>
-    <xacro:sensor_d405
-      name="${name}_camera_rgbd"
-      parent="${name}_camera_link"
-      topics_ns="triago_end_effector">
-      <origin
-      xyz="0.0 0.0 0.0"
-      rpy="0.0 0.0 0.0"/>
-    </xacro:sensor_d405>
-  </xacro:if>
   </xacro:macro>
 </robot>
