Commit message: Split ros2_control hardware into two RobotControl components

File: triago_description/ros2_control/ros2_control.urdf.xacro (robot description, xacro)
@@ -13,4 +13,75 @@
  -->
 <robot xmlns:xacro="http://ros.org/wiki/xacro" name="triago">
+  <xacro:macro name="ros2_control_wheels">
+    <xacro:ros2_control_wheel side="front_right" />
+    <xacro:ros2_control_wheel side="front_left" />
+    <xacro:ros2_control_wheel side="rear_right" />
+    <xacro:ros2_control_wheel side="rear_left" />
+  </xacro:macro>
+  <xacro:macro name="ros2_control_arms">
+    <!-- arm left -->
+    <xacro:if value="${has_arm_left}">
+      <xacro:ros2_control_arm name="arm_left_1" reduction="1.0" offset_value="${arm_left_1_joint_offset}" />
+      <xacro:ros2_control_arm name="arm_left_2" reduction="1.0" offset_value="${arm_left_2_joint_offset}" />
+      <xacro:ros2_control_arm name="arm_left_3" reduction="1.0" offset_value="${arm_left_3_joint_offset}" />
+      <xacro:ros2_control_arm name="arm_left_4" reduction="1.0" offset_value="${arm_left_4_joint_offset}" />
+      <xacro:ros2_control_arm name="arm_left_5" reduction="1.0" offset_value="${arm_left_5_joint_offset}" />
+      <xacro:ros2_control_arm name="arm_left_6" reduction="1.0" offset_value="${arm_left_6_joint_offset}" />
+      <xacro:ros2_control_arm name="arm_left_7" reduction="1.0" offset_value="${arm_left_7_joint_offset}" />
+      <xacro:if value="${has_ft_sensor_left}">
+        <xacro:include filename="$(find pal_sea_arm_description)/urdf/sensors/ft_sensor/sensor.ros2_control.xacro"/>
+        <xacro:ros2_control_force_torque_sensor name="wrist_left_sensor"/>
+      </xacro:if>
+      <xacro:if value="${end_effector_left == 'pal-pro-gripper'}">
+        <xacro:ros2_control_pal_pro_gripper name="gripper_left" reduction="1.0" />
+      </xacro:if>
+      <xacro:if value="${end_effector_left == 'allegro-hand'}">
+        <!-- allegro-hand -->
+        <xacro:ros2_control_allegro_hand name="gripper_left" pid_controllers="$(arg pid_controllers)" reduction="1.0" />
+      </xacro:if>
+    </xacro:if>
+    <!-- arm right -->
+    <xacro:if value="${has_arm_right}">
+      <xacro:ros2_control_arm name="arm_right_1" reduction="1.0" offset_value="${arm_right_1_joint_offset}" />
+      <xacro:ros2_control_arm name="arm_right_2" reduction="1.0" offset_value="${arm_right_2_joint_offset}" />
+      <xacro:ros2_control_arm name="arm_right_3" reduction="1.0" offset_value="${arm_right_3_joint_offset}" />
+      <xacro:ros2_control_arm name="arm_right_4" reduction="1.0" offset_value="${arm_right_4_joint_offset}" />
+      <xacro:ros2_control_arm name="arm_right_5" reduction="1.0" offset_value="${arm_right_5_joint_offset}" />
+      <xacro:ros2_control_arm name="arm_right_6" reduction="1.0" offset_value="${arm_right_6_joint_offset}" />
+      <xacro:ros2_control_arm name="arm_right_7" reduction="1.0" offset_value="${arm_right_7_joint_offset}" />
+      <xacro:if value="${has_ft_sensor_right}">
+        <xacro:include filename="$(find pal_sea_arm_description)/urdf/sensors/ft_sensor/sensor.ros2_control.xacro"/>
+        <xacro:ros2_control_force_torque_sensor name="wrist_right_sensor"/>
+      </xacro:if>
+      <xacro:if value="${end_effector_right == 'pal-pro-gripper'}">
+        <!-- pal-pro-gripper -->
+        <xacro:ros2_control_pal_pro_gripper name="gripper_right" reduction="1.0" />
+      </xacro:if>
+      <xacro:if value="${end_effector_right == 'allegro-hand'}">
+        <!-- allegro-hand -->
+        <xacro:ros2_control_allegro_hand name="gripper_right" pid_controllers="$(arg pid_controllers)" reduction="1.0" />
+      </xacro:if>
+    </xacro:if>
+      <!-- arm head -->
+    <xacro:if value="${has_arm_head}">
+      <xacro:ros2_control_arm name="arm_head_1" reduction="1.0" offset_value="${arm_head_1_joint_offset}" />
+      <xacro:ros2_control_arm name="arm_head_2" reduction="1.0" offset_value="${arm_head_2_joint_offset}" />
+      <xacro:ros2_control_arm name="arm_head_3" reduction="1.0" offset_value="${arm_head_3_joint_offset}" />
+      <xacro:ros2_control_arm name="arm_head_4" reduction="1.0" offset_value="${arm_head_4_joint_offset}" />
+      <xacro:ros2_control_arm name="arm_head_5" reduction="1.0" offset_value="${arm_head_5_joint_offset}" />
+      <xacro:ros2_control_arm name="arm_head_6" reduction="1.0" offset_value="${arm_head_6_joint_offset}" />
+      <xacro:ros2_control_arm name="arm_head_7" reduction="1.0" offset_value="${arm_head_7_joint_offset}" />
+      <xacro:if value="${has_ft_sensor_head}">
+        <xacro:include filename="$(find pal_sea_arm_description)/urdf/sensors/ft_sensor/sensor.ros2_control.xacro"/>
+        <xacro:ros2_control_force_torque_sensor name="wrist_head_sensor"/>
+      </xacro:if>
+      <xacro:if value="${end_effector_head == 'pal-pro-gripper'}">
+        <xacro:ros2_control_pal_pro_gripper name="gripper_head" reduction="1.0" />
+      </xacro:if>
+      <xacro:if value="${end_effector_head == 'allegro-hand'}">
+        <xacro:ros2_control_allegro_hand name="gripper_head" pid_controllers="$(arg pid_controllers)" reduction="1.0" />
+      </xacro:if>
+    </xacro:if>
+  </xacro:macro>
   <xacro:macro name="triago_ros2_control" params="use_sim_time:=^|false">
     <xacro:arg name="arm_type_left" default="triago"/>
@@ -49,6 +120,7 @@
     <!-- calibration offsets -->
     <xacro:include filename="$(arg description_calibration_dir)/calibration_constants.urdf.xacro" />
-    <!-- Init the ROS 2 control gazebo interface -->
-    <xacro:if value="${use_sim_time}">
+    <!-- Simulation -->
+    <xacro:if value="$(arg use_sim_time)">
+      <!-- Init the ROS 2 control gazebo interface -->
       <gazebo>
         <plugin filename="libgazebo_ros2_control.so" name="gazebo_ros2_control">
@@ -56,90 +128,43 @@
         </plugin>
       </gazebo>
+      <ros2_control name="ros2_control_gazebo_system" type="system">
+        <hardware>
+          <plugin>gazebo_ros2_control/GazeboSystem</plugin>
+        </hardware>
+        <!-- wheels -->
+        <xacro:ros2_control_wheels/>
+        <!-- IMU -->
+        <xacro:ros2_control_imu name="base_imu_sensor"/>
+        <!-- torso -->
+        <xacro:ros2_control_torso name="torso_lift" reduction="1.0" />
+        <xacro:arg name="pid_controllers" default="false"/>
+        <!-- arms -->
+        <xacro:ros2_control_arms />
+      </ros2_control>
     </xacro:if>
-    <ros2_control name="ros2_control_triago_system" type="system">
-      <hardware>
-        <xacro:if value="$(arg use_sim_time)">
-          <plugin>gazebo_ros2_control/GazeboSystem</plugin>
-        </xacro:if>
-        <xacro:unless value="$(arg use_sim_time)">
+    <!-- Hardware -->
+    <xacro:unless value="$(arg use_sim_time)">
+      <ros2_control name="ros2_control_triago_system_can" type="system" rw_rate="100">
+        <hardware>
           <plugin>robot_control/RobotControl</plugin>
-        </xacro:unless>
-      </hardware>
-      <!-- wheels -->
-      <xacro:ros2_control_wheel side="front_right" />
-      <xacro:ros2_control_wheel side="front_left" />
-      <xacro:ros2_control_wheel side="rear_right" />
-      <xacro:ros2_control_wheel side="rear_left" />
-      <!-- IMU -->
-      <xacro:if value="$(arg use_sim_time)">
-        <xacro:ros2_control_imu name="base_imu_sensor"/>
-      </xacro:if>
-      <!-- torso -->
-      <xacro:ros2_control_torso name="torso_lift" reduction="1.0" />
-      <xacro:arg name="pid_controllers" default="false"/>
-      <!-- arm left -->
-      <xacro:if value="${has_arm_left}">
-        <xacro:ros2_control_arm name="arm_left_1" reduction="1.0" offset_value="${arm_left_1_joint_offset}" />
-        <xacro:ros2_control_arm name="arm_left_2" reduction="1.0" offset_value="${arm_left_2_joint_offset}" />
-        <xacro:ros2_control_arm name="arm_left_3" reduction="1.0" offset_value="${arm_left_3_joint_offset}" />
-        <xacro:ros2_control_arm name="arm_left_4" reduction="1.0" offset_value="${arm_left_4_joint_offset}" />
-        <xacro:ros2_control_arm name="arm_left_5" reduction="1.0" offset_value="${arm_left_5_joint_offset}" />
-        <xacro:ros2_control_arm name="arm_left_6" reduction="1.0" offset_value="${arm_left_6_joint_offset}" />
-        <xacro:ros2_control_arm name="arm_left_7" reduction="1.0" offset_value="${arm_left_7_joint_offset}" />
-        <xacro:if value="${has_ft_sensor_left}">
-          <xacro:include filename="$(find pal_sea_arm_description)/urdf/sensors/ft_sensor/sensor.ros2_control.xacro"/>
-          <xacro:ros2_control_force_torque_sensor name="wrist_left_sensor"/>
-        </xacro:if>
-        <xacro:if value="${end_effector_left == 'pal-pro-gripper'}">
-          <xacro:ros2_control_pal_pro_gripper name="gripper_left" reduction="1.0" />
-        </xacro:if>
-        <xacro:if value="${end_effector_left == 'allegro-hand'}">
-          <!-- allegro-hand -->
-          <xacro:ros2_control_allegro_hand name="gripper_left" pid_controllers="$(arg pid_controllers)" reduction="1.0" />
-        </xacro:if>
-      </xacro:if>
-      <!-- arm right -->
-      <xacro:if value="${has_arm_right}">
-        <xacro:ros2_control_arm name="arm_right_1" reduction="1.0" offset_value="${arm_right_1_joint_offset}" />
-        <xacro:ros2_control_arm name="arm_right_2" reduction="1.0" offset_value="${arm_right_2_joint_offset}" />
-        <xacro:ros2_control_arm name="arm_right_3" reduction="1.0" offset_value="${arm_right_3_joint_offset}" />
-        <xacro:ros2_control_arm name="arm_right_4" reduction="1.0" offset_value="${arm_right_4_joint_offset}" />
-        <xacro:ros2_control_arm name="arm_right_5" reduction="1.0" offset_value="${arm_right_5_joint_offset}" />
-        <xacro:ros2_control_arm name="arm_right_6" reduction="1.0" offset_value="${arm_right_6_joint_offset}" />
-        <xacro:ros2_control_arm name="arm_right_7" reduction="1.0" offset_value="${arm_right_7_joint_offset}" />
-        <xacro:if value="${has_ft_sensor_right}">
-          <xacro:include filename="$(find pal_sea_arm_description)/urdf/sensors/ft_sensor/sensor.ros2_control.xacro"/>
-          <xacro:ros2_control_force_torque_sensor name="wrist_right_sensor"/>
-        </xacro:if>
-        <xacro:if value="${end_effector_right == 'pal-pro-gripper'}">
-          <!-- pal-pro-gripper -->
-          <xacro:ros2_control_pal_pro_gripper name="gripper_right" reduction="1.0" />
-        </xacro:if>
-        <xacro:if value="${end_effector_right == 'allegro-hand'}">
-          <!-- allegro-hand -->
-          <xacro:ros2_control_allegro_hand name="gripper_right" pid_controllers="$(arg pid_controllers)" reduction="1.0" />
-        </xacro:if>
-      </xacro:if>
-       <!-- arm head -->
-      <xacro:if value="${has_arm_head}">
-        <xacro:ros2_control_arm name="arm_head_1" reduction="1.0" offset_value="${arm_head_1_joint_offset}" />
-        <xacro:ros2_control_arm name="arm_head_2" reduction="1.0" offset_value="${arm_head_2_joint_offset}" />
-        <xacro:ros2_control_arm name="arm_head_3" reduction="1.0" offset_value="${arm_head_3_joint_offset}" />
-        <xacro:ros2_control_arm name="arm_head_4" reduction="1.0" offset_value="${arm_head_4_joint_offset}" />
-        <xacro:ros2_control_arm name="arm_head_5" reduction="1.0" offset_value="${arm_head_5_joint_offset}" />
-        <xacro:ros2_control_arm name="arm_head_6" reduction="1.0" offset_value="${arm_head_6_joint_offset}" />
-        <xacro:ros2_control_arm name="arm_head_7" reduction="1.0" offset_value="${arm_head_7_joint_offset}" />
-        <xacro:if value="${has_ft_sensor_head}">
-          <xacro:include filename="$(find pal_sea_arm_description)/urdf/sensors/ft_sensor/sensor.ros2_control.xacro"/>
-          <xacro:ros2_control_force_torque_sensor name="wrist_head_sensor"/>
-        </xacro:if>
-        <xacro:if value="${end_effector_head == 'pal-pro-gripper'}">
-          <xacro:ros2_control_pal_pro_gripper name="gripper_head" reduction="1.0" />
-        </xacro:if>
-        <xacro:if value="${end_effector_head == 'allegro-hand'}">
-          <xacro:ros2_control_allegro_hand name="gripper_head" pid_controllers="$(arg pid_controllers)" reduction="1.0" />
-        </xacro:if>
-      </xacro:if>
-    </ros2_control>
+          <param name="group">can</param>
+        </hardware>
+        <!-- wheels -->
+        <xacro:ros2_control_wheels/>
+        <!-- IMU -->
+        <!-- <xacro:ros2_control_imu name="base_imu_sensor"/> -->
+      </ros2_control>
+      <ros2_control name="ros2_control_triago_system_ethercat" type="system" rw_rate="1000">
+        <hardware>
+          <plugin>robot_control/RobotControl</plugin>
+          <param name="group">ethercat</param>
+        </hardware>
+        <!-- torso -->
+        <xacro:ros2_control_torso name="torso_lift" reduction="1.0" />
+        <xacro:arg name="pid_controllers" default="true"/>
+        <!-- arms -->
+        <xacro:ros2_control_arms />
+      </ros2_control>
+    </xacro:unless>
   </xacro:macro>
 </robot>

Commit message: Add allegro hand as different system

File: triago_description/ros2_control/ros2_control.urdf.xacro (robot description, xacro)
@@ -36,8 +36,8 @@
         <xacro:ros2_control_pal_pro_gripper name="gripper_left" reduction="1.0" />
       </xacro:if>
-      <xacro:if value="${end_effector_left == 'allegro-hand'}">
-        <!-- allegro-hand -->
+      <!-- <xacro:if value="${end_effector_left == 'allegro-hand'}">
+        allegro-hand
         <xacro:ros2_control_allegro_hand name="gripper_left" pid_controllers="$(arg pid_controllers)" reduction="1.0" />
-      </xacro:if>
+      </xacro:if> -->
     </xacro:if>
     <!-- arm right -->
@@ -58,8 +58,8 @@
         <xacro:ros2_control_pal_pro_gripper name="gripper_right" reduction="1.0" />
       </xacro:if>
-      <xacro:if value="${end_effector_right == 'allegro-hand'}">
-        <!-- allegro-hand -->
+      <!-- <xacro:if value="${end_effector_right == 'allegro-hand'}">
+        allegro-hand
         <xacro:ros2_control_allegro_hand name="gripper_right" pid_controllers="$(arg pid_controllers)" reduction="1.0" />
-      </xacro:if>
+      </xacro:if> -->
     </xacro:if>
       <!-- arm head -->
@@ -79,7 +79,7 @@
         <xacro:ros2_control_pal_pro_gripper name="gripper_head" reduction="1.0" />
       </xacro:if>
-      <xacro:if value="${end_effector_head == 'allegro-hand'}">
+      <!-- <xacro:if value="${end_effector_head == 'allegro-hand'}">
         <xacro:ros2_control_allegro_hand name="gripper_head" pid_controllers="$(arg pid_controllers)" reduction="1.0" />
-      </xacro:if>
+      </xacro:if> -->
     </xacro:if>
   </xacro:macro>
@@ -108,4 +108,6 @@
     <xacro:property name="has_arm_right" value="${arm_type_right != 'no-arm'}" />
     <xacro:property name="has_arm_head" value="${arm_type_head != 'no-arm'}" />
+    <xacro:property name="can_device_name" value="can_device" />
+    <xacro:property name="can_device" value="can2" />
     <xacro:include filename="$(find omni_base_description)/urdf/sensors/sensors.ros2_control.xacro" />
     <xacro:include filename="$(find omni_base_description)/urdf/wheels/wheel.ros2_control.xacro" />
@@ -166,4 +168,35 @@
         <xacro:ros2_control_arms />
       </ros2_control>
+        <xacro:if value="${end_effector_right == 'allegro-hand'}">
+          <ros2_control name="ros2_control_allegro_hand_system_right" type="system" rw_rate="1000">
+            <hardware>
+              <plugin>allegro_hand_system/AllegroHandSystem</plugin>
+              <param name="${can_device_name}">can0</param>
+              <param name="side">right</param>
+            </hardware>
+            <xacro:ros2_control_allegro_hand name="gripper_right" pid_controllers="$(arg pid_controllers)" reduction="1.0" />
+          </ros2_control>
+        </xacro:if>
+        <xacro:if value="${end_effector_left == 'allegro-hand'}">
+          <ros2_control name="ros2_control_allegro_hand_system_left" type="system" rw_rate="1000">
+            <hardware>
+              <plugin>allegro_hand_system/AllegroHandSystem</plugin>
+              <param name="${can_device_name}">can2</param>
+              <param name="side">left</param>
+            </hardware>
+            <xacro:ros2_control_allegro_hand name="gripper_left" pid_controllers="$(arg pid_controllers)" reduction="1.0" />
+          </ros2_control>
+        </xacro:if>
+        <!-- <xacro:if value="${end_effector_head == 'allegro-hand'}">
+          <xacro:ros2_control_allegro_hand name="gripper_head" pid_controllers="$(arg pid_controllers)" reduction="1.0" />
+        </xacro:if> -->
+      <!-- <xacro:if value="$(arg use_xela_sensor)"> -->
+      <ros2_control name="ros2_control_xela_sensor" type="sensor" rw_rate="1000">
+        <hardware>
+          <plugin>xela_uskin_sensor/XelaUskinSensor</plugin>
+          <param name="${can_device_name}">can3</param>
+        </hardware>
+      </ros2_control>
+    <!-- </xacro:if> -->
     </xacro:unless>
   </xacro:macro>

Commit message: Add macro for allegro hand system and xela

File: triago_description/ros2_control/ros2_control.urdf.xacro (robot description, xacro)
@@ -72,4 +72,20 @@
       </xacro:if>
     </xacro:if>
+  </xacro:macro>
+  <xacro:macro name="allegro_ros2_control" params="side allegro_can xela_can">
+    <ros2_control name="$ros2_control_allegro_hand_system_{side}" type="system" rw_rate="1000">
+      <hardware>
+        <plugin>allegro_hand_system/AllegroHandSystem</plugin>
+        <param name="${can_device_name}">allegro_can</param>
+        <param name="side">side</param>
+      </hardware>
+      <xacro:ros2_control_allegro_hand name="gripper_left" pid_controllers="$(arg pid_controllers)" reduction="1.0" />
+    </ros2_control>
+    <ros2_control name="$ros2_control_xela_sensor_{side}" type="sensor" rw_rate="1000">
+      <hardware>
+        <plugin>xela_uskin_sensor/XelaUskinSensor</plugin>
+        <param name="${can_device_name}">xela_can</param>
+      </hardware>
+    </ros2_control>
   </xacro:macro>
   <xacro:macro name="triago_ros2_control" params="use_sim_time:=^|false">
@@ -158,50 +174,11 @@
       </ros2_control>
       <xacro:if value="${end_effector_right == 'allegro-hand'}">
-        <ros2_control name="ros2_control_allegro_hand_system_right" type="system" rw_rate="1000">
-          <hardware>
-            <plugin>allegro_hand_system/AllegroHandSystem</plugin>
-            <param name="${can_device_name}">can0</param>
-            <param name="side">right</param>
-          </hardware>
-          <xacro:ros2_control_allegro_hand name="gripper_right" pid_controllers="$(arg pid_controllers)" reduction="1.0" />
-        </ros2_control>
-        <ros2_control name="ros2_control_xela_sensor_right" type="sensor" rw_rate="1000">
-          <hardware>
-            <plugin>xela_uskin_sensor/XelaUskinSensor</plugin>
-            <param name="${can_device_name}">can1</param>
-          </hardware>
-        </ros2_control>
+        <allegro_ros2_control side="right" allegro_can="can0" xela_can="can1"/>
       </xacro:if>
       <xacro:if value="${end_effector_left == 'allegro-hand'}">
-        <ros2_control name="ros2_control_allegro_hand_system_left" type="system" rw_rate="1000">
-          <hardware>
-            <plugin>allegro_hand_system/AllegroHandSystem</plugin>
-            <param name="${can_device_name}">can2</param>
-            <param name="side">left</param>
-          </hardware>
-          <xacro:ros2_control_allegro_hand name="gripper_left" pid_controllers="$(arg pid_controllers)" reduction="1.0" />
-        </ros2_control>
-        <ros2_control name="ros2_control_xela_sensor_left" type="sensor" rw_rate="1000">
-          <hardware>
-            <plugin>xela_uskin_sensor/XelaUskinSensor</plugin>
-            <param name="${can_device_name}">can3</param>
-          </hardware>
-        </ros2_control>
+        <allegro_ros2_control side="left" allegro_can="can2" xela_can="can3"/>
       </xacro:if>
       <xacro:if value="${end_effector_head == 'allegro-hand'}">
-        <ros2_control name="ros2_control_allegro_hand_system_head" type="system" rw_rate="1000">
-          <hardware>
-            <plugin>allegro_hand_system/AllegroHandSystem</plugin>
-            <param name="${can_device_name}">can4</param>
-            <param name="side">right</param>
-          </hardware>
-          <xacro:ros2_control_allegro_hand name="gripper_right" pid_controllers="$(arg pid_controllers)" reduction="1.0" />
-        </ros2_control>
-        <ros2_control name="ros2_control_xela_sensor_head" type="sensor" rw_rate="1000">
-          <hardware>
-            <plugin>xela_uskin_sensor/XelaUskinSensor</plugin>
-            <param name="${can_device_name}">can5</param>
-          </hardware>
-        </ros2_control>
+        <allegro_ros2_control side="head" allegro_can="can4" xela_can="can5"/>
       </xacro:if>
     </xacro:unless>

Commit message: Remove unnecessary variable for can

File: triago_description/ros2_control/ros2_control.urdf.xacro (robot description, xacro)
@@ -114,5 +114,4 @@
     <xacro:property name="has_arm_head" value="${arm_type_head != 'no-arm'}" />
     <xacro:property name="can_device_name" value="can_device" />
-    <xacro:property name="can_device" value="can2" />
     <xacro:include filename="$(find omni_base_description)/urdf/sensors/sensors.ros2_control.xacro" />
     <xacro:include filename="$(find omni_base_description)/urdf/wheels/wheel.ros2_control.xacro" />

Commit message: Add torso_imu_link

File: triago_description/ros2_control/ros2_control.urdf.xacro (robot description, xacro)
@@ -142,5 +142,5 @@
         <xacro:ros2_control_wheels/>
         <!-- IMU -->
-        <xacro:ros2_control_imu name="base_imu_sensor"/>
+        <xacro:ros2_control_imu name="torso_imu_sensor"/>
         <!-- torso -->
         <xacro:ros2_control_torso name="torso_lift" reduction="1.0" />
@@ -189,5 +189,5 @@
         <xacro:allegro_ros2_control side="head" allegro_can="can4" xela_can="can5"/>
       </xacro:if>
-      <ros2_control name="base_imu_sensor" type="sensor" rw_rate="1000">
+      <ros2_control name="torso_imu_sensor" type="sensor" rw_rate="1000">
         <hardware>
           <plugin>pal_orientus_sensor/OrientusSensor</plugin>
@@ -195,5 +195,5 @@
         </hardware>
         <!-- IMU -->
-        <xacro:ros2_control_imu name="base_imu_sensor"/>
+        <xacro:ros2_control_imu name="torso_imu_sensor"/>
       </ros2_control>
     </xacro:unless>

File: triago_description/urdf/torso/torso_dual.urdf.xacro (robot description, xacro)
@@ -119,4 +119,7 @@
     <limit effort="0" lower="0" upper="0.34" velocity="${torso_max_vel}" />
   </joint>
+  <xacro:imu_sensor name="${name}_imu" parent="${name}_lift_link" update_rate="1000">
+    <origin xyz="0.0985 0.0014 0.38079" rpy="1.570796327 0 -1.570796327" />
+  </xacro:imu_sensor>
   <link name="${name}_arm_left_link"/>
   <joint
