Commit message: no-end-effector if there is no arm

File: triago_description/ros2_control/ros2_control.urdf.xacro (robot description, xacro)
@@ -122,4 +122,13 @@
       <xacro:include filename="$(find pal_pro_gripper_description)/urdf/gripper.ros2_control.xacro" />
     </xacro:if>
+    <xacro:if value="${not has_arm_left}">
+      <xacro:property name="end_effector_left" value="no-end-effector"/>
+    </xacro:if>
+    <xacro:if value="${not has_arm_right}">
+      <xacro:property name="end_effector_right" value="no-end-effector"/>
+    </xacro:if>
+    <xacro:if value="${not has_arm_head}">
+      <xacro:property name="end_effector_head" value="no-end-effector"/>
+    </xacro:if>
     <xacro:if value="${end_effector_left == 'allegro-hand' or end_effector_right == 'allegro-hand' or end_effector_head== 'allegro-hand'}">
       <xacro:include filename="$(find allegro_hand_description)/urdf/allegro_hand.ros2_control.xacro" />
