Commit message: Torso + base

File: triago_description/robots/triago.urdf.xacro (robot description, xacro)
@@ -71,51 +71,5 @@
   <xacro:include filename="$(find pal_urdf_utils)/urdf/deg_to_rad.urdf.xacro" />
   <!-- Base -->
-  <xacro:include filename="$(find omni_base_description)/urdf/base/base_sensors.urdf.xacro" />
   <!-- Torso -->
   <xacro:include filename="$(find t_descririagoption)/urdf/torso/triago_torso.urdf.xacro" />
-  <!-- Materials for visualization -->
-  <xacro:include filename="$(find pal_urdf_utils)/urdf/materials.urdf.xacro" />
-  <!-- Generic simulator_gazebo plugins -->
-  <xacro:include filename="$(find tiago_pro_description)/gazebo/gazebo.urdf.xacro" />
-  <!-- ROS 2 Control -->
-  <xacro:include filename="$(find tiago_pro_description)/ros2_control/ros2_control.urdf.xacro" />
-  <!-- ROBOT DEFINITION -->
-  <!-- Base -->
-  <xacro:base_sensors name="base" front_laser_model="$(arg laser_model)" rear_laser_model="$(arg laser_model)"/>
-  <!-- Torso. TODO:change for custom torso -->
-  <xacro:tiago_pro_torso name="torso" parent="base_link"/>
-  <!-- Head -->
-  <xacro:tiago_pro_head name="head" parent="torso_lift_link"/>
-  <!-- Left arm -->
-  <xacro:if value="${has_arm_left}">
-    <!-- Arm -->
-    <xacro:pal_sea_arm name="arm_left" parent="torso_lift_link" arm_type="${arm_type_left}" reflect="1" arm_1_offset="${arm_left_1_joint_offset}" arm_2_offset="${arm_left_2_joint_offset}" arm_3_offset="${arm_left_3_joint_offset}" arm_4_offset="${arm_left_4_joint_offset}" arm_5_offset="${arm_left_5_joint_offset}" arm_6_offset="${arm_left_6_joint_offset}" arm_7_offset="${arm_left_7_joint_offset}">
-      <origin xyz="$(arg arm_x) $(arg arm_y) $(arg arm_z)" rpy="$(arg arm_roll) $(arg arm_pitch) $(arg arm_yaw)"/>
-    </xacro:pal_sea_arm>
-    <!-- End effector -->
-    <xacro:if value="${has_end_effector_left}">
-      <xacro:pal_sea_arm_end_effector name="gripper_left" parent="${end_effector_left_link}" type="${end_effector_left}" has_end_effector="${has_end_effector_left}" reflect="-1" is_dual="true"/>
-    </xacro:if>
-    <!-- FT sensors -->
-    <xacro:if value="${has_ft_sensor_left}">
-      <xacro:ft_sensor name="wrist_left" parent="arm_left_tool_link"/>
-    </xacro:if>
-  </xacro:if>
-  <!-- Right arm -->
-  <xacro:if value="${has_arm_right}">
-    <!-- Arm -->
-    <xacro:pal_sea_arm name="arm_right" parent="torso_lift_link" arm_type="${arm_type_right}" reflect="1" arm_1_offset="${arm_right_1_joint_offset}" arm_2_offset="${arm_right_2_joint_offset}" arm_3_offset="${arm_right_3_joint_offset}" arm_4_offset="${arm_right_4_joint_offset}" arm_5_offset="${arm_right_5_joint_offset}" arm_6_offset="${arm_right_6_joint_offset}" arm_7_offset="${arm_right_7_joint_offset}">
-      <origin xyz="$(arg arm_x) ${-1.0*$(arg arm_y)} $(arg arm_z)" rpy="$(arg arm_roll) ${-1.0*$(arg arm_pitch)} ${-3.14159 -$(arg arm_yaw)}"/>
-    </xacro:pal_sea_arm>
-    <!-- End effector -->
-    <xacro:if value="${has_end_effector_right}">
-      <xacro:pal_sea_arm_end_effector name="gripper_right" parent="${end_effector_right_link}" type="${end_effector_right}" has_end_effector="${has_end_effector_right}" reflect="1" is_dual="true"/>
-    </xacro:if>
-    <!-- FT sensors -->
-    <xacro:if value="${has_ft_sensor_right}">
-      <xacro:ft_sensor name="wrist_right" parent="arm_right_tool_link"/>
-    </xacro:if>
-  </xacro:if>
-  <!-- ROS 2 Control -->
-  <xacro:tiago_pro_ros2_control use_sim="$(arg use_sim)" />
 </robot>
