Commit message: Refining triago model

File: triago_description/robots/triago.urdf.xacro (robot description, xacro)
@@ -12,25 +12,45 @@
   limitations under the License.
 -->
-<robot xmlns:xacro="http://ros.org/wiki/xacro" name="tiago_pro">
-  <xacro:arg name="use_sim" default="false"/>
+<robot xmlns:xacro="http://ros.org/wiki/xacro" name="triago">
+  <!-- ARGUMENTS -->
+  <!-- no-laser, sick-571-->
+  <xacro:arg name="laser_model" default="sick-571"/>
+  <!-- triago, no-arm -->
+  <xacro:arg name="arm_type_left" default="triago" />
+  <!-- triago, no-arm -->
+  <xacro:arg name="arm_type_right" default="triago" />
+  <!-- pal-pro-gripper custom-->
+  <xacro:arg name="end_effector_left" default="pal-pro-gripper" />
+  <!-- pal-pro-gripper, custom-->
+  <xacro:arg name="end_effector_right" default="pal-pro-gripper" />
+  <!-- no-ft-sensor, rokubi -->
+  <xacro:arg name="ft_sensor_left" default="no-ft-sensor" />
+  <!-- no-ft-sensor, rokubi -->
+  <xacro:arg name="ft_sensor_right" default="no-ft-sensor" />
+  <xacro:arg name="use_sim_time" default="false"/>
   <xacro:arg name="is_public_sim" default="false"/>
-  <!--xacro:arg name="description_calibration_dir" default="$(find tiago_pro_description)/urdf"/>
-  <xacro:arg name="extrinsic_calibration_dir" default="$(find tiago_pro_description)/urdf"/>
-  <xacro:arg name="arm_x" default="0.08976" />
-  <xacro:arg name="arm_y" default="0.15918" />
-  <xacro:arg name="arm_z" default="-0.092008" />
-  <xacro:arg name="arm_roll" default="-2.0679" />
-  <xacro:arg name="arm_pitch" default="0.0" />
-  <xacro:arg name="arm_yaw" default="-1.2217" /-->
-  <!-- PROPERTIES >
-  <xacro:property name="use_sim" value="$(arg use_sim)" />
+  <xacro:arg name="is_multiple" default="false"/>
+  <xacro:arg name="description_calibration_dir" default="$(find triago_description)/urdf"/>
+  <xacro:arg name="extrinsic_calibration_dir" default="$(find triago_description)/urdf"/>
+  <xacro:arg name="arm_x" default="0.089428" />
+  <xacro:arg name="arm_y" default="0.15903" />
+  <xacro:arg name="arm_z" default="0.46268" />
+  <xacro:arg name="arm_roll" default="-2.0961" />
+  <xacro:arg name="arm_pitch" default="0.31441" />
+  <xacro:arg name="arm_yaw" default="-1.3991" />
+  <!-- PROPERTIES -->
+  <xacro:property name="use_sim_time" value="$(arg use_sim_time)" />
+  <xacro:property name="is_multiple" value="$(arg is_multiple)" />
   <xacro:property name="laser_model" value="$(arg laser_model)" />
   <xacro:property name="arm_type_left" value="$(arg arm_type_left)" />
   <xacro:property name="arm_type_right" value="$(arg arm_type_right)" />
+  <xacro:property name="arm_type_head" value="$(arg arm_type_head)" />
   <xacro:property name="end_effector_left" value="$(arg end_effector_left)" />
   <xacro:property name="end_effector_right" value="$(arg end_effector_right)" />
+  <xacro:property name="end_effector_head" value="$(arg end_effector_head)" />
   <xacro:property name="ft_sensor_left" value="$(arg ft_sensor_left)" />
-  <xacro:property name="ft_sensor_right" value="$(arg ft_sensor_right)" />
-  <xacro:property name="arm_type" value="tiago-pro" />
+  <xacro:property name="ft_sensor_right" value="$(arg ft_sensor_head)" />
+  <xacro:property name="ft_sensor_head" value="$(arg ft_sensor_head)" />
+  <xacro:property name="arm_type" value="triago" />
   <xacro:property name="description_calibration_dir" value="${arg description_calibration_dir}"/>
   <xacro:property name="is_public_sim" value="$(arg is_public_sim)" />
@@ -44,17 +64,28 @@
   <xacro:property name="has_end_effector_right" value="${end_effector_right not in ['no-end-effector']}" />
   <xacro:property name="end_effector_right_link" value="${'wrist_right_ft_tool_link' if has_ft_sensor_right else 'arm_right_tool_link'}" />
-  <xacro:property name="end_effector_right_name" value="gripper_right" /-->
+  <xacro:property name="end_effector_right_name" value="gripper_right" />
+  <xacro:property name="has_arm_head" value="${arm_type_head not in ['no-arm']}"/>
+  <xacro:property name="has_ft_sensor_head" value="${ft_sensor_head not in ['no-ft-sensor']}"/>
+  <xacro:property name="has_end_effector_head" value="${end_effector_head not in ['no-end-effector']}" />
+  <xacro:property name="end_effector_head_link" value="${'wrist_head_ft_tool_link' if has_ft_sensor_head else 'arm_head_tool_link'}" />
+  <xacro:property name="end_effector_head_name" value="gripper_head" />
   <!-- Properties check -->
-  <!--xacro:if value="${arm_type_left not in ['tiago-pro', 'no-arm']}">
+  <xacro:if value="${arm_type_left not in ['triago', 'no-arm']}">
     <xacro:wrong_arm_type_left />
   </xacro:if>
-  <xacro:if value="${arm_type_right not in ['tiago-pro', 'no-arm']}">
+  <xacro:if value="${arm_type_right not in ['triago', 'no-arm']}">
     <xacro:wrong_arm_type_right />
   </xacro:if>
-  <xacro:if value="${end_effector_left not in ['pal-pro-gripper', 'custom', 'no-end-effector']}">
+  <xacro:if value="${arm_type_head not in ['triago', 'no-arm']}">
+    <xacro:wrong_arm_type_head />
+  </xacro:if>
+  <xacro:if value="${end_effector_left not in ['pal-pro-gripper', 'custom', 'allegro-hand', 'no-end-effector']}">
     <xacro:wrong_end_effector_left />
   </xacro:if>
-  <xacro:if value="${end_effector_right not in ['pal-pro-gripper', 'custom', 'no-end-effector']}">
+  <xacro:if value="${end_effector_right not in ['pal-pro-gripper', 'custom', 'allegro-hand', 'no-end-effector']}">
     <xacro:wrong_end_effector_right />
+  </xacro:if>
+  <xacro:if value="${end_effector_head not in ['pal-pro-gripper', 'custom', 'allegro-hand', 'no-end-effector']}">
+    <xacro:wrong_end_effector_head />
   </xacro:if>
   <xacro:if value="${ft_sensor_left not in ['no-ft-sensor', 'rokubi']}">
@@ -64,12 +95,98 @@
     <xacro:wrong_ft_sensor_right />
   </xacro:if>
+  <xacro:if value="${ft_sensor_head not in ['no-ft-sensor', 'rokubi']}">
+    <xacro:wrong_ft_sensor_head />
+  </xacro:if>
   <xacro:if value="${laser_model not in ['no-laser', 'sick-571']}">
     <xacro:wrong_laser_model />
-  </xacro:if-->
+  </xacro:if>
   <!-- INCLUDES -->
   <!-- Tools -->
   <xacro:include filename="$(find pal_urdf_utils)/urdf/deg_to_rad.urdf.xacro" />
   <!-- Base -->
+  <xacro:include filename="$(find omni_base_description)/urdf/base/base_sensors.urdf.xacro" />
   <!-- Torso -->
-  <xacro:include filename="$(find t_descririagoption)/urdf/torso/triago_torso.urdf.xacro" />
+  <xacro:include filename="$(find triago_description)/urdf/torso/torso_dual.urdf.xacro" />
+  <!-- Calibration constants -->
+  <xacro:include filename="$(arg description_calibration_dir)/calibration_constants.urdf.xacro" />
+  <!-- Arm -->
+  <xacro:if value="${has_arm_right or has_arm_left}">
+    <xacro:include filename="$(find pal_sea_arm_description)/urdf/arm/arm.urdf.xacro" />
+  </xacro:if>
+  <!-- End effector -->
+  <xacro:if value="${(has_arm_right or has_arm_left) and (has_end_effector_right or has_end_effector_left)}">
+    <xacro:include filename="$(find pal_sea_arm_description)/urdf/end_effector/end_effector.urdf.xacro" />
+  </xacro:if>
+  <!-- Allegro hand and tool changer-->
+  <xacro:if value="${end_effector_right == 'allegro-hand'}">
+    <xacro:include filename="$(find triago_description)/urdf/tool_changer/tool_changer.urdf.xacro" />
+    <xacro:include filename="$(find allegro_hand_description)/urdf/allegro_hand.urdf.xacro" />
+  </xacro:if>
+  <!-- Force Torque sensor -->
+  <xacro:if value="${has_ft_sensor_right or has_ft_sensor_left}">
+    <xacro:include filename="$(find triago_description)/urdf/ft_sensor/ft_sensor.urdf.xacro" />
+    <xacro:include filename="$(find pal_sea_arm_description)/urdf/sensors/ft_sensor.gazebo.xacro" />
+  </xacro:if>
+  <!-- Materials for visualization -->
+  <xacro:include filename="$(find pal_urdf_utils)/urdf/materials.urdf.xacro" />
+  <!-- ROS 2 Control -->
+  <xacro:include filename="$(find triago_description)/ros2_control/ros2_control.urdf.xacro" />
+  <!-- ROBOT DEFINITION -->
+  <!-- Base -->
+  <xacro:base_sensors name="base" front_laser_model="$(arg laser_model)" rear_laser_model="$(arg laser_model)"/>
+  <!-- Torso. TODO:change for custom torso -->
+  <xacro:triago_torso name="torso" parent="base_link"/>
+  <!-- Left arm -->
+  <xacro:if value="${has_arm_left}">
+    <!-- Arm -->
+    <xacro:pal_sea_arm name="arm_left" parent="torso_lift_link" arm_type="$(arg arm_type_left)" reflect="1" arm_1_offset="${arm_left_1_joint_offset}" arm_2_offset="${arm_left_2_joint_offset}" arm_3_offset="${arm_left_3_joint_offset}" arm_4_offset="${arm_left_4_joint_offset}" arm_5_offset="${arm_left_5_joint_offset}" arm_6_offset="${arm_left_6_joint_offset}" arm_7_offset="${arm_left_7_joint_offset}">
+      <origin xyz="$(arg arm_x) $(arg arm_y) $(arg arm_z)" rpy="$(arg arm_roll) $(arg arm_pitch) $(arg arm_yaw)"/>
+    </xacro:pal_sea_arm>
+    <!-- End effector -->
+    <xacro:if value="${has_end_effector_left}">
+      <xacro:pal_sea_arm_end_effector name="gripper_left" parent="${end_effector_left_link}" type="${end_effector_left}" has_end_effector="${has_end_effector_left}" reflect="-1" is_dual="true"/>
+    </xacro:if>
+    <!-- FT sensors -->
+    <xacro:if value="${has_ft_sensor_left}">
+      <xacro:ft_sensor name="wrist_left" parent="arm_left_tool_link"/>
+    </xacro:if>
+  </xacro:if>
+  <!-- Right arm -->
+  <xacro:if value="${has_arm_right}">
+    <!-- Arm -->
+    <xacro:pal_sea_arm name="arm_right" parent="torso_lift_link" arm_type="$(arg arm_type_right)" reflect="1" arm_1_offset="${arm_right_1_joint_offset}" arm_2_offset="${arm_right_2_joint_offset}" arm_3_offset="${arm_right_3_joint_offset}" arm_4_offset="${arm_right_4_joint_offset}" arm_5_offset="${arm_right_5_joint_offset}" arm_6_offset="${arm_right_6_joint_offset}" arm_7_offset="${arm_right_7_joint_offset}">
+      <origin xyz="$(arg arm_x) ${-1.0*$(arg arm_y)} $(arg arm_z)" rpy="$(arg arm_roll) ${-1.0*$(arg arm_pitch)} ${-3.14159 -$(arg arm_yaw)}"/>
+    </xacro:pal_sea_arm>
+    <!-- End effector -->
+    <xacro:if value="${has_end_effector_right}">
+      <xacro:pal_sea_arm_end_effector name="gripper_right" parent="${end_effector_right_link}" type="${end_effector_right}" has_end_effector="${has_end_effector_right}" reflect="1" is_dual="true"/>
+    </xacro:if>
+    <xacro:if value="${end_effector_right == 'allegro-hand'}">
+      <xacro:tool_changer name="tool_changer_right" parent="arm_right_tool_link"/>
+      <xacro:allegro_hand name="gripper_right" parent="tool_changer_right_tc_tool_link" reflect="1">
+              <origin xyz="0 0 0.0" rpy="0 0 0"/>
+      </xacro:allegro_hand>
+    </xacro:if>
+    <!-- FT sensors -->
+    <xacro:if value="${has_ft_sensor_right}">
+      <xacro:ft_sensor name="wrist_right" parent="arm_right_tool_link"/>
+    </xacro:if>
+  </xacro:if>
+  <!-- Third arm -->
+  <xacro:if value="${has_arm_head}">
+    <!-- Arm -->
+    <xacro:pal_sea_arm name="arm_head" parent="torso_lift_link" arm_type="$(arg arm_type_head)" reflect="1" arm_1_offset="${arm_right_1_joint_offset}" arm_2_offset="${arm_right_2_joint_offset}" arm_3_offset="${arm_right_3_joint_offset}" arm_4_offset="${arm_right_4_joint_offset}" arm_5_offset="${arm_right_5_joint_offset}" arm_6_offset="${arm_right_6_joint_offset}" arm_7_offset="${arm_right_7_joint_offset}">
+      <origin xyz="0.00733452377915612 0.0 0.630632193308821" rpy="0 0.785398163397445 0"/>
+    </xacro:pal_sea_arm>
+    <!-- End effector -->
+    <xacro:if value="${has_end_effector_head}">
+      <xacro:pal_sea_arm_end_effector name="gripper_head" parent="${end_effector_head_link}" type="${end_effector_head}" has_end_effector="${has_end_effector_head}" reflect="1" is_dual="true"/>
+    </xacro:if>
+    <!-- FT sensors -->
+    <xacro:if value="${has_ft_sensor_head}">
+      <xacro:ft_sensor name="wrist_right" parent="arm_head_tool_link"/>
+    </xacro:if>
+  </xacro:if>
+  <!-- ROS 2 Control -->
+  <xacro:triago_ros2_control use_sim_time="$(arg use_sim_time)" />
 </robot>

File: triago_description/ros2_control/ros2_control.urdf.xacro (robot description, xacro)
@@ -12,16 +12,18 @@
   limitations under the License.
  -->
-<robot xmlns:xacro="http://ros.org/wiki/xacro" name="tiago_pro">
-  <xacro:macro name="tiago_pro_ros2_control" params="use_sim:=^|false">
-    <xacro:arg name="arm_type_left" default="tiago-pro"/>
-    <xacro:arg name="arm_type_right" default="tiago-pro"/>
+<robot xmlns:xacro="http://ros.org/wiki/xacro" name="triago">
+  <xacro:macro name="triago_ros2_control" params="use_sim_time:=^|false">
+    <xacro:arg name="arm_type_left" default="triago"/>
+    <xacro:arg name="arm_type_right" default="triago"/>
+    <xacro:arg name="arm_type_head" default="triago"/>
     <xacro:arg name="end_effector_left" default="pal-pro-pripper"/>
     <xacro:arg name="end_effector_right" default="pal-pro-gripper"/>
     <xacro:arg name="ft_sensor_left" default="no-ft-sensor"/>
     <xacro:arg name="ft_sensor_right" default="no-ft-sensor"/>
-    <xacro:arg name="description_calibration_dir" default="$(find tiago_pro_description)/urdf/calibration" />
+    <xacro:arg name="description_calibration_dir" default="$(find triago_description)/urdf/calibration" />
     <!-- TODO-->
     <xacro:property name="arm_type_left" value="$(arg arm_type_left)" />
     <xacro:property name="arm_type_right" value="$(arg arm_type_right)" />
+    <xacro:property name="arm_type_head" value="$(arg arm_type_head)" />
     <xacro:property name="end_effector_left" value="$(arg end_effector_left)" />
     <xacro:property name="end_effector_right" value="$(arg end_effector_right)" />
@@ -32,6 +34,5 @@
     <xacro:include filename="$(find omni_base_description)/urdf/sensors/sensors.ros2_control.xacro" />
     <xacro:include filename="$(find omni_base_description)/urdf/wheels/wheel.ros2_control.xacro" />
-    <xacro:include filename="$(find tiago_pro_description)/urdf/torso/torso.ros2_control.xacro" />
-    <xacro:include filename="$(find tiago_pro_description)/urdf/head/head.ros2_control.xacro" />
+    <xacro:include filename="$(find triago_description)/urdf/torso/torso.ros2_control.xacro" />
     <xacro:include filename="$(find pal_sea_arm_description)/urdf/arm/arm.ros2_control.xacro" />
     <xacro:if value="${end_effector_left == 'pal-pro-gripper' or end_effector_right == 'pal-pro-gripper'}">
@@ -40,10 +41,18 @@
     <!-- calibration offsets -->
     <xacro:include filename="$(arg description_calibration_dir)/calibration_constants.urdf.xacro" />
-    <ros2_control name="ros2_control_tiago_pro_system" type="system">
+    <!-- Init the ROS 2 control gazebo interface -->
+    <xacro:if value="${use_sim_time}">
+      <gazebo>
+        <plugin filename="libgazebo_ros2_control.so" name="gazebo_ros2_control">
+          <parameters>$(find triago_description)/ros2_control/gazebo_controller_manager_cfg.yaml</parameters>
+        </plugin>
+      </gazebo>
+    </xacro:if>
+    <ros2_control name="ros2_control_triago_system" type="system">
       <hardware>
-        <xacro:if value="$(arg use_sim)">
+        <xacro:if value="$(arg use_sim_time)">
           <plugin>gazebo_ros2_control/GazeboSystem</plugin>
         </xacro:if>
-        <xacro:unless value="$(arg use_sim)">
+        <xacro:unless value="$(arg use_sim_time)">
           <plugin>robot_control/RobotControl</plugin>
         </xacro:unless>
@@ -55,12 +64,9 @@
       <xacro:ros2_control_wheel side="rear_left" />
       <!-- IMU -->
-      <xacro:if value="$(arg use_sim)">
+      <xacro:if value="$(arg use_sim_time)">
         <xacro:ros2_control_imu name="base_imu_sensor"/>
       </xacro:if>
       <!-- torso -->
       <xacro:ros2_control_torso name="torso_lift" reduction="1.0" />
-      <!-- head -->
-      <xacro:ros2_control_head name="head_1" reduction="1.0" offset_value="${head_1_joint_offset}" />
-      <xacro:ros2_control_head name="head_2" reduction="1.0" offset_value="${head_2_joint_offset}" />
       <!-- arm left -->
       <xacro:if value="${has_arm_left}">

File: triago_description/urdf/head/head.urdf.xacro (robot description, xacro)
@@ -136,5 +136,5 @@
     </gazebo>
     <!-- Head camera:Intel D435 -->
-    <xacro:sensor_d435 parent="${name}_2_link" name="${name}_front_camera" topics_ns="${name}_front_camera" use_nominal_extrinsics="${use_sim}">
+    <xacro:sensor_d435 parent="${name}_2_link" name="${name}_front_camera" topics_ns="${name}_front_camera" use_nominal_extrinsics="${use_sim_time}">
        <origin xyz="0.03815 0.14750 0.0"
                 rpy="${-90.0 * deg_to_rad} 0.0 0.0"/>

File: triago_description/urdf/torso/torso.ros2_control.xacro (robot description, xacro)
@@ -20,5 +20,5 @@
       <state_interface name="effort" />
     </joint>
-    <xacro:include filename="$(find tiago_pro_description)/urdf/torso/torso.transmission.urdf.xacro" />
+    <xacro:include filename="$(find triago_description)/urdf/torso/torso.transmission.urdf.xacro" />
     <xacro:torso_simple_transmission name="${name}" reduction="${reduction}" />
   </xacro:macro>

File: triago_description/urdf/torso/torso_dual.urdf.xacro (robot description, xacro)
@@ -16,5 +16,5 @@
   <xacro:property name="torso_max_vel"  value="0.07" />
   <xacro:property name="torso_eps"      value="0.02" />
-  <xacro:macro name="tiago_pro_torso" params="name parent">
+  <xacro:macro name="triago_torso" params="name parent">
   <!-- Bottom fixed part of column -->
   <link name="${name}_fixed_link">
@@ -22,7 +22,8 @@
       <origin  xyz="0.0014857 -0.0077054 0.14693" rpy="0 0 0" />
       <mass
-        value="15.527" />
-      <inertia ixx="0.17904" ixy="0.00019412" ixz="-0.0049479"
-               iyy="0.20082" iyz="0.00015981" izz="0.084141" />
+        value="14.56648" />
+      <inertia
+        ixx="499.42373004E-03" ixy="1.75882948E-03" ixz="11.19298375E-03"
+        iyy="526.82969543E-03" iyz="6.04744042E-03" izz="132.79782947E-03" />
     </inertial>
     <visual>
@@ -32,28 +33,20 @@
       <geometry>
         <mesh
-          filename="package://tiago_pro_description/meshes/torso/torso_fixed_link.stl" />
+          filename="package://triago_description/meshes/torso/torso_fixed.STL" />
       </geometry>
-      <material name="pal/DarkGrey"/>
+      <material
+        name="">
+        <color
+          rgba="0.298039215686275 0.298039215686275 0.298039215686275 1" />
+      </material>
     </visual>
     <collision>
-      <origin rpy="0 0 0" xyz="0 0 0.1" />
+      <origin
+        xyz="0 0 0.0"
+        rpy="0 0 0" />
       <geometry>
-        <box size="0.23 0.253 0.2"/>
+        <mesh
+          filename="package://triago_description/meshes/torso/torso_fixed.STL" />
       </geometry>
-      <material name="pal/DarkGrey"/>
-    </collision>
-    <collision>
-      <origin rpy="0 0 0" xyz="0.18 0 0.03" />
-      <geometry>
-        <box size="0.15 0.253 0.06"/>
-      </geometry>
-      <material name="pal/DarkGrey"/>
-    </collision>
-    <collision>
-      <origin rpy="0 0 0" xyz="-0.09 0 0.0" />
-      <geometry>
-        <box size="0.47 0.5 0.02"/>
-      </geometry>
-      <material name="pal/DarkGrey"/>
     </collision>
   </link>
@@ -68,5 +61,5 @@
   </joint>
   <!-- Middle extending  -->
-  <link name="${name}_fixed_column_link">
+  <!--link name="${name}_fixed_column_link">
     <inertial>
       <origin rpy="0 0 0" xyz="0 0 0" />
@@ -99,20 +92,20 @@
     <child link="${name}_fixed_column_link" />
     <axis xyz="0 0 0" />
-  </joint>
+  </joint-->
   <link
     name="${name}_lift_link">
     <inertial>
       <origin
-        xyz="0.0014742 0.0065278 -0.20301"
+        xyz="-29.57E-03 2.01E-03 371.47E-03"
         rpy="0 0 0" />
       <mass
-        value="9.547" />
+        value="12.11844" />
       <inertia
-        ixx="0.042078"
-        ixy="5.6766E-05"
-        ixz="0.00014731"
-        iyy="0.031115"
-        iyz="-5.0165E-05"
-        izz="0.018659" />
+        ixx="377.29243241E-03"
+        ixy="2.00311792E-03"
+        ixz="-103.51344863E-03"
+        iyy="449.91209878E-03"
+        iyz="0.27176838E-03"
+        izz="224.52741499E-03" />
     </inertial>
     <visual>
@@ -122,7 +115,11 @@
       <geometry>
         <mesh
-          filename="package://tiago_pro_description/meshes/torso/torso_lift_link.stl" />
+          filename="package://triago_description/meshes/torso/torso_lift_link.STL" />
       </geometry>
-      <material name="White"/>
+      <material
+        name="">
+        <color
+          rgba="0.29804 0.29804 0.29804 1" />
+      </material>
     </visual>
     <collision>
@@ -132,24 +129,15 @@
       <geometry>
         <mesh
-          filename="package://tiago_pro_description/meshes/torso/torso_lift_link_collision.stl" />
+          filename="package://triago_description/meshes/torso/torso_lift_link.STL" />
       </geometry>
     </collision>
   </link>
   <joint name="${name}_lift_joint" type="prismatic">
-    <origin rpy="0.0 0.0 0.0" xyz="0.0 0.0 0.5545" />
+    <origin rpy="0.0 0.0 0.0" xyz="0.0 0.0 0.0" />
     <parent link="${name}_fixed_link" />
     <child link="${name}_lift_link" />
     <axis xyz="0 0 1" />
-    <limit effort="2000" lower="0" upper="0.35" velocity="${torso_max_vel}" />
-    <calibration rising="0.0" />
-    <dynamics damping="1000" />
-    <safety_controller k_position="20"
-                         k_velocity="20"
-                         soft_lower_limit="0.0"
-                         soft_upper_limit="0.35" />
+    <limit effort="0" lower="0" upper="0.35" velocity="0" />
   </joint>
-  <gazebo reference="${name}_lift_joint">
-     <implicitSpringDamper>1</implicitSpringDamper>
-  </gazebo>
   </xacro:macro>
 </robot>
