Commit message: addnig allegro hand option

File: triago_description/robots/triago.urdf.xacro (robot description, xacro)
@@ -145,5 +145,13 @@
     <!-- End effector -->
     <xacro:if value="${has_end_effector_left}">
-      <xacro:pal_sea_arm_end_effector name="gripper_left" parent="${end_effector_left_link}" type="${end_effector_left}" has_end_effector="${has_end_effector_left}" reflect="-1" is_dual="true"/>
+      <xacro:if value="${end_effector_left == 'allegro-hand'}">
+        <xacro:tool_changer name="tool_changer_left" parent="${end_effector_left_link}"/>
+        <xacro:allegro_hand name="gripper_left" parent="tool_changer_left_tc_tool_link" reflect="-1">
+                <origin xyz="0 0 0.0" rpy="0 0 0"/>
+        </xacro:allegro_hand>
+      </xacro:if>
+      <xacro:unless value="${end_effector_left == 'allegro-hand'}">
+        <xacro:pal_sea_arm_end_effector name="gripper_left" parent="${end_effector_left_link}" type="${end_effector_left}" has_end_effector="${has_end_effector_left}" reflect="-1" is_dual="true"/>
+      </xacro:unless>
     </xacro:if>
     <!-- FT sensors -->
@@ -160,11 +168,13 @@
     <!-- End effector -->
     <xacro:if value="${has_end_effector_right}">
-      <xacro:pal_sea_arm_end_effector name="gripper_right" parent="${end_effector_right_link}" type="${end_effector_right}" has_end_effector="${has_end_effector_right}" reflect="1" is_dual="true"/>
-    </xacro:if>
-    <xacro:if value="${end_effector_right == 'allegro-hand'}">
-      <xacro:tool_changer name="tool_changer_right" parent="arm_right_tool_link"/>
-      <xacro:allegro_hand name="gripper_right" parent="tool_changer_right_tc_tool_link" reflect="1">
-              <origin xyz="0 0 0.0" rpy="0 0 0"/>
-      </xacro:allegro_hand>
+      <xacro:if value="${end_effector_right == 'allegro-hand'}">
+        <xacro:tool_changer name="tool_changer_right" parent="${end_effector_right_link}"/>
+        <xacro:allegro_hand name="gripper_right" parent="tool_changer_right_tc_tool_link" reflect="1">
+                <origin xyz="0 0 0.0" rpy="0 0 0"/>
+        </xacro:allegro_hand>
+      </xacro:if>
+      <xacro:unless value="${end_effector_right == 'allegro-hand'}">
+        <xacro:pal_sea_arm_end_effector name="gripper_right" parent="${end_effector_right_link}" type="${end_effector_right}" has_end_effector="${has_end_effector_right}" reflect="1" is_dual="true"/>
+      </xacro:unless>
     </xacro:if>
     <!-- FT sensors -->
@@ -181,5 +191,13 @@
     <!-- End effector -->
     <xacro:if value="${has_end_effector_head}">
-      <xacro:pal_sea_arm_end_effector name="gripper_head" parent="${end_effector_head_link}" type="${end_effector_head}" has_end_effector="${has_end_effector_head}" reflect="1" is_dual="true"/>
+      <xacro:if  value="${end_effector_head == 'allegro-hand'}">
+        <xacro:tool_changer name="tool_changer_head" parent="${end_effector_head_link}"/>
+        <xacro:allegro-hand name="gripper_head" parent="tool_changer_head_tc_tool_link" reflect="1">
+                <origin xyz="0 0 0.0" rpy="0 0 0"/>
+        </xacro:allegro-hand>
+      </xacro:if>
+      <xacro:unless value="${end_effector_head == 'allegro-hand'}">
+        <xacro:pal_sea_arm_end_effector name="gripper_head" parent="${end_effector_head_link}" type="${end_effector_head}" has_end_effector="${has_end_effector_head}" reflect="1" is_dual="true"/>
+      </xacro:unless>
     </xacro:if>
     <!-- FT sensors -->

Commit message: Fixing orientation arms

File: triago_description/robots/triago.urdf.xacro (robot description, xacro)
@@ -140,6 +140,6 @@
   <xacro:if value="${has_arm_left}">
     <!-- Arm -->
-    <xacro:pal_sea_arm name="arm_left" parent="torso_lift_link" arm_type="$(arg arm_type_left)" reflect="1" arm_1_offset="${arm_left_1_joint_offset}" arm_2_offset="${arm_left_2_joint_offset}" arm_3_offset="${arm_left_3_joint_offset}" arm_4_offset="${arm_left_4_joint_offset}" arm_5_offset="${arm_left_5_joint_offset}" arm_6_offset="${arm_left_6_joint_offset}" arm_7_offset="${arm_left_7_joint_offset}">
-      <origin xyz="$(arg arm_x) $(arg arm_y) $(arg arm_z)" rpy="$(arg arm_roll) $(arg arm_pitch) $(arg arm_yaw)"/>
+    <xacro:pal_sea_arm name="arm_left" parent="arm_left_link" arm_type="$(arg arm_type_left)" reflect="1" arm_1_offset="${arm_left_1_joint_offset}" arm_2_offset="${arm_left_2_joint_offset}" arm_3_offset="${arm_left_3_joint_offset}" arm_4_offset="${arm_left_4_joint_offset}" arm_5_offset="${arm_left_5_joint_offset}" arm_6_offset="${arm_left_6_joint_offset}" arm_7_offset="${arm_left_7_joint_offset}">
+      <origin xyz="0.0 0.0 0.0" rpy="0.0 0.0 -1.5708"/>
     </xacro:pal_sea_arm>
     <!-- End effector -->
@@ -163,6 +163,6 @@
   <xacro:if value="${has_arm_right}">
     <!-- Arm -->
-    <xacro:pal_sea_arm name="arm_right" parent="torso_lift_link" arm_type="$(arg arm_type_right)" reflect="1" arm_1_offset="${arm_right_1_joint_offset}" arm_2_offset="${arm_right_2_joint_offset}" arm_3_offset="${arm_right_3_joint_offset}" arm_4_offset="${arm_right_4_joint_offset}" arm_5_offset="${arm_right_5_joint_offset}" arm_6_offset="${arm_right_6_joint_offset}" arm_7_offset="${arm_right_7_joint_offset}">
-      <origin xyz="$(arg arm_x) ${-1.0*$(arg arm_y)} $(arg arm_z)" rpy="$(arg arm_roll) ${-1.0*$(arg arm_pitch)} ${-3.14159 -$(arg arm_yaw)}"/>
+    <xacro:pal_sea_arm name="arm_right" parent="arm_right_link" arm_type="$(arg arm_type_right)" reflect="1" arm_1_offset="${arm_right_1_joint_offset}" arm_2_offset="${arm_right_2_joint_offset}" arm_3_offset="${arm_right_3_joint_offset}" arm_4_offset="${arm_right_4_joint_offset}" arm_5_offset="${arm_right_5_joint_offset}" arm_6_offset="${arm_right_6_joint_offset}" arm_7_offset="${arm_right_7_joint_offset}">
+      <origin xyz="0.0 0.0 0.0" rpy="0.0 0.0 -1.5708"/>
     </xacro:pal_sea_arm>
     <!-- End effector -->
@@ -171,5 +171,5 @@
         <xacro:tool_changer name="tool_changer_right" parent="${end_effector_right_link}"/>
         <xacro:allegro_hand name="gripper_right" parent="tool_changer_right_tc_tool_link" reflect="1">
-                <origin xyz="0 0 0.0" rpy="0 0 0"/>
+                <origin xyz="0.0 0.0 0.0" rpy="0.0 0.0 0.0"/>
         </xacro:allegro_hand>
       </xacro:if>

File: triago_description/urdf/torso/torso_dual.urdf.xacro (robot description, xacro)
@@ -140,4 +140,163 @@
     <limit effort="0" lower="0" upper="0.35" velocity="0" />
   </joint>
+  <link
+    name="arm_left_link">
+    <inertial>
+      <origin
+        xyz="0.024927 -0.0093838 -0.030755"
+        rpy="0 0 0" />
+      <mass
+        value="0.23047" />
+      <inertia
+        ixx="0.00026511"
+        ixy="1.3047E-06"
+        ixz="7.8189E-05"
+        iyy="0.00035859"
+        iyz="-5.3396E-05"
+        izz="0.00040319" />
+    </inertial>
+    <visual>
+      <origin
+        xyz="0 0 0"
+        rpy="0 0 0" />
+      <geometry>
+        <mesh
+          filename="package://triago_description/meshes/torso/arm_left_link.STL" />
+      </geometry>
+      <material
+        name="">
+        <color
+          rgba="0.25098 0.25098 0.25098 1" />
+      </material>
+    </visual>
+    <collision>
+      <origin
+        xyz="0 0 0"
+        rpy="0 0 0" />
+      <geometry>
+        <mesh
+          filename="package://triago_description/meshes/torso/arm_left_link.STL" />
+      </geometry>
+    </collision>
+  </link>
+  <joint
+    name="arm_left_link"
+    type="fixed">
+    <origin
+      xyz="0.089428 0.15903 0.46268"
+      rpy="-2.0961 0.31441 -1.3991" />
+    <parent
+      link="${name}_lift_link" />
+    <child
+      link="arm_left_link" />
+    <axis
+      xyz="0 0 0" />
+  </joint>
+ <link
+    name="arm_right_link">
+    <inertial>
+      <origin
+        xyz="-0.025026 -0.009123 -0.031256"
+        rpy="0 0 0" />
+      <mass
+        value="0.23047" />
+      <inertia
+        ixx="0.00026509"
+        ixy="-3.1836E-07"
+        ixz="-7.8741E-05"
+        iyy="0.00035861"
+        iyz="-5.257E-05"
+        izz="0.00040319" />
+    </inertial>
+    <visual>
+      <origin
+        xyz="0 0 0"
+        rpy="0 0 0" />
+      <geometry>
+        <mesh
+          filename="package://triago_description/meshes/torso/arm_right_link.STL" />
+      </geometry>
+      <material
+        name="">
+        <color
+          rgba="0.25098 0.25098 0.25098 1" />
+      </material>
+    </visual>
+    <collision>
+      <origin
+        xyz="0 0 0"
+        rpy="0 0 0" />
+      <geometry>
+        <mesh
+          filename="package://triago_description/meshes/torso/arm_right_link.STL" />
+      </geometry>
+    </collision>
+  </link>
+  <joint
+    name="arm_right_joint"
+    type="fixed">
+    <origin
+      xyz="0.0898413194899457 -0.159181203217083 0.462445262450827"
+      rpy="-2.09439510239319 -0.305349554638743 -1.74800742587503" />
+    <parent
+      link="${name}_lift_link" />
+    <child
+      link="arm_right_link" />
+    <axis
+      xyz="0 0 0" />
+  </joint>
+ <link
+    name="arm_head_link">
+    <inertial>
+      <origin
+        xyz="0.01289 -1.9489E-07 -0.017393"
+        rpy="0 0 0" />
+      <mass
+        value="0.18229" />
+      <inertia
+        ixx="0.00027537"
+        ixy="7.4919E-10"
+        ixz="7.2758E-06"
+        iyy="0.00018169"
+        iyz="-2.2164E-10"
+        izz="0.00037953" />
+    </inertial>
+    <visual>
+      <origin
+        xyz="0 0 0"
+        rpy="0 0 0" />
+      <geometry>
+        <mesh
+          filename="package://triago_description/meshes/torso/arm_head_link.STL" />
+      </geometry>
+      <material
+        name="">
+        <color
+          rgba="0.25098 0.25098 0.25098 1" />
+      </material>
+    </visual>
+    <collision>
+      <origin
+        xyz="0 0 0"
+        rpy="0 0 0" />
+      <geometry>
+        <mesh
+          filename="package://triago_description/meshes/torso/arm_head_link.STL" />
+      </geometry>
+    </collision>
+  </link>
+  <joint
+    name="arm_head_joint"
+    type="fixed">
+    <origin
+      xyz="0.00733452377915612 0 0.630632193308821"
+      rpy="0 0.785398163397445 0" />
+    <parent
+      link="${name}_lift_link" />
+    <child
+      link="arm_head_link" />
+    <axis
+      xyz="0 0 0" />
+  </joint>
   </xacro:macro>
 </robot>

Commit message: Add arm head controller

File: triago_description/robots/triago.urdf.xacro (robot description, xacro)
@@ -119,5 +119,5 @@
   </xacro:if>
   <!-- Allegro hand and tool changer-->
-  <xacro:if value="${end_effector_right == 'allegro-hand'}">
+  <xacro:if value="${end_effector_right == 'allegro-hand' or end_effector_left == 'allegro-hand' or end_effector_head == 'allegro-hand'}">
     <xacro:include filename="$(find triago_description)/urdf/tool_changer/tool_changer.urdf.xacro" />
     <xacro:include filename="$(find allegro_hand_description)/urdf/allegro_hand.urdf.xacro" />
@@ -141,5 +141,5 @@
     <!-- Arm -->
     <xacro:pal_sea_arm name="arm_left" parent="arm_left_link" arm_type="$(arg arm_type_left)" reflect="1" arm_1_offset="${arm_left_1_joint_offset}" arm_2_offset="${arm_left_2_joint_offset}" arm_3_offset="${arm_left_3_joint_offset}" arm_4_offset="${arm_left_4_joint_offset}" arm_5_offset="${arm_left_5_joint_offset}" arm_6_offset="${arm_left_6_joint_offset}" arm_7_offset="${arm_left_7_joint_offset}">
-      <origin xyz="0.0 0.0 0.0" rpy="0.0 0.0 -1.5708"/>
+      <origin xyz="0.0 0.0 0.0" rpy="0.0 0.0 1.5708"/>
     </xacro:pal_sea_arm>
     <!-- End effector -->
@@ -148,5 +148,5 @@
         <xacro:tool_changer name="tool_changer_left" parent="${end_effector_left_link}"/>
         <xacro:allegro_hand name="gripper_left" parent="tool_changer_left_tc_tool_link" reflect="-1">
-                <origin xyz="0 0 0.0" rpy="0 0 0"/>
+                <origin xyz="0 0 0.0" rpy="0 0 3.14"/>
         </xacro:allegro_hand>
       </xacro:if>
@@ -171,5 +171,5 @@
         <xacro:tool_changer name="tool_changer_right" parent="${end_effector_right_link}"/>
         <xacro:allegro_hand name="gripper_right" parent="tool_changer_right_tc_tool_link" reflect="1">
-                <origin xyz="0.0 0.0 0.0" rpy="0.0 0.0 0.0"/>
+                <origin xyz="0.0 0.0 0.0" rpy="0.0 0.0 -1.57"/>
         </xacro:allegro_hand>
       </xacro:if>
@@ -190,15 +190,15 @@
     </xacro:pal_sea_arm>
     <!-- End effector -->
-    <!--xacro:if value="${has_end_effector_head}">
+    <xacro:if value="${has_end_effector_head}">
       <xacro:if  value="${end_effector_head == 'allegro-hand'}">
         <xacro:tool_changer name="tool_changer_head" parent="${end_effector_head_link}"/>
-        <xacro:allegro-hand name="gripper_head" parent="tool_changer_head_tc_tool_link" reflect="1">
+        <xacro:allegro_hand name="gripper_head" parent="tool_changer_head_tc_tool_link" reflect="1">
                 <origin xyz="0 0 0.0" rpy="0 0 0"/>
-        </xacro:allegro-hand>
+        </xacro:allegro_hand>
       </xacro:if>
       <xacro:unless value="${end_effector_head == 'allegro-hand'}">
         <xacro:pal_sea_arm_end_effector name="gripper_head" parent="${end_effector_head_link}" type="${end_effector_head}" has_end_effector="${has_end_effector_head}" reflect="1" is_dual="true"/>
       </xacro:unless>
-    </xacro:if-->
+    </xacro:if>
     <!-- FT sensors -->
     <!--xacro:if value="${has_ft_sensor_head}">

File: triago_description/ros2_control/ros2_control.urdf.xacro (robot description, xacro)
@@ -36,6 +36,9 @@
     <xacro:include filename="$(find triago_description)/urdf/torso/torso.ros2_control.xacro" />
     <xacro:include filename="$(find pal_sea_arm_description)/urdf/arm/arm.ros2_control.xacro" />
-    <xacro:if value="${end_effector_left == 'pal-pro-gripper' or end_effector_right == 'pal-pro-gripper'}">
+    <xacro:if value="${end_effector_left == 'pal-pro-gripper' or end_effector_right == 'pal-pro-gripper' or end_effector_head== 'pal-pro-gripper'}">
       <xacro:include filename="$(find pal_pro_gripper_description)/urdf/pal_pro_gripper.ros2_control.xacro" />
+    </xacro:if>
+    <xacro:if value="${end_effector_left == 'allegro-hand' or end_effector_right == 'allegro-hand' or end_effector_head== 'allegro-hand'}">
+      <xacro:include filename="$(find allegro_hand_description)/urdf/allegro_hand.ros2_control.xacro" />
     </xacro:if>
     <!-- calibration offsets -->
@@ -69,4 +72,5 @@
       <!-- torso -->
       <xacro:ros2_control_torso name="torso_lift" reduction="1.0" />
+    <xacro:arg name="pid_controllers" default="false"/>
       <!-- arm left -->
       <xacro:if value="${has_arm_left}">
@@ -85,4 +89,8 @@
           <xacro:ros2_control_pal_pro_gripper name="gripper_left" reduction="1.0" />
         </xacro:if>
+        <xacro:if value="${end_effector_left == 'allegro-hand'}">
+          <!-- allegro-hand -->
+          <xacro:ros2_control_allegro_hand name="gripper_left" pid_controllers="$(arg pid_controllers)" reduction="1.0" />
+        </xacro:if>
       </xacro:if>
       <!-- arm right -->
@@ -99,5 +107,14 @@
           <xacro:ros2_control_force_torque_sensor name="wrist_right_ft_sensor"/>s
         </xacro:if>
-      <!-- arm head -->
+        <xacro:if value="${end_effector_right == 'pal-pro-gripper'}">
+          <!-- pal-pro-gripper -->
+          <xacro:ros2_control_pal_pro_gripper name="gripper_right" reduction="1.0" />
+        </xacro:if>
+        <xacro:if value="${end_effector_right == 'allegro-hand'}">
+          <!-- allegro-hand -->
+          <xacro:ros2_control_allegro_hand name="gripper_right" pid_controllers="$(arg pid_controllers)" reduction="1.0" />
+        </xacro:if>
+      </xacro:if>
+       <!-- arm head -->
       <xacro:if value="${has_arm_head}">
         <xacro:ros2_control_arm name="arm_head_1" reduction="1.0" offset_value="${arm_left_1_joint_offset}" />
@@ -112,11 +129,9 @@
           <xacro:ros2_control_force_torque_sensor name="wrist_left_ft_sensor"/>
         </xacro:if-->
-        <xacro:if value="${end_effector_left == 'pal-pro-gripper'}">
-          <xacro:ros2_control_pal_pro_gripper name="gripper_left" reduction="1.0" />
+        <xacro:if value="${end_effector_head == 'pal-pro-gripper'}">
+          <xacro:ros2_control_pal_pro_gripper name="gripper_head" reduction="1.0" />
         </xacro:if>
-      </xacro:if>
-        <xacro:if value="${end_effector_right == 'pal-pro-gripper'}">
-          <!-- pal-pro-gripper -->
-          <xacro:ros2_control_pal_pro_gripper name="gripper_right" reduction="1.0" />
+        <xacro:if value="${end_effector_head == 'allegro-hand'}">
+          <xacro:ros2_control_allegro_hand name="gripper_head" pid_controllers="$(arg pid_controllers)" reduction="1.0" />
         </xacro:if>
       </xacro:if>

Commit message: Fixing tool changer and allegro hand

File: triago_description/robots/triago.urdf.xacro (robot description, xacro)
@@ -20,12 +20,15 @@
   <!-- triago, no-arm -->
   <xacro:arg name="arm_type_right" default="triago" />
+  <xacro:arg name="arm_type_head" default="triago" />
   <!-- pal-pro-gripper custom-->
   <xacro:arg name="end_effector_left" default="pal-pro-gripper" />
   <!-- pal-pro-gripper, custom-->
   <xacro:arg name="end_effector_right" default="pal-pro-gripper" />
+  <xacro:arg name="end_effector_head" default="pal-pro-gripper" />
   <!-- no-ft-sensor, rokubi -->
   <xacro:arg name="ft_sensor_left" default="no-ft-sensor" />
   <!-- no-ft-sensor, rokubi -->
   <xacro:arg name="ft_sensor_right" default="no-ft-sensor" />
+  <xacro:arg name="ft_sensor_head" default="no-ft-sensor" />
   <xacro:arg name="use_sim_time" default="false"/>
   <xacro:arg name="is_public_sim" default="false"/>
@@ -50,5 +53,5 @@
   <xacro:property name="end_effector_head" value="$(arg end_effector_head)" />
   <xacro:property name="ft_sensor_left" value="$(arg ft_sensor_left)" />
-  <xacro:property name="ft_sensor_right" value="$(arg ft_sensor_head)" />
+  <xacro:property name="ft_sensor_right" value="$(arg ft_sensor_right)" />
   <xacro:property name="ft_sensor_head" value="$(arg ft_sensor_head)" />
   <xacro:property name="arm_type" value="triago" />
@@ -141,12 +144,19 @@
     <!-- Arm -->
     <xacro:pal_sea_arm name="arm_left" parent="arm_left_link" arm_type="$(arg arm_type_left)" reflect="1" arm_1_offset="${arm_left_1_joint_offset}" arm_2_offset="${arm_left_2_joint_offset}" arm_3_offset="${arm_left_3_joint_offset}" arm_4_offset="${arm_left_4_joint_offset}" arm_5_offset="${arm_left_5_joint_offset}" arm_6_offset="${arm_left_6_joint_offset}" arm_7_offset="${arm_left_7_joint_offset}">
-      <origin xyz="0.0 0.0 0.0" rpy="0.0 0.0 1.5708"/>
+      <origin xyz="0.0 0.0 0.0" rpy="0.0 0.0 ${90.0 * deg_to_rad}"/>
     </xacro:pal_sea_arm>
     <!-- End effector -->
     <xacro:if value="${has_end_effector_left}">
       <xacro:if value="${end_effector_left == 'allegro-hand'}">
-        <xacro:tool_changer name="tool_changer_left" parent="${end_effector_left_link}"/>
+        <xacro:tool_changer name="tool_changer_left" parent="${end_effector_left_link}">
+            <xacro:if value="${has_ft_sensor_left}">
+              <origin xyz="0.0 0.0 0.0" rpy="0.0 0.0 0.0"/>
+            </xacro:if>
+            <xacro:unless value="${has_ft_sensor_left}">
+              <origin xyz="0.0 0.0 0.0" rpy="${-90.0 * deg_to_rad} ${90.0 * deg_to_rad} ${-90.0 * deg_to_rad}"/>
+            </xacro:unless>
+        </xacro:tool_changer>
         <xacro:allegro_hand name="gripper_left" parent="tool_changer_left_tc_tool_link" reflect="-1">
-                <origin xyz="0 0 0.0" rpy="0 0 3.14"/>
+                <origin xyz="-0.00956 -0.001 0.094" rpy="0.0 0.0 ${-180.0 * deg_to_rad}"/>
         </xacro:allegro_hand>
       </xacro:if>
@@ -164,12 +174,19 @@
     <!-- Arm -->
     <xacro:pal_sea_arm name="arm_right" parent="arm_right_link" arm_type="$(arg arm_type_right)" reflect="1" arm_1_offset="${arm_right_1_joint_offset}" arm_2_offset="${arm_right_2_joint_offset}" arm_3_offset="${arm_right_3_joint_offset}" arm_4_offset="${arm_right_4_joint_offset}" arm_5_offset="${arm_right_5_joint_offset}" arm_6_offset="${arm_right_6_joint_offset}" arm_7_offset="${arm_right_7_joint_offset}">
-      <origin xyz="0.0 0.0 0.0" rpy="0.0 0.0 -1.5708"/>
+      <origin xyz="0.0 0.0 0.0" rpy="0.0 0.0 ${-90.0 * deg_to_rad}"/>
     </xacro:pal_sea_arm>
     <!-- End effector -->
     <xacro:if value="${has_end_effector_right}">
       <xacro:if value="${end_effector_right == 'allegro-hand'}">
-        <xacro:tool_changer name="tool_changer_right" parent="${end_effector_right_link}"/>
+        <xacro:tool_changer name="tool_changer_right" parent="${end_effector_right_link}">
+         <xacro:if value="${has_ft_sensor_left}">
+              <origin xyz="0.0 0.0 0.0" rpy="0.0 0.0 0.0"/>
+            </xacro:if>
+            <xacro:unless value="${has_ft_sensor_left}">
+              <origin xyz="0.0 0.0 0.0" rpy="${-90.0 * deg_to_rad} ${90.0 * deg_to_rad} ${-90.0 * deg_to_rad}"/>
+            </xacro:unless>
+        </xacro:tool_changer>
         <xacro:allegro_hand name="gripper_right" parent="tool_changer_right_tc_tool_link" reflect="1">
-                <origin xyz="0.0 0.0 0.0" rpy="0.0 0.0 -1.57"/>
+                <origin xyz="-0.00956 -0.001 0.094" rpy="0.0 0.0 ${-180.0 * deg_to_rad}"/>
         </xacro:allegro_hand>
       </xacro:if>

File: triago_description/urdf/ft_sensor/ft_sensor.urdf.xacro (robot description, xacro)
@@ -49,5 +49,5 @@
       <parent link="${parent}" />
       <child link="${name}_ft_base_link" />
-      <origin xyz="0.0 0 0" rpy="${-90.0 * deg_to_rad} ${45.0 * deg_to_rad} ${-90.0 * deg_to_rad}" />
+      <origin xyz="-0.0184 -0 0" rpy="${-90.0 * deg_to_rad} ${90.0 * deg_to_rad} ${-90.0 * deg_to_rad}" />
     </joint>
     <gazebo reference="${name}_ft_base_link">
@@ -125,5 +125,5 @@
       <parent link="${name}_ft_base_link" />
       <child link="${name}_ft_tool_link" />
-      <origin xyz="0 0 0.039998" rpy="${45.0 * deg_to_rad} ${-90.0 * deg_to_rad} ${0.0 * deg_to_rad}" />
+      <origin xyz="0 0 0.039998" rpy="0 0 0" />
     </joint>
 </xacro:macro>

File: triago_description/urdf/tool_changer/tool_changer.urdf.xacro (robot description, xacro)
@@ -13,5 +13,5 @@
 -->
 <robot xmlns:xacro="http://ros.org/wiki/xacro">
-  <xacro:macro name="tool_changer" params="name parent">
+  <xacro:macro name="tool_changer" params="name parent *origin">
     <!--************************-->
     <!--        ft sensor       -->
@@ -59,5 +59,5 @@
       <parent link="${parent}" />
       <child link="${name}_tc_base_link" />
-      <origin xyz="0.0 0 0" rpy="${-90.0 * deg_to_rad} ${45.0 * deg_to_rad} ${-90.0 * deg_to_rad}" />
+      <xacro:insert_block name="origin"/>
     </joint>
     <link
