Commit message: Unifying end effector script

File: triago_description/robots/triago.urdf.xacro (robot description, xacro)
@@ -119,15 +119,14 @@
   <!-- End effector -->
   <xacro:if value="${(has_arm_right or has_arm_left) and (has_end_effector_right or has_end_effector_left)}">
-    <xacro:include filename="$(find pal_sea_arm_description)/urdf/end_effector/end_effector.urdf.xacro" />
+    <xacro:include filename="$(find triago_description)/urdf/end_effector/end_effector.urdf.xacro" />
+    <xacro:include filename="$(find triago_description)/urdf/tool_changer/tool_changer.urdf.xacro" />
   </xacro:if>
   <!-- Allegro hand and tool changer-->
   <xacro:if value="${end_effector_right == 'allegro-hand' or end_effector_left == 'allegro-hand' or end_effector_head == 'allegro-hand'}">
-    <xacro:include filename="$(find triago_description)/urdf/tool_changer/tool_changer.urdf.xacro" />
     <xacro:include filename="$(find allegro_hand_description)/urdf/allegro_hand.urdf.xacro" />
   </xacro:if>
   <!-- Force Torque sensor -->
-  <xacro:if value="${has_ft_sensor_right or has_ft_sensor_left}">
+  <xacro:if value="${has_ft_sensor_right or has_ft_sensor_left or has_ft_sensor_head}">
     <xacro:include filename="$(find triago_description)/urdf/ft_sensor/ft_sensor.urdf.xacro" />
-    <xacro:include filename="$(find pal_sea_arm_description)/urdf/sensors/ft_sensor.gazebo.xacro" />
   </xacro:if>
   <!-- Materials for visualization -->
@@ -148,7 +147,6 @@
     <!-- End effector -->
     <xacro:if value="${has_end_effector_left}">
-      <xacro:if value="${end_effector_left == 'allegro-hand'}">
-        <xacro:tool_changer name="tool_changer_left" parent="${end_effector_left_link}">
-            <xacro:if value="${has_ft_sensor_left}">
+       <xacro:tool_changer name="tool_changer_left" parent="${end_effector_left_link}">
+         <xacro:if value="${has_ft_sensor_left}">
               <origin xyz="0.0 0.0 0.0" rpy="0.0 0.0 0.0"/>
             </xacro:if>
@@ -157,11 +155,5 @@
             </xacro:unless>
         </xacro:tool_changer>
-        <xacro:allegro_hand name="gripper_left" parent="tool_changer_left_tc_tool_link" reflect="-1">
-                <origin xyz="-0.00956 -0.001 0.094" rpy="0.0 0.0 ${-180.0 * deg_to_rad}"/>
-        </xacro:allegro_hand>
-      </xacro:if>
-      <xacro:unless value="${end_effector_left == 'allegro-hand'}">
-        <xacro:pal_sea_arm_end_effector name="gripper_left" parent="${end_effector_left_link}" type="${end_effector_left}" has_end_effector="${has_end_effector_left}" reflect="-1" is_dual="true"/>
-      </xacro:unless>
+      <xacro:triago_end_effector name="gripper_left" parent="tool_changer_left_tc_tool_link" type="${end_effector_left}" has_end_effector="${has_end_effector_left}" reflect="-1" is_dual="true"/>
     </xacro:if>
     <!-- FT sensors -->
@@ -178,20 +170,13 @@
     <!-- End effector -->
     <xacro:if value="${has_end_effector_right}">
-      <xacro:if value="${end_effector_right == 'allegro-hand'}">
-        <xacro:tool_changer name="tool_changer_right" parent="${end_effector_right_link}">
-         <xacro:if value="${has_ft_sensor_left}">
+       <xacro:tool_changer name="tool_changer_right" parent="${end_effector_right_link}">
+         <xacro:if value="${has_ft_sensor_right}">
               <origin xyz="0.0 0.0 0.0" rpy="0.0 0.0 0.0"/>
             </xacro:if>
-            <xacro:unless value="${has_ft_sensor_left}">
+            <xacro:unless value="${has_ft_sensor_right}">
               <origin xyz="0.0 0.0 0.0" rpy="${-90.0 * deg_to_rad} ${90.0 * deg_to_rad} ${-90.0 * deg_to_rad}"/>
             </xacro:unless>
         </xacro:tool_changer>
-        <xacro:allegro_hand name="gripper_right" parent="tool_changer_right_tc_tool_link" reflect="1">
-                <origin xyz="-0.00956 -0.001 0.094" rpy="0.0 0.0 ${-180.0 * deg_to_rad}"/>
-        </xacro:allegro_hand>
-      </xacro:if>
-      <xacro:unless value="${end_effector_right == 'allegro-hand'}">
-        <xacro:pal_sea_arm_end_effector name="gripper_right" parent="${end_effector_right_link}" type="${end_effector_right}" has_end_effector="${has_end_effector_right}" reflect="1" is_dual="true"/>
-      </xacro:unless>
+      <xacro:triago_end_effector name="gripper_right" parent="tool_changer_right_tc_tool_link" type="${end_effector_right}" has_end_effector="${has_end_effector_right}" reflect="1" is_dual="true"/>
     </xacro:if>
     <!-- FT sensors -->
@@ -208,18 +193,18 @@
     <!-- End effector -->
     <xacro:if value="${has_end_effector_head}">
-      <xacro:if  value="${end_effector_head == 'allegro-hand'}">
-        <xacro:tool_changer name="tool_changer_head" parent="${end_effector_head_link}"/>
-        <xacro:allegro_hand name="gripper_head" parent="tool_changer_head_tc_tool_link" reflect="1">
-                <origin xyz="0 0 0.0" rpy="0 0 0"/>
-        </xacro:allegro_hand>
-      </xacro:if>
-      <xacro:unless value="${end_effector_head == 'allegro-hand'}">
-        <xacro:pal_sea_arm_end_effector name="gripper_head" parent="${end_effector_head_link}" type="${end_effector_head}" has_end_effector="${has_end_effector_head}" reflect="1" is_dual="true"/>
-      </xacro:unless>
+       <xacro:tool_changer name="tool_changer_head" parent="${end_effector_head_link}">
+         <xacro:if value="${has_ft_sensor_head}">
+              <origin xyz="0.0 0.0 0.0" rpy="0.0 0.0 0.0"/>
+            </xacro:if>
+            <xacro:unless value="${has_ft_sensor_head}">
+              <origin xyz="0.0 0.0 0.0" rpy="${-90.0 * deg_to_rad} ${90.0 * deg_to_rad} ${-90.0 * deg_to_rad}"/>
+            </xacro:unless>
+        </xacro:tool_changer>
+      <xacro:triago_end_effector name="gripper_head" parent="tool_changer_head_tc_tool_link" type="${end_effector_head}" has_end_effector="${has_end_effector_head}" reflect="1" is_dual="true"/>
     </xacro:if>
     <!-- FT sensors -->
-    <!--xacro:if value="${has_ft_sensor_head}">
-      <xacro:ft_sensor name="wrist_right" parent="arm_head_tool_link"/>
-    </xacro:if-->
+    <xacro:if value="${has_ft_sensor_head}">
+      <xacro:ft_sensor name="wrist_head" parent="arm_head_tool_link"/>
+    </xacro:if>
   </xacro:if>
   <!-- ROS 2 Control -->

Commit message: Fixing play motion launch

File: triago_description/robots/triago.urdf.xacro (robot description, xacro)
@@ -22,10 +22,10 @@
   <xacro:arg name="arm_type_head" default="triago" />
   <!-- pal-pro-gripper custom-->
-  <xacro:arg name="end_effector_left" default="pal-pro-gripper" />
+  <xacro:arg name="end_effector_left" default="allegro-hand" />
   <!-- pal-pro-gripper, custom-->
-  <xacro:arg name="end_effector_right" default="pal-pro-gripper" />
+  <xacro:arg name="end_effector_right" default="allegro-hand" />
   <xacro:arg name="end_effector_head" default="pal-pro-gripper" />
   <!-- no-ft-sensor, ati-mini45 -->
-  <xacro:arg name="ft_sensor_left" default="no-ft-sensor" />
+  <xacro:arg name="ft_sensor_left" default="ati-mini45" />
   <!-- no-ft-sensor, ati-mini45 -->
   <xacro:arg name="ft_sensor_right" default="no-ft-sensor" />
@@ -114,9 +114,9 @@
   <xacro:include filename="$(arg description_calibration_dir)/calibration_constants.urdf.xacro" />
   <!-- Arm -->
-  <xacro:if value="${has_arm_right or has_arm_left}">
+  <xacro:if value="${has_arm_right or has_arm_left or has_arm_head}">
     <xacro:include filename="$(find pal_sea_arm_description)/urdf/arm/arm.urdf.xacro" />
   </xacro:if>
   <!-- End effector -->
-  <xacro:if value="${(has_arm_right or has_arm_left) and (has_end_effector_right or has_end_effector_left)}">
+  <xacro:if value="${(has_arm_right or has_arm_left or has_arm_head) and (has_end_effector_right or has_end_effector_left or has_end_effector_head)}">
     <xacro:include filename="$(find triago_description)/urdf/end_effector/end_effector.urdf.xacro" />
     <xacro:include filename="$(find pal_sea_arm_description)/urdf/tool_changer/tool_changer.urdf.xacro" />
@@ -139,5 +139,5 @@
     <!-- Arm -->
     <xacro:pal_sea_arm name="arm_left" parent="arm_left_link" arm_type="$(arg arm_type_left)" reflect="1" arm_1_offset="${arm_left_1_joint_offset}" arm_2_offset="${arm_left_2_joint_offset}" arm_3_offset="${arm_left_3_joint_offset}" arm_4_offset="${arm_left_4_joint_offset}" arm_5_offset="${arm_left_5_joint_offset}" arm_6_offset="${arm_left_6_joint_offset}" arm_7_offset="${arm_left_7_joint_offset}">
-      <origin xyz="0.0 0.0 0.0" rpy="0.0 0.0 ${90.0 * deg_to_rad}"/>
+      <origin xyz="0.0 0.0 0.0" rpy="0.0 0.0 ${-111.0 * deg_to_rad}"/>
     </xacro:pal_sea_arm>
     <!-- End effector -->
@@ -145,5 +145,5 @@
        <xacro:tool_changer name="tool_changer_left" parent="${end_effector_left_link}">
          <xacro:if value="${has_ft_sensor_left}">
-              <origin xyz="0.0 0.0 0.0" rpy="0.0 0.0 0.0"/>
+              <origin xyz="0.0 0.0 0.0" rpy="0.0 0.0 ${-180.0 * deg_to_rad}"/>
             </xacro:if>
             <xacro:unless value="${has_ft_sensor_left}">
@@ -162,5 +162,5 @@
     <!-- Arm -->
     <xacro:pal_sea_arm name="arm_right" parent="arm_right_link" arm_type="$(arg arm_type_right)" reflect="1" arm_1_offset="${arm_right_1_joint_offset}" arm_2_offset="${arm_right_2_joint_offset}" arm_3_offset="${arm_right_3_joint_offset}" arm_4_offset="${arm_right_4_joint_offset}" arm_5_offset="${arm_right_5_joint_offset}" arm_6_offset="${arm_right_6_joint_offset}" arm_7_offset="${arm_right_7_joint_offset}">
-      <origin xyz="0.0 0.0 0.0" rpy="0.0 0.0 ${-90.0 * deg_to_rad}"/>
+      <origin xyz="0.0 0.0 0.0" rpy="0.0 0.0 ${-69.0 * deg_to_rad}"/>
     </xacro:pal_sea_arm>
     <!-- End effector -->
@@ -184,6 +184,6 @@
   <xacro:if value="${has_arm_head}">
     <!-- Arm -->
-    <xacro:pal_sea_arm name="arm_head" parent="torso_lift_link" arm_type="$(arg arm_type_head)" reflect="1" arm_1_offset="${arm_right_1_joint_offset}" arm_2_offset="${arm_right_2_joint_offset}" arm_3_offset="${arm_right_3_joint_offset}" arm_4_offset="${arm_right_4_joint_offset}" arm_5_offset="${arm_right_5_joint_offset}" arm_6_offset="${arm_right_6_joint_offset}" arm_7_offset="${arm_right_7_joint_offset}">
-      <origin xyz="0.00733452377915612 0.0 0.630632193308821" rpy="0 0.785398163397445 0"/>
+    <xacro:pal_sea_arm name="arm_head" parent="arm_head_link" arm_type="$(arg arm_type_head)" reflect="1" arm_1_offset="${arm_right_1_joint_offset}" arm_2_offset="${arm_right_2_joint_offset}" arm_3_offset="${arm_right_3_joint_offset}" arm_4_offset="${arm_right_4_joint_offset}" arm_5_offset="${arm_right_5_joint_offset}" arm_6_offset="${arm_right_6_joint_offset}" arm_7_offset="${arm_right_7_joint_offset}">
+      <origin xyz="0.0 0.0 0.0" rpy="0 0 0"/>
     </xacro:pal_sea_arm>
     <!-- End effector -->

Commit message: Fixing controller head gripper

File: triago_description/robots/triago.urdf.xacro (robot description, xacro)
@@ -197,5 +197,5 @@
          </xacro:unless>
         </xacro:tool_changer>
-      <xacro:triago_end_effector name="gripper_head" parent="tool_changer_head_tc_tool_link" type="${end_effector_head}" has_end_effector="${has_end_effector_head}" reflect="1" is_dual="true"/>
+      <xacro:triago_end_effector name="gripper" parent="tool_changer_head_tc_tool_link" type="${end_effector_head}" has_end_effector="${has_end_effector_head}" reflect="1" is_dual="true"/>
     </xacro:if>
     <!-- FT sensors -->

File: triago_description/ros2_control/ros2_control.urdf.xacro (robot description, xacro)
@@ -17,8 +17,10 @@
     <xacro:arg name="arm_type_right" default="triago"/>
     <xacro:arg name="arm_type_head" default="triago"/>
-    <xacro:arg name="end_effector_left" default="pal-pro-pripper"/>
-    <xacro:arg name="end_effector_right" default="pal-pro-gripper"/>
+    <xacro:arg name="end_effector_left" default="allegro-hand"/>
+    <xacro:arg name="end_effector_right" default="allegro-hand"/>
+    <xacro:arg name="end_effector_head" default="pal-pro-gripper"/>
     <xacro:arg name="ft_sensor_left" default="no-ft-sensor"/>
     <xacro:arg name="ft_sensor_right" default="no-ft-sensor"/>
+    <xacro:arg name="ft_sensor_head" default="no-ft-sensor"/>
     <xacro:arg name="description_calibration_dir" default="$(find triago_description)/urdf/calibration" />
     <!-- TODO-->
@@ -28,8 +30,11 @@
     <xacro:property name="end_effector_left" value="$(arg end_effector_left)" />
     <xacro:property name="end_effector_right" value="$(arg end_effector_right)" />
+    <xacro:property name="end_effector_head" value="$(arg end_effector_head)" />
     <xacro:property name="has_ft_sensor_left" value="${ft_sensor_left != 'no-ft-sensor'}" />
     <xacro:property name="has_ft_sensor_right" value="${ft_sensor_right != 'no-ft-sensor'}" />
+    <xacro:property name="has_ft_sensor_head" value="${ft_sensor_head != 'no-ft-sensor'}" />
     <xacro:property name="has_arm_left" value="${arm_type_left != 'no-arm'}" />
     <xacro:property name="has_arm_right" value="${arm_type_right != 'no-arm'}" />
+    <xacro:property name="has_arm_head" value="${arm_type_head != 'no-arm'}" />
     <xacro:include filename="$(find omni_base_description)/urdf/sensors/sensors.ros2_control.xacro" />
     <xacro:include filename="$(find omni_base_description)/urdf/wheels/wheel.ros2_control.xacro" />
@@ -130,5 +135,5 @@
         </xacro:if-->
         <xacro:if value="${end_effector_head == 'pal-pro-gripper'}">
-          <xacro:ros2_control_pal_pro_gripper name="gripper_head" reduction="1.0" />
+          <xacro:ros2_control_pal_pro_gripper name="gripper" reduction="1.0" />
         </xacro:if>
         <xacro:if value="${end_effector_head == 'allegro-hand'}">

Commit message: Adding side option for end effector of the head

File: triago_description/robots/triago.urdf.xacro (robot description, xacro)
@@ -26,4 +26,5 @@
   <xacro:arg name="end_effector_right" default="allegro-hand" />
   <xacro:arg name="end_effector_head" default="pal-pro-gripper" />
+  <xacro:arg name="hand_head_type" default="" />
   <!-- no-ft-sensor, ati-mini45 -->
   <xacro:arg name="ft_sensor_left" default="ati-mini45" />
@@ -72,5 +73,12 @@
   <xacro:property name="has_end_effector_head" value="${end_effector_head not in ['no-end-effector']}" />
   <xacro:property name="end_effector_head_link" value="${'wrist_head_ft_tool_link' if has_ft_sensor_head else 'arm_head_tool_link'}" />
-  <xacro:property name="end_effector_head_name" value="gripper_head" />
+  <xacro:property name="hand_head_type" value="$(arg hand_head_type)" />
+  <xacro:property name="end_effector_head_name" value="gripper" />
+  <xacro:if value="${hand_head_type == 'left'}">
+    <xacro:property name="head_hand_reflect" value="-1" />
+  </xacro:if>
+  <xacro:unless value="${hand_head_type == 'left'}">
+    <xacro:property name="head_hand_reflect" value="1" />
+  </xacro:unless>
   <!-- Properties check -->
   <xacro:if value="${arm_type_left not in ['triago', 'no-arm']}">
@@ -197,5 +205,5 @@
          </xacro:unless>
         </xacro:tool_changer>
-      <xacro:triago_end_effector name="gripper" parent="tool_changer_head_tc_tool_link" type="${end_effector_head}" has_end_effector="${has_end_effector_head}" reflect="1" is_dual="true"/>
+      <xacro:triago_end_effector name="gripper" parent="tool_changer_head_tc_tool_link" type="${end_effector_head}" has_end_effector="${has_end_effector_head}" reflect="${head_hand_reflect}" is_dual="true"/>
     </xacro:if>
     <!-- FT sensors -->

File: triago_description/ros2_control/ros2_control.urdf.xacro (robot description, xacro)
@@ -138,5 +138,5 @@
         </xacro:if>
         <xacro:if value="${end_effector_head == 'allegro-hand'}">
-          <xacro:ros2_control_allegro_hand name="gripper_head" pid_controllers="$(arg pid_controllers)" reduction="1.0" />
+          <xacro:ros2_control_allegro_hand name="gripper" pid_controllers="$(arg pid_controllers)" reduction="1.0" />
         </xacro:if>
       </xacro:if>
