Commit message: Using tiago_pro arm

File: triago_description/robots/triago.urdf.xacro (robot description, xacro)
@@ -17,8 +17,8 @@
   <xacro:arg name="laser_model" default="sick-571"/>
   <!-- triago, no-arm -->
-  <xacro:arg name="arm_type_left" default="triago" />
+  <xacro:arg name="arm_type_left" default="tiago-pro" />
   <!-- triago, no-arm -->
-  <xacro:arg name="arm_type_right" default="triago" />
-  <xacro:arg name="arm_type_head" default="triago" />
+  <xacro:arg name="arm_type_right" default="tiago-pro" />
+  <xacro:arg name="arm_type_head" default="tiago-pro" />
   <!-- pal-pro-gripper custom-->
   <xacro:arg name="end_effector_left" default="allegro-hand" />
@@ -56,5 +56,4 @@
   <xacro:property name="ft_sensor_right" value="$(arg ft_sensor_right)" />
   <xacro:property name="ft_sensor_head" value="$(arg ft_sensor_head)" />
-  <xacro:property name="arm_type" value="triago" />
   <xacro:property name="description_calibration_dir" value="${arg description_calibration_dir}"/>
   <xacro:property name="is_public_sim" value="$(arg is_public_sim)" />
@@ -82,11 +81,11 @@
   </xacro:unless>
   <!-- Properties check -->
-  <xacro:if value="${arm_type_left not in ['triago', 'no-arm']}">
+  <xacro:if value="${arm_type_left not in ['tiago-pro', 'no-arm']}">
     <xacro:wrong_arm_type_left />
   </xacro:if>
-  <xacro:if value="${arm_type_right not in ['triago', 'no-arm']}">
+  <xacro:if value="${arm_type_right not in ['tiago-pro', 'no-arm']}">
     <xacro:wrong_arm_type_right />
   </xacro:if>
-  <xacro:if value="${arm_type_head not in ['triago', 'no-arm']}">
+  <xacro:if value="${arm_type_head not in ['tiago-pro', 'no-arm']}">
     <xacro:wrong_arm_type_head />
   </xacro:if>
@@ -146,6 +145,6 @@
   <xacro:if value="${has_arm_left}">
     <!-- Arm -->
-    <xacro:pal_sea_arm name="arm_left" parent="arm_left_link" arm_type="$(arg arm_type_left)" reflect="1" arm_1_offset="${arm_left_1_joint_offset}" arm_2_offset="${arm_left_2_joint_offset}" arm_3_offset="${arm_left_3_joint_offset}" arm_4_offset="${arm_left_4_joint_offset}" arm_5_offset="${arm_left_5_joint_offset}" arm_6_offset="${arm_left_6_joint_offset}" arm_7_offset="${arm_left_7_joint_offset}">
-      <origin xyz="0.0 0.0 0.0" rpy="0.0 0.0 ${-111.0 * deg_to_rad}"/>
+    <xacro:pal_sea_arm name="arm_left" parent="torso_lift_link" arm_type="$(arg arm_type_left)" reflect="1" arm_1_offset="${arm_left_1_joint_offset}" arm_2_offset="${arm_left_2_joint_offset}" arm_3_offset="${arm_left_3_joint_offset}" arm_4_offset="${arm_left_4_joint_offset}" arm_5_offset="${arm_left_5_joint_offset}" arm_6_offset="${arm_left_6_joint_offset}" arm_7_offset="${arm_left_7_joint_offset}">
+      <origin xyz="$(arg arm_x) $(arg arm_y) $(arg arm_z)" rpy="$(arg arm_roll) $(arg arm_pitch) $(arg arm_yaw)"/>
     </xacro:pal_sea_arm>
     <!-- End effector -->
@@ -153,5 +152,5 @@
        <xacro:tool_changer name="tool_changer_left" parent="${end_effector_left_link}">
          <xacro:if value="${has_ft_sensor_left}">
-              <origin xyz="0.0 0.0 0.0" rpy="0.0 0.0 ${-180.0 * deg_to_rad}"/>
+              <origin xyz="0.0 0.0 0.0" rpy="0.0 0.0 0.0"/>
             </xacro:if>
             <xacro:unless value="${has_ft_sensor_left}">
@@ -169,6 +168,6 @@
   <xacro:if value="${has_arm_right}">
     <!-- Arm -->
-    <xacro:pal_sea_arm name="arm_right" parent="arm_right_link" arm_type="$(arg arm_type_right)" reflect="1" arm_1_offset="${arm_right_1_joint_offset}" arm_2_offset="${arm_right_2_joint_offset}" arm_3_offset="${arm_right_3_joint_offset}" arm_4_offset="${arm_right_4_joint_offset}" arm_5_offset="${arm_right_5_joint_offset}" arm_6_offset="${arm_right_6_joint_offset}" arm_7_offset="${arm_right_7_joint_offset}">
-      <origin xyz="0.0 0.0 0.0" rpy="0.0 0.0 ${-69.0 * deg_to_rad}"/>
+    <xacro:pal_sea_arm name="arm_right" parent="torso_lift_link" arm_type="$(arg arm_type_right)" reflect="1" arm_1_offset="${arm_right_1_joint_offset}" arm_2_offset="${arm_right_2_joint_offset}" arm_3_offset="${arm_right_3_joint_offset}" arm_4_offset="${arm_right_4_joint_offset}" arm_5_offset="${arm_right_5_joint_offset}" arm_6_offset="${arm_right_6_joint_offset}" arm_7_offset="${arm_right_7_joint_offset}">
+      <origin xyz="$(arg arm_x) ${-1.0*$(arg arm_y)} $(arg arm_z)" rpy="$(arg arm_roll) ${-1.0*$(arg arm_pitch)} ${-3.14159 -$(arg arm_yaw)}"/>
     </xacro:pal_sea_arm>
     <!-- End effector -->
@@ -176,5 +175,5 @@
        <xacro:tool_changer name="tool_changer_right" parent="${end_effector_right_link}">
          <xacro:if value="${has_ft_sensor_right}">
-              <origin xyz="0.0 0.0 0.0" rpy="0.0 0.0 0.0"/>
+              <origin xyz="0.0 0.0 0.0" rpy="0.0 0.0 ${-180.0 * deg_to_rad}"/>
             </xacro:if>
             <xacro:unless value="${has_ft_sensor_right}">
@@ -192,6 +191,6 @@
   <xacro:if value="${has_arm_head}">
     <!-- Arm -->
-    <xacro:pal_sea_arm name="arm_head" parent="arm_head_link" arm_type="$(arg arm_type_head)" reflect="1" arm_1_offset="${arm_right_1_joint_offset}" arm_2_offset="${arm_right_2_joint_offset}" arm_3_offset="${arm_right_3_joint_offset}" arm_4_offset="${arm_right_4_joint_offset}" arm_5_offset="${arm_right_5_joint_offset}" arm_6_offset="${arm_right_6_joint_offset}" arm_7_offset="${arm_right_7_joint_offset}">
-      <origin xyz="0.0 0.0 0.0" rpy="0 0 0"/>
+    <xacro:pal_sea_arm name="arm_head" parent="torso_lift_link" arm_type="$(arg arm_type_head)" reflect="1" arm_1_offset="${arm_right_1_joint_offset}" arm_2_offset="${arm_right_2_joint_offset}" arm_3_offset="${arm_right_3_joint_offset}" arm_4_offset="${arm_right_4_joint_offset}" arm_5_offset="${arm_right_5_joint_offset}" arm_6_offset="${arm_right_6_joint_offset}" arm_7_offset="${arm_right_7_joint_offset}">
+      <origin xyz="0.00733452377915612 0 0.630632193308821" rpy="0 0.785398163397445 0" />
     </xacro:pal_sea_arm>
     <!-- End effector -->

File: triago_description/urdf/torso/torso_dual.urdf.xacro (robot description, xacro)
@@ -141,8 +141,8 @@
   </joint>
   <link
-    name="arm_left_link">
-    <inertial>
-      <origin
-        xyz="0.024927 -0.0093838 -0.030755"
+    name="${name}_arm_left_link">
+    <inertial>
+      <origin
+        xyz="0 0 0"
         rpy="0 0 0" />
       <mass
@@ -181,21 +181,19 @@
   </link>
   <joint
-    name="arm_left_link"
+    name="${name}_arm_left_joint"
     type="fixed">
-    <origin
-      xyz="0.089428 0.15903 0.46268"
-      rpy="-2.0961 0.31441 -1.3991" />
+    <origin xyz="0.0898413194899453 0.159181203216899 -0.0920547375491735" rpy="-2.06788770984932 0 -1.22173047639603" />
     <parent
       link="${name}_lift_link" />
     <child
-      link="arm_left_link" />
+      link="${name}_arm_left_link" />
     <axis
       xyz="0 0 0" />
   </joint>
  <link
-    name="arm_right_link">
-    <inertial>
-      <origin
-        xyz="-0.025026 -0.009123 -0.031256"
+    name="${name}_arm_right_link">
+    <inertial>
+      <origin
+        xyz="0 0 0"
         rpy="0 0 0" />
       <mass
@@ -234,21 +232,19 @@
   </link>
   <joint
-    name="arm_right_joint"
+    name="${name}_arm_right_joint"
     type="fixed">
-    <origin
-      xyz="0.0898413194899457 -0.159181203217083 0.462445262450827"
-      rpy="-2.09439510239319 -0.305349554638743 -1.74800742587503" />
+    <origin xyz="0.0898413194899453 -0.1591812032169 -0.0920547375491731" rpy="-2.06788770984932 0 -1.91986217719377" />
     <parent
       link="${name}_lift_link" />
     <child
-      link="arm_right_link" />
+      link="${name}_arm_right_link" />
     <axis
       xyz="0 0 0" />
   </joint>
  <link
-    name="arm_head_link">
-    <inertial>
-      <origin
-        xyz="0.01289 -1.9489E-07 -0.017393"
+    name="${name}_arm_head_link">
+    <inertial>
+      <origin
+        xyz="0 0 0"
         rpy="0 0 0" />
       <mass
@@ -287,5 +283,5 @@
   </link>
   <joint
-    name="arm_head_joint"
+    name="${name}_arm_head_joint"
     type="fixed">
     <origin
@@ -295,5 +291,5 @@
       link="${name}_lift_link" />
     <child
-      link="arm_head_link" />
+      link="${name}_arm_head_link" />
     <axis
       xyz="0 0 0" />

Commit message: Adapting to new pal sea arm

File: triago_description/robots/triago.urdf.xacro (robot description, xacro)
@@ -27,9 +27,19 @@
   <xacro:arg name="end_effector_head" default="pal-pro-gripper" />
   <xacro:arg name="hand_head_type" default="" />
-  <!-- no-ft-sensor, ati-mini45 -->
-  <xacro:arg name="ft_sensor_left" default="ati-mini45" />
-  <!-- no-ft-sensor, ati-mini45 -->
-  <xacro:arg name="ft_sensor_right" default="ati-mini45" />
+  <!-- straight-wrist, spherical-wrist -->
+  <xacro:arg name="wrist_model_left" default="spherical-wrist" />
+  <!-- straight-wrist, spherical-wrist -->
+  <xacro:arg name="wrist_model_right" default="spherical-wrist" />
+  <xacro:arg name="wrist_model_head" default="spherical-wrist" />
+  <!-- no-ft-sensor, ati -->
+  <xacro:arg name="ft_sensor_left" default="ati" />
+  <!-- no-ft-sensor, ati -->
+  <xacro:arg name="ft_sensor_right" default="ati" />
   <xacro:arg name="ft_sensor_head" default="no-ft-sensor" />
+  <!-- Tool changer-->
+  <xacro:arg name="tool_changer_left" default="true" />
+  <!-- no-ft-sensor, ati -->
+  <xacro:arg name="tool_changer_right" default="true" />
+  <xacro:arg name="tool_changer_head" default="true" />
   <xacro:arg name="use_sim_time" default="false"/>
   <xacro:arg name="is_public_sim" default="false"/>
@@ -56,4 +66,7 @@
   <xacro:property name="ft_sensor_right" value="$(arg ft_sensor_right)" />
   <xacro:property name="ft_sensor_head" value="$(arg ft_sensor_head)" />
+  <xacro:property name="wrist_model_left" value="$(arg wrist_model_left)" />
+  <xacro:property name="wrist_model_right" value="$(arg wrist_model_right)" />
+  <xacro:property name="wrist_model_head" value="$(arg wrist_model_head)" />
   <xacro:property name="description_calibration_dir" value="${arg description_calibration_dir}"/>
   <xacro:property name="is_public_sim" value="$(arg is_public_sim)" />
@@ -63,4 +76,5 @@
   <xacro:property name="end_effector_left_link" value="${'wrist_left_ft_tool_link' if has_ft_sensor_left else 'arm_left_tool_link'}" />
   <xacro:property name="end_effector_left_name" value="gripper_left" />
+  <xacro:property name="tool_changer_left" value="${has_end_effector_left}"/>
   <xacro:property name="has_arm_right" value="${arm_type_right not in ['no-arm']}"/>
   <xacro:property name="has_ft_sensor_right" value="${ft_sensor_right not in ['no-ft-sensor']}"/>
@@ -68,4 +82,5 @@
   <xacro:property name="end_effector_right_link" value="${'wrist_right_ft_tool_link' if has_ft_sensor_right else 'arm_right_tool_link'}" />
   <xacro:property name="end_effector_right_name" value="gripper_right" />
+  <xacro:property name="tool_changer_right" value="${has_end_effector_right}"/>
   <xacro:property name="has_arm_head" value="${arm_type_head not in ['no-arm']}"/>
   <xacro:property name="has_ft_sensor_head" value="${ft_sensor_head not in ['no-ft-sensor']}"/>
@@ -74,4 +89,5 @@
   <xacro:property name="hand_head_type" value="$(arg hand_head_type)" />
   <xacro:property name="end_effector_head_name" value="gripper" />
+  <xacro:property name="tool_changer_head" value="${has_end_effector_head}"/>
   <xacro:if value="${hand_head_type == 'left'}">
     <xacro:property name="head_hand_reflect" value="-1" />
@@ -99,11 +115,11 @@
     <xacro:wrong_end_effector_head />
   </xacro:if>
-  <xacro:if value="${ft_sensor_left not in ['no-ft-sensor', 'ati-mini45']}">
+  <xacro:if value="${ft_sensor_left not in ['no-ft-sensor', 'ati']}">
     <xacro:wrong_ft_sensor_left />
   </xacro:if>
-  <xacro:if value="${ft_sensor_right not in ['no-ft-sensor', 'ati-mini45']}">
+  <xacro:if value="${ft_sensor_right not in ['no-ft-sensor', 'ati']}">
     <xacro:wrong_ft_sensor_right />
   </xacro:if>
-  <xacro:if value="${ft_sensor_head not in ['no-ft-sensor', 'ati-mini45']}">
+  <xacro:if value="${ft_sensor_head not in ['no-ft-sensor', 'ati']}">
     <xacro:wrong_ft_sensor_head />
   </xacro:if>
@@ -127,9 +143,9 @@
   <xacro:if value="${(has_arm_right or has_arm_left or has_arm_head) and (has_end_effector_right or has_end_effector_left or has_end_effector_head)}">
     <xacro:include filename="$(find triago_description)/urdf/end_effector/end_effector.urdf.xacro" />
-    <xacro:include filename="$(find pal_sea_arm_description)/urdf/tool_changer/tool_changer.urdf.xacro" />
   </xacro:if>
   <!-- Force Torque sensor -->
   <xacro:if value="${has_ft_sensor_right or has_ft_sensor_left or has_ft_sensor_head}">
-    <xacro:include filename="$(find pal_sea_arm_description)/urdf/sensors/ft_sensor_ati_mini45.urdf.xacro" />
+    <xacro:include filename="$(find pal_sea_arm_description)/urdf/sensors/ft_sensor/ft_sensor.urdf.xacro" />
+    <xacro:include filename="$(find pal_sea_arm_description)/urdf/sensors/ft_sensor/ft_sensor.gazebo.xacro" />
   </xacro:if>
   <!-- Materials for visualization -->
@@ -145,22 +161,14 @@
   <xacro:if value="${has_arm_left}">
     <!-- Arm -->
-    <xacro:pal_sea_arm name="arm_left" parent="torso_lift_link" arm_type="$(arg arm_type_left)" reflect="1" arm_1_offset="${arm_left_1_joint_offset}" arm_2_offset="${arm_left_2_joint_offset}" arm_3_offset="${arm_left_3_joint_offset}" arm_4_offset="${arm_left_4_joint_offset}" arm_5_offset="${arm_left_5_joint_offset}" arm_6_offset="${arm_left_6_joint_offset}" arm_7_offset="${arm_left_7_joint_offset}">
+    <xacro:pal_sea_arm name="arm_left" parent="torso_lift_link" arm_type="${arm_type_left}" wrist_model="${wrist_model_left}" tool_changer="${tool_changer_left}" reflect="1" arm_1_offset="${arm_left_1_joint_offset}" arm_2_offset="${arm_left_2_joint_offset}" arm_3_offset="${arm_left_3_joint_offset}" arm_4_offset="${arm_left_4_joint_offset}" arm_5_offset="${arm_left_5_joint_offset}" arm_6_offset="${arm_left_6_joint_offset}" arm_7_offset="${arm_left_7_joint_offset}">
       <origin xyz="$(arg arm_x) $(arg arm_y) $(arg arm_z)" rpy="$(arg arm_roll) $(arg arm_pitch) $(arg arm_yaw)"/>
     </xacro:pal_sea_arm>
     <!-- End effector -->
     <xacro:if value="${has_end_effector_left}">
-       <xacro:tool_changer name="tool_changer_left" parent="${end_effector_left_link}">
-         <xacro:if value="${has_ft_sensor_left}">
-              <origin xyz="0.0 0.0 0.0" rpy="0.0 0.0 0.0"/>
-            </xacro:if>
-            <xacro:unless value="${has_ft_sensor_left}">
-              <origin xyz="0.0 0.0 0.0" rpy="${-90.0 * deg_to_rad} ${90.0 * deg_to_rad} ${-90.0 * deg_to_rad}"/>
-            </xacro:unless>
-        </xacro:tool_changer>
-      <xacro:triago_end_effector name="gripper_left" parent="tool_changer_left_tc_tool_link" type="${end_effector_left}" has_end_effector="${has_end_effector_left}" reflect="-1" is_dual="true"/>
+      <xacro:triago_end_effector name="gripper_left" parent="${end_effector_left_link}" type="${end_effector_left}" has_end_effector="${has_end_effector_left}" reflect="-1" is_dual="true"/>
     </xacro:if>
     <!-- FT sensors -->
     <xacro:if value="${has_ft_sensor_left}">
-      <xacro:ft_sensor name="wrist_left" parent="arm_left_tool_link"/>
+      <xacro:ft_sensor type="${ft_sensor_left}" name="wrist_left" parent="arm_left_tool_link"/>
     </xacro:if>
   </xacro:if>
@@ -168,22 +176,14 @@
   <xacro:if value="${has_arm_right}">
     <!-- Arm -->
-    <xacro:pal_sea_arm name="arm_right" parent="torso_lift_link" arm_type="$(arg arm_type_right)" reflect="1" arm_1_offset="${arm_right_1_joint_offset}" arm_2_offset="${arm_right_2_joint_offset}" arm_3_offset="${arm_right_3_joint_offset}" arm_4_offset="${arm_right_4_joint_offset}" arm_5_offset="${arm_right_5_joint_offset}" arm_6_offset="${arm_right_6_joint_offset}" arm_7_offset="${arm_right_7_joint_offset}">
+    <xacro:pal_sea_arm name="arm_right" parent="torso_lift_link" arm_type="${arm_type_right}" wrist_model="${wrist_model_right}" tool_changer="${tool_changer_right}" reflect="1" arm_1_offset="${arm_right_1_joint_offset}" arm_2_offset="${arm_right_2_joint_offset}" arm_3_offset="${arm_right_3_joint_offset}" arm_4_offset="${arm_right_4_joint_offset}" arm_5_offset="${arm_right_5_joint_offset}" arm_6_offset="${arm_right_6_joint_offset}" arm_7_offset="${arm_right_7_joint_offset}">
       <origin xyz="$(arg arm_x) ${-1.0*$(arg arm_y)} $(arg arm_z)" rpy="$(arg arm_roll) ${-1.0*$(arg arm_pitch)} ${-3.14159 -$(arg arm_yaw)}"/>
     </xacro:pal_sea_arm>
     <!-- End effector -->
     <xacro:if value="${has_end_effector_right}">
-       <xacro:tool_changer name="tool_changer_right" parent="${end_effector_right_link}">
-         <xacro:if value="${has_ft_sensor_right}">
-              <origin xyz="0.0 0.0 0.0" rpy="0.0 0.0 ${-180.0 * deg_to_rad}"/>
-            </xacro:if>
-            <xacro:unless value="${has_ft_sensor_right}">
-              <origin xyz="0.0 0.0 0.0" rpy="${-90.0 * deg_to_rad} ${90.0 * deg_to_rad} ${-90.0 * deg_to_rad}"/>
-            </xacro:unless>
-        </xacro:tool_changer>
-      <xacro:triago_end_effector name="gripper_right" parent="tool_changer_right_tc_tool_link" type="${end_effector_right}" has_end_effector="${has_end_effector_right}" reflect="1" is_dual="true"/>
+      <xacro:triago_end_effector name="gripper_right" parent="${end_effector_right_link}" type="${end_effector_right}" has_end_effector="${has_end_effector_right}" reflect="1" is_dual="true"/>
     </xacro:if>
     <!-- FT sensors -->
     <xacro:if value="${has_ft_sensor_right}">
-      <xacro:ft_sensor name="wrist_right" parent="arm_right_tool_link"/>
+      <xacro:ft_sensor type="${ft_sensor_right}" name="wrist_right" parent="arm_right_tool_link"/>
     </xacro:if>
   </xacro:if>
@@ -191,22 +191,14 @@
   <xacro:if value="${has_arm_head}">
     <!-- Arm -->
-    <xacro:pal_sea_arm name="arm_head" parent="torso_lift_link" arm_type="$(arg arm_type_head)" reflect="1" arm_1_offset="${arm_right_1_joint_offset}" arm_2_offset="${arm_right_2_joint_offset}" arm_3_offset="${arm_right_3_joint_offset}" arm_4_offset="${arm_right_4_joint_offset}" arm_5_offset="${arm_right_5_joint_offset}" arm_6_offset="${arm_right_6_joint_offset}" arm_7_offset="${arm_right_7_joint_offset}">
+    <xacro:pal_sea_arm name="arm_head" parent="torso_lift_link" arm_type="${arm_type_head}" wrist_model="${wrist_model_head}" tool_changer="${tool_changer_head}" reflect="1" arm_1_offset="${arm_right_1_joint_offset}" arm_2_offset="${arm_right_2_joint_offset}" arm_3_offset="${arm_right_3_joint_offset}" arm_4_offset="${arm_right_4_joint_offset}" arm_5_offset="${arm_right_5_joint_offset}" arm_6_offset="${arm_right_6_joint_offset}" arm_7_offset="${arm_right_7_joint_offset}">
       <origin xyz="0.00733452377915612 0 0.630632193308821" rpy="0 0.785398163397445 0" />
     </xacro:pal_sea_arm>
     <!-- End effector -->
     <xacro:if value="${has_end_effector_head}">
-       <xacro:tool_changer name="tool_changer_head" parent="${end_effector_head_link}">
-         <xacro:if value="${has_ft_sensor_head}">
-              <origin xyz="0.0 0.0 0.0" rpy="0.0 0.0 0.0"/>
-         </xacro:if>
-         <xacro:unless value="${has_ft_sensor_head}">
-              <origin xyz="0.0 0.0 0.0" rpy="${-90.0 * deg_to_rad} ${90.0 * deg_to_rad} ${-90.0 * deg_to_rad}"/>
-         </xacro:unless>
-        </xacro:tool_changer>
-      <xacro:triago_end_effector name="gripper_head" parent="tool_changer_head_tc_tool_link" type="${end_effector_head}" has_end_effector="${has_end_effector_head}" reflect="${head_hand_reflect}" is_dual="true"/>
+      <xacro:triago_end_effector name="gripper_head" parent="${end_effector_head_link}" type="${end_effector_head}" has_end_effector="${has_end_effector_head}" reflect="${head_hand_reflect}" is_dual="true"/>
     </xacro:if>
     <!-- FT sensors -->
     <xacro:if value="${has_ft_sensor_head}">
-      <xacro:ft_sensor name="wrist_head" parent="arm_head_tool_link"/>
+      <xacro:ft_sensor type="${ft_sensor_left}" name="wrist_head" parent="arm_head_tool_link"/>
     </xacro:if>
   </xacro:if>

File: triago_description/ros2_control/ros2_control.urdf.xacro (robot description, xacro)
@@ -88,5 +88,5 @@
         <xacro:ros2_control_arm name="arm_left_7" reduction="1.0" offset_value="${arm_left_7_joint_offset}" />
         <xacro:if value="${has_ft_sensor_left}">
-          <xacro:include filename="$(find pal_sea_arm_description)/urdf/sensors/sensors.ros2_control.xacro"/>
+          <xacro:include filename="$(find pal_sea_arm_description)/urdf/sensors/ft_sensor/sensor.ros2_control.xacro"/>
           <xacro:ros2_control_force_torque_sensor name="wrist_left_sensor"/>
         </xacro:if>
@@ -109,5 +109,5 @@
         <xacro:ros2_control_arm name="arm_right_7" reduction="1.0" offset_value="${arm_right_7_joint_offset}" />
         <xacro:if value="${has_ft_sensor_right}">
-          <xacro:include filename="$(find pal_sea_arm_description)/urdf/sensors/sensors.ros2_control.xacro"/>
+          <xacro:include filename="$(find pal_sea_arm_description)/urdf/sensors/ft_sensor/sensor.ros2_control.xacro"/>
           <xacro:ros2_control_force_torque_sensor name="wrist_right_sensor"/>
         </xacro:if>
@@ -130,6 +130,6 @@
         <xacro:ros2_control_arm name="arm_head_6" reduction="1.0" offset_value="${arm_left_6_joint_offset}" />
         <xacro:ros2_control_arm name="arm_head_7" reduction="1.0" offset_value="${arm_left_7_joint_offset}" />
-        <xacro:if value="${has_ft_sensor_left}">
-          <xacro:include filename="$(find pal_sea_arm_description)/urdf/sensors/sensors.ros2_control.xacro"/>
+        <xacro:if value="${has_ft_sensor_head}">
+          <xacro:include filename="$(find pal_sea_arm_description)/urdf/sensors/ft_sensor/sensor.ros2_control.xacro"/>
           <xacro:ros2_control_force_torque_sensor name="wrist_head_sensor"/>
         </xacro:if>
