Commit message: Adapting to the arm!

File: triago_description/robots/triago.urdf.xacro (robot description, xacro)
@@ -137,6 +137,9 @@
   <xacro:include filename="$(arg description_calibration_dir)/calibration_constants.urdf.xacro" />
   <!-- Arm -->
-  <xacro:if value="${has_arm_right or has_arm_left or has_arm_head}">
+  <xacro:if value="${has_arm_right or has_arm_left }">
     <xacro:include filename="$(find pal_sea_arm_description)/urdf/arm/arm.urdf.xacro" />
+  </xacro:if>
+  <xacro:if value="${has_arm_head}">
+    <xacro:include filename="$(find triago_description)/urdf/head_arm/arm.urdf.xacro" />
   </xacro:if>
   <!-- End effector -->
@@ -161,5 +164,5 @@
   <xacro:if value="${has_arm_left}">
     <!-- Arm -->
-    <xacro:pal_sea_arm name="arm_left" parent="torso_lift_link" arm_type="${arm_type_left}" wrist_model="${wrist_model_left}" tool_changer="${tool_changer_left}" reflect="1" arm_1_offset="${arm_left_1_joint_offset}" arm_2_offset="${arm_left_2_joint_offset}" arm_3_offset="${arm_left_3_joint_offset}" arm_4_offset="${arm_left_4_joint_offset}" arm_5_offset="${arm_left_5_joint_offset}" arm_6_offset="${arm_left_6_joint_offset}" arm_7_offset="${arm_left_7_joint_offset}">
+    <xacro:pal_sea_arm name="arm_left" parent="torso_lift_link" arm_type="${arm_type_left}" wrist_model="${wrist_model_left}" tool_changer="${tool_changer_left}" reflect="1" first_joint_reflect="-1" arm_1_offset="${arm_left_1_joint_offset}" arm_2_offset="${arm_left_2_joint_offset}" arm_3_offset="${arm_left_3_joint_offset}" arm_4_offset="${arm_left_4_joint_offset}" arm_5_offset="${arm_left_5_joint_offset}" arm_6_offset="${arm_left_6_joint_offset}" arm_7_offset="${arm_left_7_joint_offset}">
       <origin xyz="$(arg arm_x) $(arg arm_y) $(arg arm_z)" rpy="$(arg arm_roll) $(arg arm_pitch) $(arg arm_yaw)"/>
     </xacro:pal_sea_arm>
@@ -176,5 +179,5 @@
   <xacro:if value="${has_arm_right}">
     <!-- Arm -->
-    <xacro:pal_sea_arm name="arm_right" parent="torso_lift_link" arm_type="${arm_type_right}" wrist_model="${wrist_model_right}" tool_changer="${tool_changer_right}" reflect="1" arm_1_offset="${arm_right_1_joint_offset}" arm_2_offset="${arm_right_2_joint_offset}" arm_3_offset="${arm_right_3_joint_offset}" arm_4_offset="${arm_right_4_joint_offset}" arm_5_offset="${arm_right_5_joint_offset}" arm_6_offset="${arm_right_6_joint_offset}" arm_7_offset="${arm_right_7_joint_offset}">
+    <xacro:pal_sea_arm name="arm_right" parent="torso_lift_link" arm_type="${arm_type_right}" wrist_model="${wrist_model_right}" tool_changer="${tool_changer_right}" reflect="1" first_joint_reflect="1" arm_1_offset="${arm_right_1_joint_offset}" arm_2_offset="${arm_right_2_joint_offset}" arm_3_offset="${arm_right_3_joint_offset}" arm_4_offset="${arm_right_4_joint_offset}" arm_5_offset="${arm_right_5_joint_offset}" arm_6_offset="${arm_right_6_joint_offset}" arm_7_offset="${arm_right_7_joint_offset}">
       <origin xyz="$(arg arm_x) ${-1.0*$(arg arm_y)} $(arg arm_z)" rpy="$(arg arm_roll) ${-1.0*$(arg arm_pitch)} ${-3.14159 -$(arg arm_yaw)}"/>
     </xacro:pal_sea_arm>
@@ -191,7 +194,7 @@
   <xacro:if value="${has_arm_head}">
     <!-- Arm -->
-    <xacro:pal_sea_arm name="arm_head" parent="torso_lift_link" arm_type="${arm_type_head}" wrist_model="${wrist_model_head}" tool_changer="${tool_changer_head}" reflect="1" arm_1_offset="${arm_right_1_joint_offset}" arm_2_offset="${arm_right_2_joint_offset}" arm_3_offset="${arm_right_3_joint_offset}" arm_4_offset="${arm_right_4_joint_offset}" arm_5_offset="${arm_right_5_joint_offset}" arm_6_offset="${arm_right_6_joint_offset}" arm_7_offset="${arm_right_7_joint_offset}">
+    <xacro:head_arm name="arm_head" parent="torso_lift_link" wrist_model="${wrist_model_head}" tool_changer="${tool_changer_head}" reflect="1" arm_1_offset="${arm_right_1_joint_offset}" arm_2_offset="${arm_right_2_joint_offset}" arm_3_offset="${arm_right_3_joint_offset}" arm_4_offset="${arm_right_4_joint_offset}" arm_5_offset="${arm_right_5_joint_offset}" arm_6_offset="${arm_right_6_joint_offset}" arm_7_offset="${arm_right_7_joint_offset}">
       <origin xyz="0.00733452377915612 0 0.630632193308821" rpy="0 0.785398163397445 0" />
-    </xacro:pal_sea_arm>
+    </xacro:head_arm>
     <!-- End effector -->
     <xacro:if value="${has_end_effector_head}">

File: triago_description/urdf/torso/torso_dual.urdf.xacro (robot description, xacro)
@@ -125,10 +125,16 @@
     <collision>
       <origin
-        xyz="0 0 0"
-        rpy="0 0 0" />
-      <geometry>
-        <mesh
-          filename="package://triago_description/meshes/torso/torso_lift_link.STL" />
-      </geometry>
+        xyz="0.0 0.0 0.5545"
+        rpy="0 0 0" />
+      <geometry>
+        <mesh
+          filename="package://triago_description/meshes/torso/torso_lift_link_collision.stl" />
+      </geometry>
+    </collision>
+    <collision>
+          <origin xyz="-0.226436438571948 3.12797385809451E-05 0.55984038105676683" rpy="0 0 -1.5707963267949" />
+          <geometry>
+            <mesh filename="package://triago_description/meshes/torso/laptop_tray_collision.stl" />
+          </geometry>
     </collision>
   </link>
@@ -176,5 +182,5 @@
       <geometry>
         <mesh
-          filename="package://triago_description/meshes/torso/arm_left_link.STL" />
+          filename="package://triago_description/meshes/torso/arm_left_link_collision.stl" />
       </geometry>
     </collision>
@@ -227,5 +233,5 @@
       <geometry>
         <mesh
-          filename="package://triago_description/meshes/torso/arm_right_link.STL" />
+          filename="package://triago_description/meshes/torso/arm_right_link_collision.stl" />
       </geometry>
     </collision>

Commit message: Adjus tool_changer

File: triago_description/robots/triago.urdf.xacro (robot description, xacro)
@@ -76,5 +76,5 @@
   <xacro:property name="end_effector_left_link" value="${'wrist_left_ft_tool_link' if has_ft_sensor_left else 'arm_left_tool_link'}" />
   <xacro:property name="end_effector_left_name" value="gripper_left" />
-  <xacro:property name="tool_changer_left" value="${has_end_effector_left}"/>
+  <xacro:property name="tool_changer_left" value="${has_end_effector_left || has_ft_sensor_left}"/>
   <xacro:property name="has_arm_right" value="${arm_type_right not in ['no-arm']}"/>
   <xacro:property name="has_ft_sensor_right" value="${ft_sensor_right not in ['no-ft-sensor']}"/>
@@ -82,5 +82,5 @@
   <xacro:property name="end_effector_right_link" value="${'wrist_right_ft_tool_link' if has_ft_sensor_right else 'arm_right_tool_link'}" />
   <xacro:property name="end_effector_right_name" value="gripper_right" />
-  <xacro:property name="tool_changer_right" value="${has_end_effector_right}"/>
+  <xacro:property name="tool_changer_right" value="${has_end_effector_right || has_ft_sensor_right }"/>
   <xacro:property name="has_arm_head" value="${arm_type_head not in ['no-arm']}"/>
   <xacro:property name="has_ft_sensor_head" value="${ft_sensor_head not in ['no-ft-sensor']}"/>
@@ -89,5 +89,5 @@
   <xacro:property name="hand_head_type" value="$(arg hand_head_type)" />
   <xacro:property name="end_effector_head_name" value="gripper" />
-  <xacro:property name="tool_changer_head" value="${has_end_effector_head}"/>
+  <xacro:property name="tool_changer_head" value="${has_end_effector_head || has_ft_sensor_head}"/>
   <xacro:if value="${hand_head_type == 'left'}">
     <xacro:property name="head_hand_reflect" value="-1" />

Commit message: Adjus tool_changer

File: triago_description/robots/triago.urdf.xacro (robot description, xacro)
@@ -76,5 +76,5 @@
   <xacro:property name="end_effector_left_link" value="${'wrist_left_ft_tool_link' if has_ft_sensor_left else 'arm_left_tool_link'}" />
   <xacro:property name="end_effector_left_name" value="gripper_left" />
-  <xacro:property name="tool_changer_left" value="${has_end_effector_left || has_ft_sensor_left}"/>
+  <xacro:property name="tool_changer_left" value="${has_end_effector_left or has_ft_sensor_left}"/>
   <xacro:property name="has_arm_right" value="${arm_type_right not in ['no-arm']}"/>
   <xacro:property name="has_ft_sensor_right" value="${ft_sensor_right not in ['no-ft-sensor']}"/>
@@ -82,5 +82,5 @@
   <xacro:property name="end_effector_right_link" value="${'wrist_right_ft_tool_link' if has_ft_sensor_right else 'arm_right_tool_link'}" />
   <xacro:property name="end_effector_right_name" value="gripper_right" />
-  <xacro:property name="tool_changer_right" value="${has_end_effector_right || has_ft_sensor_right }"/>
+  <xacro:property name="tool_changer_right" value="${has_end_effector_right or has_ft_sensor_right }"/>
   <xacro:property name="has_arm_head" value="${arm_type_head not in ['no-arm']}"/>
   <xacro:property name="has_ft_sensor_head" value="${ft_sensor_head not in ['no-ft-sensor']}"/>
@@ -89,5 +89,5 @@
   <xacro:property name="hand_head_type" value="$(arg hand_head_type)" />
   <xacro:property name="end_effector_head_name" value="gripper" />
-  <xacro:property name="tool_changer_head" value="${has_end_effector_head || has_ft_sensor_head}"/>
+  <xacro:property name="tool_changer_head" value="${has_end_effector_head or has_ft_sensor_head}"/>
   <xacro:if value="${hand_head_type == 'left'}">
     <xacro:property name="head_hand_reflect" value="-1" />

Commit message: Flip 1st joint for the head + adapt motions

File: triago_description/robots/triago.urdf.xacro (robot description, xacro)
@@ -195,5 +195,5 @@
     <!-- Arm -->
     <xacro:head_arm name="arm_head" parent="torso_lift_link" wrist_model="${wrist_model_head}" tool_changer="${tool_changer_head}" reflect="1" arm_1_offset="${arm_right_1_joint_offset}" arm_2_offset="${arm_right_2_joint_offset}" arm_3_offset="${arm_right_3_joint_offset}" arm_4_offset="${arm_right_4_joint_offset}" arm_5_offset="${arm_right_5_joint_offset}" arm_6_offset="${arm_right_6_joint_offset}" arm_7_offset="${arm_right_7_joint_offset}">
-      <origin xyz="0.00733452377915612 0 0.630632193308821" rpy="0 0.785398163397445 0" />
+      <origin xyz="0.00733452377915612 0 0.630632193308821" rpy="0 -0.785398163397445 3.14" />
     </xacro:head_arm>
     <!-- End effector -->

Commit message: Add camera position as an argument

File: triago_description/robots/triago.urdf.xacro (robot description, xacro)
@@ -25,5 +25,5 @@
   <!-- pal-pro-gripper, custom-->
   <xacro:arg name="end_effector_right" default="allegro-hand" />
-  <xacro:arg name="end_effector_head" default="no-end-effector" />
+  <xacro:arg name="end_effector_head" default="camera-tools" />
   <xacro:arg name="hand_head_type" default="" />
   <!-- straight-wrist, spherical-wrist -->
@@ -53,4 +53,5 @@
   <xacro:arg name="arm_pitch" default="0.0" />
   <xacro:arg name="arm_yaw" default="-1.2217" />
+  <xacro:arg name="camera_position" default="down" />
   <!-- PROPERTIES -->
   <xacro:property name="use_sim_time" value="$(arg use_sim_time)" />
@@ -71,6 +72,7 @@
   <xacro:property name="description_calibration_dir" value="${arg description_calibration_dir}"/>
   <xacro:property name="is_public_sim" value="$(arg is_public_sim)" />
+  <xacro:property name="camera_position" value="$(arg camera_position)"/>
   <xacro:property name="has_arm_left" value="${arm_type_left not in ['no-arm']}"/>
-  <xacro:property name="has_ft_sensor_left" value="${ft_sensor_left not in ['no-ft-sensor']}"/>
+  <xacro:property name="has_ft_sensor_left" value="${ft_sensor_left not in ['no-ft-sensor'] and end_effector_left not in ['camera-tools']}"/>
   <xacro:property name="has_end_effector_left" value="${end_effector_left not in ['no-end-effector']}" />
   <xacro:property name="end_effector_left_link" value="${'wrist_left_ft_tool_link' if has_ft_sensor_left else 'arm_left_tool_link'}" />
@@ -78,5 +80,5 @@
   <xacro:property name="tool_changer_left" value="${has_end_effector_left or has_ft_sensor_left}"/>
   <xacro:property name="has_arm_right" value="${arm_type_right not in ['no-arm']}"/>
-  <xacro:property name="has_ft_sensor_right" value="${ft_sensor_right not in ['no-ft-sensor']}"/>
+  <xacro:property name="has_ft_sensor_right" value="${ft_sensor_right not in ['no-ft-sensor'] and end_effector_right not in ['camera-tools']}"/>
   <xacro:property name="has_end_effector_right" value="${end_effector_right not in ['no-end-effector']}" />
   <xacro:property name="end_effector_right_link" value="${'wrist_right_ft_tool_link' if has_ft_sensor_right else 'arm_right_tool_link'}" />
@@ -84,5 +86,5 @@
   <xacro:property name="tool_changer_right" value="${has_end_effector_right or has_ft_sensor_right }"/>
   <xacro:property name="has_arm_head" value="${arm_type_head not in ['no-arm']}"/>
-  <xacro:property name="has_ft_sensor_head" value="${ft_sensor_head not in ['no-ft-sensor']}"/>
+  <xacro:property name="has_ft_sensor_head" value="${ft_sensor_head not in ['no-ft-sensor'] and end_effector_head not in ['camera-tools']}"/>
   <xacro:property name="has_end_effector_head" value="${end_effector_head not in ['no-end-effector']}" />
   <xacro:property name="end_effector_head_link" value="${'wrist_head_ft_tool_link' if has_ft_sensor_head else 'arm_head_tool_link'}" />
@@ -106,11 +108,11 @@
     <xacro:wrong_arm_type_head />
   </xacro:if>
-  <xacro:if value="${end_effector_left not in ['pal-pro-gripper', 'custom', 'allegro-hand', 'no-end-effector']}">
+  <xacro:if value="${end_effector_left not in ['pal-pro-gripper', 'custom', 'allegro-hand', 'no-end-effector', 'camera-tools']}">
     <xacro:wrong_end_effector_left />
   </xacro:if>
-  <xacro:if value="${end_effector_right not in ['pal-pro-gripper', 'custom', 'allegro-hand', 'no-end-effector']}">
+  <xacro:if value="${end_effector_right not in ['pal-pro-gripper', 'custom', 'allegro-hand', 'no-end-effector', 'camera-tools']}">
     <xacro:wrong_end_effector_right />
   </xacro:if>
-  <xacro:if value="${end_effector_head not in ['pal-pro-gripper', 'custom', 'allegro-hand', 'no-end-effector']}">
+  <xacro:if value="${end_effector_head not in ['pal-pro-gripper', 'custom', 'allegro-hand', 'no-end-effector', 'camera-tools']}">
     <xacro:wrong_end_effector_head />
   </xacro:if>
@@ -169,5 +171,5 @@
     <!-- End effector -->
     <xacro:if value="${has_end_effector_left}">
-      <xacro:triago_end_effector name="gripper_left" parent="${end_effector_left_link}" type="${end_effector_left}" has_end_effector="${has_end_effector_left}" reflect="-1" is_dual="true"/>
+      <xacro:triago_end_effector name="gripper_left" parent="${end_effector_left_link}" type="${end_effector_left}" has_end_effector="${has_end_effector_left}" reflect="-1" is_dual="true" camera_position="${camera_position}"/>
     </xacro:if>
     <!-- FT sensors -->
@@ -184,5 +186,5 @@
     <!-- End effector -->
     <xacro:if value="${has_end_effector_right}">
-      <xacro:triago_end_effector name="gripper_right" parent="${end_effector_right_link}" type="${end_effector_right}" has_end_effector="${has_end_effector_right}" reflect="1" is_dual="true"/>
+      <xacro:triago_end_effector name="gripper_right" parent="${end_effector_right_link}" type="${end_effector_right}" has_end_effector="${has_end_effector_right}" reflect="1" is_dual="true" camera_position="${camera_position}"/>
     </xacro:if>
     <!-- FT sensors -->
@@ -199,5 +201,5 @@
     <!-- End effector -->
     <xacro:if value="${has_end_effector_head}">
-      <xacro:triago_end_effector name="gripper_head" parent="${end_effector_head_link}" type="${end_effector_head}" has_end_effector="${has_end_effector_head}" reflect="${head_hand_reflect}" is_dual="true"/>
+      <xacro:triago_end_effector name="gripper_head" parent="${end_effector_head_link}" type="${end_effector_head}" has_end_effector="${has_end_effector_head}" reflect="${head_hand_reflect}" is_dual="true" camera_position="${camera_position}"/>
     </xacro:if>
     <!-- FT sensors -->

File: triago_description/urdf/end_effector/end_effector.urdf.xacro (robot description, xacro)
@@ -20,5 +20,5 @@
     - reflect: Set to 1 for a right end effector, or to -1 for a left end effector
   -->
-  <xacro:macro name="triago_end_effector" params="name parent type has_end_effector reflect is_dual:=false">
+  <xacro:macro name="triago_end_effector" params="name parent type has_end_effector reflect is_dual:=false camera_position">
   <!-- No end-effector -->
   <xacro:if value="${not has_end_effector}">
@@ -106,4 +106,44 @@
     </xacro:allegro_hand>
   </xacro:if>
+  <!--Camera-->
+  <xacro:if value="${type == 'camera-tools'}">
+    <link name="${name}_camera_link">
+      <inertial>
+        <origin xyz="-7.7517E-05 -0.00017089 0.003965" rpy="0 0 0"/>
+        <mass
+          value="0.073091" />
+        <inertia
+          ixx="2.656E-05" ixy="-2.4789E-08" ixz="-2.1125E-07"
+          iyy="1.3652E-05" iyz="-2.6011E-09"
+          izz="1.8641E-05" />
+      </inertial>
+      <visual>
+      <origin xyz="0 0 0" rpy="0 0 0" />
+        <geometry>
+          <mesh filename="package://pal_sea_arm_description/meshes/arm_tiago_pro/camera_link.STL" />
+        </geometry>
+        <material name="">
+          <color rgba="0.75294 0.75294 0.75294 1" />
+        </material>
+      </visual>
+      <collision>
+        <origin xyz="0 0 0" rpy="0 0 0" />
+        <geometry>
+          <mesh filename="package://pal_sea_arm_description/meshes/arm_tiago_pro/camera_link.STL" />
+        </geometry>
+      </collision>
+    </link>
+    <joint name="${name}_camera_joint" type="fixed">
+      <xacro:if value="${camera_position == 'up'}">
+        <origin xyz="0.0406 0 -0.003" rpy="3.1416 -1.5708 0" />
+      </xacro:if>
+      <xacro:if value="${camera_position == 'down'}">
+        <origin xyz="-0.0406 0 -0.003" rpy="0 -1.5708 0" />
+      </xacro:if>
+      <parent link="${parent}" />
+      <child link="${name}_camera_link" />
+      <axis xyz="0 0 0" />
+    </joint>
+  </xacro:if>
   </xacro:macro>
 </robot>

Commit message: Add posibility of having 3 cameras at the same time

File: triago_description/robots/triago.urdf.xacro (robot description, xacro)
@@ -53,5 +53,7 @@
   <xacro:arg name="arm_pitch" default="0.0" />
   <xacro:arg name="arm_yaw" default="-1.2217" />
-  <xacro:arg name="camera_position" default="down" />
+  <xacro:arg name="camera_position_right" default="up" />
+  <xacro:arg name="camera_position_left" default="up" />
+  <xacro:arg name="camera_position_head" default="down" />
   <!-- PROPERTIES -->
   <xacro:property name="use_sim_time" value="$(arg use_sim_time)" />
@@ -72,5 +74,7 @@
   <xacro:property name="description_calibration_dir" value="${arg description_calibration_dir}"/>
   <xacro:property name="is_public_sim" value="$(arg is_public_sim)" />
-  <xacro:property name="camera_position" value="$(arg camera_position)"/>
+  <xacro:property name="camera_position_right" value="$(arg camera_position_right)"/>
+  <xacro:property name="camera_position_left" value="$(arg camera_position_left)"/>
+  <xacro:property name="camera_position_head" value="$(arg camera_position_head)"/>
   <xacro:property name="has_arm_left" value="${arm_type_left not in ['no-arm']}"/>
   <xacro:property name="has_ft_sensor_left" value="${ft_sensor_left not in ['no-ft-sensor'] and end_effector_left not in ['camera-tools']}"/>
@@ -171,5 +175,5 @@
     <!-- End effector -->
     <xacro:if value="${has_end_effector_left}">
-      <xacro:triago_end_effector name="gripper_left" parent="${end_effector_left_link}" type="${end_effector_left}" has_end_effector="${has_end_effector_left}" reflect="-1" is_dual="true" camera_position="${camera_position}"/>
+      <xacro:triago_end_effector name="gripper_left" parent="${end_effector_left_link}" type="${end_effector_left}" has_end_effector="${has_end_effector_left}" reflect="-1" is_dual="true" camera_position="${camera_position_left}"/>
     </xacro:if>
     <!-- FT sensors -->
@@ -186,5 +190,5 @@
     <!-- End effector -->
     <xacro:if value="${has_end_effector_right}">
-      <xacro:triago_end_effector name="gripper_right" parent="${end_effector_right_link}" type="${end_effector_right}" has_end_effector="${has_end_effector_right}" reflect="1" is_dual="true" camera_position="${camera_position}"/>
+      <xacro:triago_end_effector name="gripper_right" parent="${end_effector_right_link}" type="${end_effector_right}" has_end_effector="${has_end_effector_right}" reflect="1" is_dual="true" camera_position="${camera_position_right}"/>
     </xacro:if>
     <!-- FT sensors -->
@@ -201,5 +205,5 @@
     <!-- End effector -->
     <xacro:if value="${has_end_effector_head}">
-      <xacro:triago_end_effector name="gripper_head" parent="${end_effector_head_link}" type="${end_effector_head}" has_end_effector="${has_end_effector_head}" reflect="${head_hand_reflect}" is_dual="true" camera_position="${camera_position}"/>
+      <xacro:triago_end_effector name="gripper_head" parent="${end_effector_head_link}" type="${end_effector_head}" has_end_effector="${has_end_effector_head}" reflect="${head_hand_reflect}" is_dual="true" camera_position="${camera_position_head}"/>
     </xacro:if>
     <!-- FT sensors -->
