Commit message: Add simplify models + remove unecessary models

File: triago_description/robots/triago.urdf.xacro (robot description, xacro)
@@ -27,7 +27,7 @@
   <xacro:arg name="end_effector_head" default="camera-tools" />
   <xacro:arg name="hand_head_type" default="" />
-  <!-- straight-wrist, spherical-wrist -->
+  <!-- spherical-wrist -->
   <xacro:arg name="wrist_model_left" default="spherical-wrist" />
-  <!-- straight-wrist, spherical-wrist -->
+  <!-- spherical-wrist -->
   <xacro:arg name="wrist_model_right" default="spherical-wrist" />
   <xacro:arg name="wrist_model_head" default="spherical-wrist" />

File: triago_description/urdf/head_arm/arm.urdf.xacro (robot description, xacro)
@@ -220,20 +220,5 @@
     <!-- With tool changer (the tool link is the tool changer)-->
     <xacro:if value="${tool_changer}">
-      <link name="${name}_tool_link">
-        <xacro:inertial_tool_changer_link reflect="${reflect}"/>
-        <visual>
-          <origin xyz="0 0 0" rpy="0 0 0" />
-          <geometry>
-            <mesh filename="package://pal_sea_arm_description/meshes/${mesh_folder}/tool_changer_link.stl" scale="1 1 ${reflect}" />
-          </geometry>
-          <material name="pal/DarkGrey"/>
-        </visual>
-        <collision>
-          <origin xyz="0 0 0" rpy="0 0 0" />
-          <geometry>
-            <mesh filename="package://pal_sea_arm_description/meshes/${mesh_folder}/tool_changer_link_collision.stl" scale="1 1 ${reflect}" />
-          </geometry>
-        </collision>
-      </link>
+      <link name="${name}_tool_link"/>
       <joint name="${name}_tool_joint" type="fixed">
         <parent link="${name}_7_link" />

File: triago_description/urdf/head_arm/arm_properties/arm.properties.xacro (robot description, xacro)
@@ -50,14 +50,5 @@
         <origin xyz="-0.0199999999999971 0.17011 -0.037110000000002" rpy="-1.5707963267949 0 0" />
     </xacro:macro>
-    <!-- Tool changer (can be present in both wrists)-->
-    <xacro:macro name="inertial_tool_changer_link" params="reflect">
-        <inertial>
-            <origin xyz="0.003414871500006 0.002458561521477 -0.001077004696741" rpy="0 0 0" />
-            <mass value="0.0655061851536" />
-            <inertia ixx="1.79461992752602E-05" ixy="1.70670100210845E-06" ixz="-2.54814948767968E-09" iyy="1.47274432150498E-05" iyz="1.09471559381518E-07" izz="3.12924968277541E-05" />
-        </inertial>
-    </xacro:macro>
     <xacro:macro name="origin_joint_tool_changer" params="reflect">
-        <!-- @Lucien needs to fix -->
         <origin xyz="0 0 0.017" rpy="0 0 0" />
     </xacro:macro>

File: triago_description/urdf/head_arm/arm_properties/spherical-wrist.properties.xacro (robot description, xacro)
@@ -23,7 +23,7 @@
     <xacro:macro name="inertial_link_7" params="reflect">
         <inertial>
-            <origin xyz="0.00095120830852 -0.000268585760924 1.45881142001869E-05" rpy="0 0 0" />
-            <mass value="0.057209493908896" />
-            <inertia ixx="3.32348045580924E-05" ixy="8.53056519363846E-07" ixz="-2.89819873727239E-07" iyy="3.34386146857115E-05" iyz="8.77813050093602E-08" izz="6.16426730349172E-05" />
+            <origin xyz="0.00174 -0.00223 0.0083" rpy="0 0 0" />
+            <mass value="0.12399" />
+            <inertia ixx="0.00008" ixy="0.0" ixz="0.0" iyy="0.00006" iyz="0.0" izz="0.00012" />
         </inertial>
     </xacro:macro>

File: triago_description/urdf/torso/torso_dual.urdf.xacro (robot description, xacro)
@@ -30,5 +30,5 @@
       <geometry>
         <mesh
-          filename="package://triago_description/meshes/torso/torso_fixed.STL" />
+          filename="package://triago_description/meshes/torso/torso_fixed.stl" />
       </geometry>
       <material
@@ -44,5 +44,5 @@
       <geometry>
         <mesh
-          filename="package://triago_description/meshes/torso/torso_fixed.STL" />
+          filename="package://triago_description/meshes/torso/torso_fixed_collision.stl" />
       </geometry>
     </collision>
@@ -59,11 +59,4 @@
   <!-- Middle extending  -->
   <link name="${name}_fixed_column_link">
-    <inertial>
-      <origin rpy="0 0 0" xyz="0 0 0" />
-      <mass value="0.01" />
-      <inertia ixx="0.000001" ixy="0" ixz="0"
-               iyy="0.000001" iyz="0"
-               izz="0.000001" />
-    </inertial>
     <visual>
       <origin rpy="0 0 0" xyz="0 0 0.275" />
@@ -73,11 +66,4 @@
       <material name="pal/DarkGrey"/>
     </visual>
-    <collision>
-      <origin rpy="0 0 0" xyz="0 0 0.275" />
-      <geometry>
-        <box size="0.23 0.253 0.45"/>
-      </geometry>
-      <material name="pal/DarkGrey"/>
-    </collision>
   </link>
   <gazebo reference="${name}_fixed_column_link">
@@ -90,8 +76,7 @@
     <axis xyz="0 0 0" />
   </joint>
-  <link
-    name="${name}_lift_link">
+  <link name="${name}_lift_link">
      <inertial>
-      <origin xyz="0 0 0" rpy="0 0 0" />
+      <origin xyz="0 0 0.5545" rpy="0 0 0" />
         <mass value="3.24266045177967" />
         <inertia ixx="0.0295369723560087" ixy="-7.85101789883696E-07" ixz="-8.58576921315497E-05" iyy="0.0170989395656347" iyz="-8.17944373020342E-06" izz="0.0290055792681799" />
@@ -103,5 +88,5 @@
       <geometry>
         <mesh
-          filename="package://triago_description/meshes/torso/torso_lift_link.STL" />
+          filename="package://triago_description/meshes/torso/torso_lift_link.stl" />
       </geometry>
       <material
@@ -113,5 +98,5 @@
     <collision>
       <origin
-        xyz="0.0 0.0 0.5545"
+        xyz="0.0 0.0 0.0"
         rpy="0 0 0" />
       <geometry>
@@ -134,44 +119,5 @@
     <limit effort="0" lower="0" upper="0.34" velocity="${torso_max_vel}" />
   </joint>
-  <link
-    name="${name}_arm_left_link">
-    <inertial>
-      <origin
-        xyz="0 0 0"
-        rpy="0 0 0" />
-      <mass
-        value="0.23047" />
-      <inertia
-        ixx="0.00026511"
-        ixy="1.3047E-06"
-        ixz="7.8189E-05"
-        iyy="0.00035859"
-        iyz="-5.3396E-05"
-        izz="0.00040319" />
-    </inertial>
-    <visual>
-      <origin
-        xyz="0 0 0"
-        rpy="0 0 0" />
-      <geometry>
-        <mesh
-          filename="package://triago_description/meshes/torso/arm_left_link.STL" />
-      </geometry>
-      <material
-        name="">
-        <color
-          rgba="0.25098 0.25098 0.25098 1" />
-      </material>
-    </visual>
-    <collision>
-      <origin
-        xyz="0 0 0"
-        rpy="0 0 0" />
-      <geometry>
-        <mesh
-          filename="package://triago_description/meshes/torso/arm_left_link_collision.stl" />
-      </geometry>
-    </collision>
-  </link>
+  <link name="${name}_arm_left_link"/>
   <joint
     name="${name}_arm_left_joint"
@@ -185,44 +131,5 @@
       xyz="0 0 0" />
   </joint>
- <link
-    name="${name}_arm_right_link">
-    <inertial>
-      <origin
-        xyz="0 0 0"
-        rpy="0 0 0" />
-      <mass
-        value="0.23047" />
-      <inertia
-        ixx="0.00026509"
-        ixy="-3.1836E-07"
-        ixz="-7.8741E-05"
-        iyy="0.00035861"
-        iyz="-5.257E-05"
-        izz="0.00040319" />
-    </inertial>
-    <visual>
-      <origin
-        xyz="0 0 0"
-        rpy="0 0 0" />
-      <geometry>
-        <mesh
-          filename="package://triago_description/meshes/torso/arm_right_link.STL" />
-      </geometry>
-      <material
-        name="">
-        <color
-          rgba="0.25098 0.25098 0.25098 1" />
-      </material>
-    </visual>
-    <collision>
-      <origin
-        xyz="0 0 0"
-        rpy="0 0 0" />
-      <geometry>
-        <mesh
-          filename="package://triago_description/meshes/torso/arm_right_link_collision.stl" />
-      </geometry>
-    </collision>
-  </link>
+ <link name="${name}_arm_right_link"/>
   <joint
     name="${name}_arm_right_joint"
@@ -236,44 +143,5 @@
       xyz="0 0 0" />
   </joint>
- <link
-    name="${name}_arm_head_link">
-    <inertial>
-      <origin
-        xyz="0 0 0"
-        rpy="0 0 0" />
-      <mass
-        value="0.18229" />
-      <inertia
-        ixx="0.00027537"
-        ixy="7.4919E-10"
-        ixz="7.2758E-06"
-        iyy="0.00018169"
-        iyz="-2.2164E-10"
-        izz="0.00037953" />
-    </inertial>
-    <visual>
-      <origin
-        xyz="0 0 0"
-        rpy="0 0 0" />
-      <geometry>
-        <mesh
-          filename="package://triago_description/meshes/torso/arm_head_link.STL" />
-      </geometry>
-      <material
-        name="">
-        <color
-          rgba="0.25098 0.25098 0.25098 1" />
-      </material>
-    </visual>
-    <collision>
-      <origin
-        xyz="0 0 0"
-        rpy="0 0 0" />
-      <geometry>
-        <mesh
-          filename="package://triago_description/meshes/torso/arm_head_link.STL" />
-      </geometry>
-    </collision>
-  </link>
+ <link name="${name}_arm_head_link"/>
   <joint
     name="${name}_arm_head_joint"

Commit message: Handle properly invalid simultaneous camera-tools and ft sensor

File: triago_description/robots/triago.urdf.xacro (robot description, xacro)
@@ -78,5 +78,5 @@
   <xacro:property name="camera_position_head" value="$(arg camera_position_head)"/>
   <xacro:property name="has_arm_left" value="${arm_type_left not in ['no-arm']}"/>
-  <xacro:property name="has_ft_sensor_left" value="${ft_sensor_left not in ['no-ft-sensor'] and end_effector_left not in ['camera-tools']}"/>
+  <xacro:property name="has_ft_sensor_left" value="${ft_sensor_left not in ['no-ft-sensor']}"/>
   <xacro:property name="has_end_effector_left" value="${end_effector_left not in ['no-end-effector']}" />
   <xacro:property name="end_effector_left_link" value="${'wrist_left_ft_tool_link' if has_ft_sensor_left else 'arm_left_tool_link'}" />
@@ -84,5 +84,5 @@
   <xacro:property name="tool_changer_left" value="${has_end_effector_left or has_ft_sensor_left}"/>
   <xacro:property name="has_arm_right" value="${arm_type_right not in ['no-arm']}"/>
-  <xacro:property name="has_ft_sensor_right" value="${ft_sensor_right not in ['no-ft-sensor'] and end_effector_right not in ['camera-tools']}"/>
+  <xacro:property name="has_ft_sensor_right" value="${ft_sensor_right not in ['no-ft-sensor']}"/>
   <xacro:property name="has_end_effector_right" value="${end_effector_right not in ['no-end-effector']}" />
   <xacro:property name="end_effector_right_link" value="${'wrist_right_ft_tool_link' if has_ft_sensor_right else 'arm_right_tool_link'}" />
@@ -90,5 +90,5 @@
   <xacro:property name="tool_changer_right" value="${has_end_effector_right or has_ft_sensor_right }"/>
   <xacro:property name="has_arm_head" value="${arm_type_head not in ['no-arm']}"/>
-  <xacro:property name="has_ft_sensor_head" value="${ft_sensor_head not in ['no-ft-sensor'] and end_effector_head not in ['camera-tools']}"/>
+  <xacro:property name="has_ft_sensor_head" value="${ft_sensor_head not in ['no-ft-sensor']}"/>
   <xacro:property name="has_end_effector_head" value="${end_effector_head not in ['no-end-effector']}" />
   <xacro:property name="end_effector_head_link" value="${'wrist_head_ft_tool_link' if has_ft_sensor_head else 'arm_head_tool_link'}" />
@@ -129,4 +129,13 @@
   <xacro:if value="${ft_sensor_head not in ['no-ft-sensor', 'ati']}">
     <xacro:wrong_ft_sensor_head />
+  </xacro:if>
+  <xacro:if value="${end_effector_left == 'camera-tools' and has_ft_sensor_left}">
+    <xacro:wrong_ft_sensor_left_camera_tools />
+  </xacro:if>
+  <xacro:if value="${end_effector_right == 'camera-tools' and has_ft_sensor_right}">
+    <xacro:wrong_ft_sensor_right_camera_tools />
+  </xacro:if>
+  <xacro:if value="${end_effector_head == 'camera-tools' and has_ft_sensor_head}">
+    <xacro:wrong_ft_sensor_head_camera_tools />
   </xacro:if>
   <xacro:if value="${laser_model not in ['no-laser', 'sick-571']}">

Commit message: Add has_torque_estimation

File: triago_description/robots/triago.urdf.xacro (robot description, xacro)
@@ -42,4 +42,6 @@
   <xacro:arg name="tool_changer_right" default="true" />
   <xacro:arg name="tool_changer_head" default="true" />
+  <!-- False, True -->
+  <xacro:arg name="torque_estimation" default="False" />
   <xacro:arg name="use_sim_time" default="false"/>
   <xacro:arg name="is_public_sim" default="false"/>
@@ -57,4 +59,5 @@
   <xacro:arg name="camera_position_head" default="down" />
   <!-- PROPERTIES -->
+  <xacro:property name="torque_estimation" value="$(arg torque_estimation)" />
   <xacro:property name="use_sim_time" value="$(arg use_sim_time)" />
   <xacro:property name="is_multiple" value="$(arg is_multiple)" />

File: triago_description/ros2_control/ros2_control.urdf.xacro (robot description, xacro)
@@ -22,11 +22,11 @@
     <!-- arm left -->
     <xacro:if value="${has_arm_left}">
-      <xacro:ros2_control_arm name="arm_left_1" reduction="1.0" offset_value="${arm_left_1_joint_offset}" />
-      <xacro:ros2_control_arm name="arm_left_2" reduction="1.0" offset_value="${arm_left_2_joint_offset}" />
-      <xacro:ros2_control_arm name="arm_left_3" reduction="1.0" offset_value="${arm_left_3_joint_offset}" />
-      <xacro:ros2_control_arm name="arm_left_4" reduction="1.0" offset_value="${arm_left_4_joint_offset}" />
-      <xacro:ros2_control_arm name="arm_left_5" reduction="1.0" offset_value="${arm_left_5_joint_offset}" />
-      <xacro:ros2_control_arm name="arm_left_6" reduction="1.0" offset_value="${arm_left_6_joint_offset}" />
-      <xacro:ros2_control_arm name="arm_left_7" reduction="1.0" offset_value="${arm_left_7_joint_offset}" />
+      <xacro:ros2_control_arm name="arm_left_1" reduction="121.0" offset_value="${arm_left_1_joint_offset}" use_sea_transmission="${torque_estimation}" />
+      <xacro:ros2_control_arm name="arm_left_2" reduction="121.0" offset_value="${arm_left_2_joint_offset}" use_sea_transmission="${torque_estimation}" />
+      <xacro:ros2_control_arm name="arm_left_3" reduction="101.0" offset_value="${arm_left_3_joint_offset}" use_sea_transmission="${torque_estimation}" />
+      <xacro:ros2_control_arm name="arm_left_4" reduction="101.0" offset_value="${arm_left_4_joint_offset}" use_sea_transmission="${torque_estimation}" />
+      <xacro:ros2_control_arm name="arm_left_5" reduction="101.0" offset_value="${arm_left_5_joint_offset}" use_sea_transmission="${torque_estimation}" />
+      <xacro:ros2_control_arm name="arm_left_6" reduction="101.0" offset_value="${arm_left_6_joint_offset}" use_sea_transmission="${torque_estimation}" />
+      <xacro:ros2_control_arm name="arm_left_7" reduction="101.0" offset_value="${arm_left_7_joint_offset}" use_sea_transmission="${torque_estimation}" />
       <xacro:if value="${has_ft_sensor_left}">
         <xacro:include filename="$(find pal_sea_arm_description)/urdf/sensors/ft_sensor/sensor.ros2_control.xacro"/>
@@ -39,11 +39,11 @@
     <!-- arm right -->
     <xacro:if value="${has_arm_right}">
-      <xacro:ros2_control_arm name="arm_right_1" reduction="1.0" offset_value="${arm_right_1_joint_offset}" />
-      <xacro:ros2_control_arm name="arm_right_2" reduction="1.0" offset_value="${arm_right_2_joint_offset}" />
-      <xacro:ros2_control_arm name="arm_right_3" reduction="1.0" offset_value="${arm_right_3_joint_offset}" />
-      <xacro:ros2_control_arm name="arm_right_4" reduction="1.0" offset_value="${arm_right_4_joint_offset}" />
-      <xacro:ros2_control_arm name="arm_right_5" reduction="1.0" offset_value="${arm_right_5_joint_offset}" />
-      <xacro:ros2_control_arm name="arm_right_6" reduction="1.0" offset_value="${arm_right_6_joint_offset}" />
-      <xacro:ros2_control_arm name="arm_right_7" reduction="1.0" offset_value="${arm_right_7_joint_offset}" />
+      <xacro:ros2_control_arm name="arm_right_1" reduction="121.0" offset_value="${arm_right_1_joint_offset}" use_sea_transmission="${torque_estimation}" />
+      <xacro:ros2_control_arm name="arm_right_2" reduction="121.0" offset_value="${arm_right_2_joint_offset}" use_sea_transmission="${torque_estimation}" />
+      <xacro:ros2_control_arm name="arm_right_3" reduction="101.0" offset_value="${arm_right_3_joint_offset}" use_sea_transmission="${torque_estimation}" />
+      <xacro:ros2_control_arm name="arm_right_4" reduction="101.0" offset_value="${arm_right_4_joint_offset}" use_sea_transmission="${torque_estimation}" />
+      <xacro:ros2_control_arm name="arm_right_5" reduction="101.0" offset_value="${arm_right_5_joint_offset}" use_sea_transmission="${torque_estimation}" />
+      <xacro:ros2_control_arm name="arm_right_6" reduction="101.0" offset_value="${arm_right_6_joint_offset}" use_sea_transmission="${torque_estimation}" />
+      <xacro:ros2_control_arm name="arm_right_7" reduction="101.0" offset_value="${arm_right_7_joint_offset}" use_sea_transmission="${torque_estimation}" />
       <xacro:if value="${has_ft_sensor_right}">
         <xacro:include filename="$(find pal_sea_arm_description)/urdf/sensors/ft_sensor/sensor.ros2_control.xacro"/>
@@ -57,11 +57,11 @@
       <!-- arm head -->
     <xacro:if value="${has_arm_head}">
-      <xacro:ros2_control_arm name="arm_head_1" reduction="1.0" offset_value="${arm_head_1_joint_offset}" />
-      <xacro:ros2_control_arm name="arm_head_2" reduction="1.0" offset_value="${arm_head_2_joint_offset}" />
-      <xacro:ros2_control_arm name="arm_head_3" reduction="1.0" offset_value="${arm_head_3_joint_offset}" />
-      <xacro:ros2_control_arm name="arm_head_4" reduction="1.0" offset_value="${arm_head_4_joint_offset}" />
-      <xacro:ros2_control_arm name="arm_head_5" reduction="1.0" offset_value="${arm_head_5_joint_offset}" />
-      <xacro:ros2_control_arm name="arm_head_6" reduction="1.0" offset_value="${arm_head_6_joint_offset}" />
-      <xacro:ros2_control_arm name="arm_head_7" reduction="1.0" offset_value="${arm_head_7_joint_offset}" />
+      <xacro:ros2_control_arm name="arm_head_1" reduction="121.0" offset_value="${arm_head_1_joint_offset}" use_sea_transmission="${torque_estimation}" />
+      <xacro:ros2_control_arm name="arm_head_2" reduction="121.0" offset_value="${arm_head_2_joint_offset}" use_sea_transmission="${torque_estimation}" />
+      <xacro:ros2_control_arm name="arm_head_3" reduction="101.0" offset_value="${arm_head_3_joint_offset}" use_sea_transmission="${torque_estimation}" />
+      <xacro:ros2_control_arm name="arm_head_4" reduction="101.0" offset_value="${arm_head_4_joint_offset}" use_sea_transmission="${torque_estimation}" />
+      <xacro:ros2_control_arm name="arm_head_5" reduction="101.0" offset_value="${arm_head_5_joint_offset}" use_sea_transmission="${torque_estimation}" />
+      <xacro:ros2_control_arm name="arm_head_6" reduction="101.0" offset_value="${arm_head_6_joint_offset}" use_sea_transmission="${torque_estimation}" />
+      <xacro:ros2_control_arm name="arm_head_7" reduction="101.0" offset_value="${arm_head_7_joint_offset}" use_sea_transmission="${torque_estimation}" />
       <xacro:if value="${has_ft_sensor_head}">
         <xacro:include filename="$(find pal_sea_arm_description)/urdf/sensors/ft_sensor/sensor.ros2_control.xacro"/>

Commit message: Update triago.urdf.xacro

File: triago_description/robots/triago.urdf.xacro (robot description, xacro)
@@ -47,4 +47,5 @@
   <xacro:arg name="is_public_sim" default="false"/>
   <xacro:arg name="is_multiple" default="false"/>
+  <xacro:arg name="namespace" default="" />
   <xacro:arg name="description_calibration_dir" default="$(find triago_description)/urdf"/>
   <xacro:arg name="extrinsic_calibration_dir" default="$(find triago_description)/urdf"/>
@@ -62,4 +63,5 @@
   <xacro:property name="use_sim_time" value="$(arg use_sim_time)" />
   <xacro:property name="is_multiple" value="$(arg is_multiple)" />
+  <xacro:property name="namespace" value="$(arg namespace)" />
   <xacro:property name="laser_model" value="$(arg laser_model)" />
   <xacro:property name="arm_type_left" value="$(arg arm_type_left)" />
