Commit message: Adding cameras in urdf

File: triago_description/robots/triago.urdf.xacro (robot description, xacro)
@@ -59,4 +59,7 @@
   <xacro:arg name="camera_position_left" default="up" />
   <xacro:arg name="camera_position_head" default="down" />
+  <xacro:arg name="camera_right" default="no-camera" />
+  <xacro:arg name="camera_left" default="no-camera" />
+  <xacro:arg name="camera_head" default="no-camera" />
   <!-- PROPERTIES -->
   <xacro:property name="torque_estimation" value="$(arg torque_estimation)" />
@@ -71,4 +74,7 @@
   <xacro:property name="end_effector_right" value="$(arg end_effector_right)" />
   <xacro:property name="end_effector_head" value="$(arg end_effector_head)" />
+  <xacro:property name="camera_right" value="$(arg camera_right)" />
+  <xacro:property name="camera_left" value="$(arg camera_left)" />
+  <xacro:property name="camera_head" value="$(arg camera_head)" />
   <xacro:property name="ft_sensor_left" value="$(arg ft_sensor_left)" />
   <xacro:property name="ft_sensor_right" value="$(arg ft_sensor_right)" />
@@ -88,4 +94,5 @@
   <xacro:property name="end_effector_left_name" value="gripper_left" />
   <xacro:property name="tool_changer_left" value="${has_end_effector_left or has_ft_sensor_left}"/>
+  <xacro:property name="has_camera_left" value="${camera_left not in ['no-camera']}" />
   <xacro:property name="has_arm_right" value="${arm_type_right not in ['no-arm']}"/>
   <xacro:property name="has_ft_sensor_right" value="${ft_sensor_right not in ['no-ft-sensor']}"/>
@@ -94,4 +101,5 @@
   <xacro:property name="end_effector_right_name" value="gripper_right" />
   <xacro:property name="tool_changer_right" value="${has_end_effector_right or has_ft_sensor_right }"/>
+  <xacro:property name="has_camera_right" value="${camera_right not in ['no-camera']}"/>
   <xacro:property name="has_arm_head" value="${arm_type_head not in ['no-arm']}"/>
   <xacro:property name="has_ft_sensor_head" value="${ft_sensor_head not in ['no-ft-sensor']}"/>
@@ -107,4 +115,5 @@
     <xacro:property name="head_hand_reflect" value="1" />
   </xacro:unless>
+  <xacro:property name="has_camera_head" value="${camera_head not in ['no-camera']}" />
   <!-- Properties check -->
   <xacro:if value="${arm_type_left not in ['tiago-pro', 'tiago-pro-s', 'no-arm']}">
@@ -166,4 +175,8 @@
   <xacro:if value="${(has_arm_right or has_arm_left or has_arm_head) and (has_end_effector_right or has_end_effector_left or has_end_effector_head)}">
     <xacro:include filename="$(find triago_description)/urdf/end_effector/end_effector.urdf.xacro" />
+  </xacro:if>
+  <!-- Cameras -->
+  <xacro:if value="${(has_camera_right or has_camera_left or has_camera_head)}">
+    <xacro:include filename="$(find triago_description)/urdf/camera_tool/camera_tool.urdf.xacro" />
   </xacro:if>
   <!-- Force Torque sensor -->
@@ -191,4 +204,8 @@
       <xacro:triago_end_effector name="gripper_left" parent="${end_effector_left_link}" type="${end_effector_left}" has_end_effector="${has_end_effector_left}" reflect="-1" is_dual="true" camera_position="${camera_position_left}"/>
     </xacro:if>
+     <!-- Cameras -->
+    <xacro:if value="${has_camera_left}">
+        <xacro:triago_camera_tool name="camera_left" parent="${end_effector_left_link}" type="${camera_left}" has_camera="${has_camera_left}" camera_position="${camera_position_left}"/>
+    </xacro:if>
     <!-- FT sensors -->
     <xacro:if value="${has_ft_sensor_left}">
@@ -206,4 +223,8 @@
       <xacro:triago_end_effector name="gripper_right" parent="${end_effector_right_link}" type="${end_effector_right}" has_end_effector="${has_end_effector_right}" reflect="1" is_dual="true" camera_position="${camera_position_right}"/>
     </xacro:if>
+    <!-- Cameras -->
+    <xacro:if value="${has_camera_right}">
+            <xacro:triago_camera_tool name="camera_right" parent="${end_effector_right_link}" type="${camera_right}" has_camera="${has_camera_right}" camera_position="${camera_position_right}"/>
+    </xacro:if>
     <!-- FT sensors -->
     <xacro:if value="${has_ft_sensor_right}">
@@ -221,4 +242,8 @@
       <xacro:triago_end_effector name="gripper_head" parent="${end_effector_head_link}" type="${end_effector_head}" has_end_effector="${has_end_effector_head}" reflect="${head_hand_reflect}" is_dual="true" camera_position="${camera_position_head}"/>
     </xacro:if>
+     <!-- Cameras -->
+    <xacro:if value="${has_camera_head}">
+        <xacro:triago_camera_tool name="camera_head" parent="${end_effector_head_link}" type="${camera_head}" has_camera="${has_camera_head}" camera_position="${camera_position_head}"/>
+    </xacro:if>
     <!-- FT sensors -->
     <xacro:if value="${has_ft_sensor_head}">

Commit message: Fix position camera tool

File: triago_description/robots/triago.urdf.xacro (robot description, xacro)
@@ -93,5 +93,5 @@
   <xacro:property name="end_effector_left_link" value="${'wrist_left_ft_tool_link' if has_ft_sensor_left else 'arm_left_tool_link'}" />
   <xacro:property name="end_effector_left_name" value="gripper_left" />
-  <xacro:property name="tool_changer_left" value="${has_end_effector_left or has_ft_sensor_left}"/>
+  <xacro:property name="tool_changer_left" value="$(arg tool_changer_left)"/>
   <xacro:property name="has_camera_left" value="${camera_left not in ['no-camera']}" />
   <xacro:property name="has_arm_right" value="${arm_type_right not in ['no-arm']}"/>
@@ -100,5 +100,5 @@
   <xacro:property name="end_effector_right_link" value="${'wrist_right_ft_tool_link' if has_ft_sensor_right else 'arm_right_tool_link'}" />
   <xacro:property name="end_effector_right_name" value="gripper_right" />
-  <xacro:property name="tool_changer_right" value="${has_end_effector_right or has_ft_sensor_right }"/>
+  <xacro:property name="tool_changer_right" value="$(arg tool_changer_right)"/>
   <xacro:property name="has_camera_right" value="${camera_right not in ['no-camera']}"/>
   <xacro:property name="has_arm_head" value="${arm_type_head not in ['no-arm']}"/>
@@ -108,5 +108,5 @@
   <xacro:property name="hand_head_type" value="$(arg hand_head_type)" />
   <xacro:property name="end_effector_head_name" value="gripper" />
-  <xacro:property name="tool_changer_head" value="${has_end_effector_head or has_ft_sensor_head}"/>
+  <xacro:property name="tool_changer_head" value="$(arg tool_changer_head)"/>
   <xacro:if value="${hand_head_type == 'left'}">
     <xacro:property name="head_hand_reflect" value="-1" />
@@ -152,13 +152,4 @@
   <xacro:if value="${ft_sensor_head not in ['no-ft-sensor', 'ati']}">
     <xacro:wrong_ft_sensor_head />
-  </xacro:if>
-  <xacro:if value="${end_effector_left == 'camera-tools' and has_ft_sensor_left}">
-    <xacro:wrong_ft_sensor_left_camera_tools />
-  </xacro:if>
-  <xacro:if value="${end_effector_right == 'camera-tools' and has_ft_sensor_right}">
-    <xacro:wrong_ft_sensor_right_camera_tools />
-  </xacro:if>
-  <xacro:if value="${end_effector_head == 'camera-tools' and has_ft_sensor_head}">
-    <xacro:wrong_ft_sensor_head_camera_tools />
   </xacro:if>
   <xacro:if value="${laser_model not in ['no-laser', 'sick-571']}">
@@ -215,5 +206,5 @@
      <!-- Cameras -->
     <xacro:if value="${has_camera_left}">
-        <xacro:triago_camera_tool name="camera_left" parent="${end_effector_left_link}" type="${camera_left}" has_camera="${has_camera_left}" camera_position="${camera_position_left}"/>
+        <xacro:triago_camera_tool name="camera_left" parent="arm_left_tool_link" type="${camera_left}" has_camera="${has_camera_left}" camera_position="${camera_position_left}"/>
     </xacro:if>
     <!-- FT sensors -->
@@ -234,5 +225,5 @@
     <!-- Cameras -->
     <xacro:if value="${has_camera_right}">
-            <xacro:triago_camera_tool name="camera_right" parent="${end_effector_right_link}" type="${camera_right}" has_camera="${has_camera_right}" camera_position="${camera_position_right}"/>
+            <xacro:triago_camera_tool name="camera_right" parent="arm_right_tool_link" type="${camera_right}" has_camera="${has_camera_right}" camera_position="${camera_position_right}"/>
     </xacro:if>
     <!-- FT sensors -->
@@ -253,5 +244,5 @@
      <!-- Cameras -->
     <xacro:if value="${has_camera_head}">
-        <xacro:triago_camera_tool name="camera_head" parent="${end_effector_head_link}" type="${camera_head}" has_camera="${has_camera_head}" camera_position="${camera_position_head}"/>
+        <xacro:triago_camera_tool name="camera_head" parent="arm_head_tool_link" type="${camera_head}" has_camera="${has_camera_head}" camera_position="${camera_position_head}"/>
     </xacro:if>
     <!-- FT sensors -->

Commit message: Add gazebo_version xacro argument

File: triago_description/robots/triago.urdf.xacro (robot description, xacro)
@@ -44,4 +44,5 @@
   <!-- False, True -->
   <xacro:arg name="torque_estimation" default="False" />
+  <xacro:arg name="gazebo_version" default="classic"/>
   <xacro:arg name="use_sim_time" default="false"/>
   <xacro:arg name="is_public_sim" default="false"/>
@@ -64,4 +65,5 @@
   <!-- PROPERTIES -->
   <xacro:property name="torque_estimation" value="$(arg torque_estimation)" />
+  <xacro:property name="gazebo_version" value="$(arg gazebo_version)"/>
   <xacro:property name="use_sim_time" value="$(arg use_sim_time)" />
   <xacro:property name="is_multiple" value="$(arg is_multiple)" />

Commit message: Add arguments to support the new gazebo

File: triago_description/robots/triago.urdf.xacro (robot description, xacro)
@@ -254,4 +254,4 @@
   </xacro:if>
   <!-- ROS 2 Control -->
-  <xacro:triago_ros2_control use_sim_time="$(arg use_sim_time)" />
+  <xacro:triago_ros2_control use_sim_time="$(arg use_sim_time)" gazebo_version="${gazebo_version}" />
 </robot>

File: triago_description/ros2_control/ros2_control.urdf.xacro (robot description, xacro)
@@ -90,5 +90,5 @@
     </ros2_control>
   </xacro:macro>
-  <xacro:macro name="triago_ros2_control" params="use_sim_time:=^|false">
+  <xacro:macro name="triago_ros2_control" params="use_sim_time:=^|false gazebo_version:=^|classic">
     <xacro:arg name="arm_type_left" default="triago"/>
     <xacro:arg name="arm_type_right" default="triago"/>
@@ -131,11 +131,25 @@
       <!-- Init the ROS 2 control gazebo interface -->
       <gazebo>
-        <plugin filename="libgazebo_ros2_control.so" name="gazebo_ros2_control">
-          <parameters>$(find triago_description)/ros2_control/gazebo_controller_manager_cfg.yaml</parameters>
-        </plugin>
+        <xacro:if value="${gazebo_version == 'classic'}">
+          <plugin filename="libgazebo_ros2_control.so" name="gazebo_ros2_control">
+            <parameters>$(find tiago_pro_description)/ros2_control/gazebo_controller_manager_cfg.yaml</parameters>
+          </plugin>
+        </xacro:if>
+        <xacro:if value="${gazebo_version == 'gazebo'}">
+          <plugin filename="gz_ros2_control-system" name="gz_ros2_control::GazeboSimROS2ControlPlugin">
+            <robot_param>robot_description</robot_param>
+            <robot_param_node>robot_state_publisher</robot_param_node>
+            <parameters>$(find tiago_pro_description)/ros2_control/gazebo_controller_manager_cfg.yaml</parameters>
+          </plugin>
+        </xacro:if>
       </gazebo>
       <ros2_control name="ros2_control_gazebo_system" type="system">
         <hardware>
-          <plugin>gazebo_ros2_control/GazeboSystem</plugin>
+          <xacro:if value="${gazebo_version == 'classic'}">
+            <plugin>gazebo_ros2_control/GazeboSystem</plugin>
+          </xacro:if>
+          <xacro:if value="${gazebo_version == 'gazebo'}">
+            <plugin>gz_ros2_control/GazeboSimSystem</plugin>
+          </xacro:if>
         </hardware>
         <!-- wheels -->

File: triago_description/urdf/torso/torso.ros2_control.xacro (robot description, xacro)
@@ -16,5 +16,7 @@
     <joint name="${name}_joint">
       <command_interface name="position" />
-      <command_interface name="velocity" />
+      <xacro:if value="${gazebo_version == 'classic'}">
+        <command_interface name="velocity" />
+      </xacro:if>
       <state_interface name="position" />
       <state_interface name="velocity" />

File: triago_description/urdf/torso/torso_dual.urdf.xacro (robot description, xacro)
@@ -112,4 +112,12 @@
     </collision>
   </link>
+  <!-- TODO: set lower limit back to 0 when moving to Gazebo Harmonic or ROS 2 Jazzy -->
+  <!-- See https://github.com/gazebosim/gz-sim/issues/1684 for more information -->
+  <xacro:if value="${gazebo_version == 'classic'}">
+    <xacro:property name="torso_lower_limit" value="0.0"/>
+  </xacro:if>
+  <xacro:if value="${gazebo_version == 'gazebo'}">
+    <xacro:property name="torso_lower_limit" value="-1e-3"/>
+  </xacro:if>
   <joint name="${name}_lift_joint" type="prismatic">
     <origin rpy="0.0 0.0 0.0" xyz="0.0 0.0 0.005" />
@@ -117,5 +125,5 @@
     <child link="${name}_lift_link" />
     <axis xyz="0 0 1" />
-    <limit effort="0" lower="0" upper="0.34" velocity="${torso_max_vel}" />
+    <limit effort="1000.0" lower="${torso_lower_limit}" upper="0.34" velocity="${torso_max_vel}" />
   </joint>
   <xacro:include filename="$(find pal_urdf_utils)/urdf/interaction_sensors/imu.urdf.xacro"/>

Commit message: remove _d405.urdf.xacro include

File: triago_description/robots/triago.urdf.xacro (robot description, xacro)
@@ -204,5 +204,5 @@
     <!-- End effector -->
     <xacro:if value="${has_end_effector_left}">
-      <xacro:triago_end_effector name="gripper_left" parent="${end_effector_left_link}" type="${end_effector_left}" has_end_effector="${has_end_effector_left}" reflect="-1" is_dual="true" camera_position="${camera_position_left}"/>
+      <xacro:triago_end_effector name="gripper_left" parent="${end_effector_left_link}" type="${end_effector_left}" has_end_effector="${has_end_effector_left}" reflect="-1" is_dual="true"/>
     </xacro:if>
      <!-- Cameras -->
@@ -223,5 +223,5 @@
     <!-- End effector -->
     <xacro:if value="${has_end_effector_right}">
-      <xacro:triago_end_effector name="gripper_right" parent="${end_effector_right_link}" type="${end_effector_right}" has_end_effector="${has_end_effector_right}" reflect="1" is_dual="true" camera_position="${camera_position_right}"/>
+      <xacro:triago_end_effector name="gripper_right" parent="${end_effector_right_link}" type="${end_effector_right}" has_end_effector="${has_end_effector_right}" reflect="1" is_dual="true"/>
     </xacro:if>
     <!-- Cameras -->
@@ -242,5 +242,5 @@
     <!-- End effector -->
     <xacro:if value="${has_end_effector_head}">
-      <xacro:triago_end_effector name="gripper_head" parent="${end_effector_head_link}" type="${end_effector_head}" has_end_effector="${has_end_effector_head}" reflect="${head_hand_reflect}" is_dual="true" camera_position="${camera_position_head}"/>
+      <xacro:triago_end_effector name="gripper_head" parent="${end_effector_head_link}" type="${end_effector_head}" has_end_effector="${has_end_effector_head}" reflect="${head_hand_reflect}" is_dual="true"/>
     </xacro:if>
      <!-- Cameras -->

File: triago_description/urdf/end_effector/end_effector.urdf.xacro (robot description, xacro)
@@ -20,6 +20,5 @@
     - reflect: Set to 1 for a right end effector, or to -1 for a left end effector
   -->
-  <xacro:include filename="$(find realsense2_description)/urdf/_d405.urdf.xacro" />
-  <xacro:macro name="triago_end_effector" params="name parent type has_end_effector reflect is_dual:=false camera_position">
+  <xacro:macro name="triago_end_effector" params="name parent type has_end_effector reflect is_dual:=false">
   <!-- No end-effector -->
   <xacro:if value="${not has_end_effector}">
